Commit message: change moveit config add moveit group test code no moveit servo

File: src/my_env/my_env_description/urdf/my_ur_macro.urdf.xacro (robot description, xacro)
@@ -193,4 +193,11 @@
       <origin xyz="0 0 0" rpy="0 0 0" />
     </xacro:robotiq_gripper>
+    <!-- 创建 tcp  -->
+    <link name="${tf_prefix}_tcp"/>
+    <joint name="${tf_prefix}_tcp_joint" type="fixed">
+        <origin xyz="0 0 0.14" rpy="0 0 0"/>
+        <parent link="${_robotiq_prefix}robotiq_85_base_link"/>
+        <child link="${tf_prefix}_tcp"/>
+    </joint>
   </xacro:macro>
 </robot>
