Commit message: add mujoco ros2 control demo

File: src/my_env/my_env_description/urdf/my_arm_macro.urdf.xacro (robot description, xacro)
@@ -170,10 +170,10 @@
     <!-- The default frame_name of the camera in mujoco ROS2 plugin is ${sensor name}_frame. -->
     <!-- I have to add this link to fix the problem. -->
-    <link name="${_realsense_prefix}_camera_frame"/>
+    <!-- <link name="${_realsense_prefix}_camera_frame"/>
     <joint name="${_realsense_prefix}_camera_frame_joint" type="fixed">
       <parent link="${_realsense_prefix}_link"/>
       <child link="${_realsense_prefix}_camera_frame"/>
       <origin xyz="0 0 0" rpy="0 0 0" />
-    </joint>
+    </joint> -->
     <!-- 创建 robotiq 夹爪底座 使用宏定义 -->
     <xacro:ur_to_robotiq

File: src/my_env/my_env_description/urdf/my_arm_mujoco_control.urdf.xacro (robot description, xacro)
@@ -72,9 +72,9 @@
       <state_interface name="effort"/>
     </joint>
-    <sensor name="${_ur_tf_prefix}ft_sensor">
+    <sensor name="${_ur_tf_prefix}tcp_fts_sensor">
       <param name="mujoco_type">fts</param>
       <!-- There is _no requirement_ for the mujoco_sensor_name to match the ros2_control sensor name -->
-      <param name="mujoco_sensor_name">${_ur_tf_prefix}ft_sensor</param>
-      <!-- ! 此处的 mujoco_sensor_name 对应 mjcf 的 sensor_name 为 "${mujoco_sensor_name}ft_sensor_force" 和 "${mujoco_sensor_name}ft_sensor_torque" -->
+      <param name="mujoco_sensor_name">${_ur_tf_prefix}tcp_fts_sensor</param>
+      <!-- ! 此处的 mujoco_sensor_name 对应 mjcf 的 sensor_name 为 "${mujoco_sensor_name}tcp_fts_sensor_force" 和 "${mujoco_sensor_name}tcp_fts_sensor_torque" -->
       <state_interface name="force.x"/>
       <state_interface name="force.y"/>
@@ -89,8 +89,8 @@
       <!-- The default frame_name of the camera in mujoco ROS2 plugin is ${sensor name}_frame. -->
       <!-- Parameters will be used as is -->
-      <!-- <param name="frame_name">${_realsense_tf_prefix}link</param> -->
-      <!-- <param name="info_topic">/${_realsense_tf_prefix}camera/camera_info</param> -->
-      <!-- <param name="image_topic">/${_realsense_tf_prefix}camera/image_raw</param> -->
-      <!-- <param name="depth_topic">/${_realsense_tf_prefix}camera/depth</param> -->
+      <param name="frame_name">${_realsense_tf_prefix}link</param>
+      <param name="info_topic">/${_realsense_tf_prefix}camera/camera_info</param>
+      <param name="image_topic">/${_realsense_tf_prefix}camera/color</param>
+      <param name="depth_topic">/${_realsense_tf_prefix}camera/depth</param>
     </sensor>
     <!-- Robotiq 2f85 Gripper 相关 -->

File: src/my_env/my_env_description/urdf/my_env_macro.urdf.xacro (robot description, xacro)
@@ -118,6 +118,6 @@
     <xacro:property name="arm_A_ur_prefix" value="${arm_A_tf_prefix}ur_"/> <!-- ! Match the prefix in my_arm_macro.urdf.xacro -->
     <xacro:property name="arm_B_ur_prefix" value="${arm_B_tf_prefix}ur_"/> <!-- ! Match the prefix in my_arm_macro.urdf.xacro -->
-    <xacro:property name="arm_A_realsense_prefix" value="${arm_A_tf_prefix}realsense"/> <!-- ! Match the prefix in my_arm_macro.urdf.xacro -->
-    <xacro:property name="arm_B_realsense_prefix" value="${arm_B_tf_prefix}realsense"/> <!-- ! Match the prefix in my_arm_macro.urdf.xacro -->
+    <xacro:property name="arm_A_realsense_prefix" value="${arm_A_tf_prefix}realsense_"/> <!-- ! append the '_' in the prefix -->
+    <xacro:property name="arm_B_realsense_prefix" value="${arm_B_tf_prefix}realsense_"/> <!-- ! append the '_' in the prefix -->
     <xacro:property name="arm_A_g2f85_prefix" value="${arm_A_tf_prefix}"/> <!-- ! Match the prefix in my_arm_macro.urdf.xacro -->
     <xacro:property name="arm_B_g2f85_prefix" value="${arm_B_tf_prefix}"/> <!-- ! Match the prefix in my_arm_macro.urdf.xacro -->

Commit message: mujoco control for lens assenbly

File: src/my_env/my_env_description/urdf/my_arm_macro.urdf.xacro (robot description, xacro)
@@ -167,13 +167,4 @@
       <origin xyz="0 0.0875 0.013" rpy="0 ${-pi/2} ${-pi/2}"/>
     </xacro:sensor_d435>
-    <!-- Fuck you, Mujoco ROS2 plugin. The parameters of the sensor camera are invalid -->
-    <!-- The default frame_name of the camera in mujoco ROS2 plugin is ${sensor name}_frame. -->
-    <!-- I have to add this link to fix the problem. -->
-    <!-- <link name="${_realsense_prefix}_camera_frame"/>
-    <joint name="${_realsense_prefix}_camera_frame_joint" type="fixed">
-      <parent link="${_realsense_prefix}_link"/>
-      <child link="${_realsense_prefix}_camera_frame"/>
-      <origin xyz="0 0 0" rpy="0 0 0" />
-    </joint> -->
     <!-- 创建 robotiq 夹爪底座 使用宏定义 -->
     <xacro:ur_to_robotiq

File: src/my_env/my_env_description/urdf/my_arm_mujoco_control.urdf.xacro (robot description, xacro)
@@ -76,5 +76,9 @@
       <!-- There is _no requirement_ for the mujoco_sensor_name to match the ros2_control sensor name -->
       <param name="mujoco_sensor_name">${_ur_tf_prefix}tcp_fts_sensor</param>
-      <!-- ! 此处的 mujoco_sensor_name 对应 mjcf 的 sensor_name 为 "${mujoco_sensor_name}tcp_fts_sensor_force" 和 "${mujoco_sensor_name}tcp_fts_sensor_torque" -->
+      <!-- Default value of force_mjcf_suffix is '_force' -->
+      <param name="force_mjcf_suffix">_force</param>
+      <!-- Default value of torque_mjcf_suffix is '_torque' -->
+      <param name="torque_mjcf_suffix">_torque</param>
+      <!-- 上述三个参数配合形成 mjcf 中的力和力矩传感器名称：{mujoco_sensor_name}{force_mjcf_suffix} 和 {mujoco_sensor_name}{torque_mjcf_suffix}  -->
       <state_interface name="force.x"/>
       <state_interface name="force.y"/>
@@ -86,6 +90,4 @@
       <!-- ! For cameras, the sensor name _must_ match the camera name in the MJCF -->
     <sensor name="${_realsense_tf_prefix}camera">
-      <!-- Fuck you, Mujoco ROS2 plugin. The parameters of the sensor camera are invalid -->
-      <!-- The default frame_name of the camera in mujoco ROS2 plugin is ${sensor name}_frame. -->
       <!-- Parameters will be used as is -->
       <param name="frame_name">${_realsense_tf_prefix}link</param>

File: src/my_env/my_env_description/urdf/my_env.urdf.xacro (robot description, xacro)
@@ -7,5 +7,5 @@
   <!-- UR_A 机器人参数 -->
   <xacro:arg name="arm_A_tf_prefix" default="arm_A_"/>
-  <xacro:arg name="ur_A_ur_type" default="ur5"/>
+  <xacro:arg name="ur_A_ur_type" default="ur5e"/>
   <!-- UR_B 机器人参数 -->
   <xacro:arg name="arm_B_tf_prefix" default="arm_B_"/>
@@ -25,4 +25,5 @@
     use_fake_sensor_commands="$(arg fake_sensor_commands)"
     generate_ros2_control="$(arg generate_ros2_control)"
+    mjcf_file_path=""
     ur_A_ur_type="$(arg ur_A_ur_type)"
     ur_B_ur_type="$(arg ur_B_ur_type)"

File: src/my_env/my_env_description/urdf/my_env_macro.urdf.xacro (robot description, xacro)
@@ -1,6 +1,9 @@
 <?xml version="1.0"?>
+<!-- xacro src/my_env/my_env_description/urdf/my_env.urdf.xacro -o src/my_env/my_env_mujoco/urdf/my_env_mujoco.urdf -->
+<!-- urdf2mjcf src/my_env/my_env_mujoco/urdf/my_env_mujoco.urdf -o ./src/my_env/my_env_mujoco/mjcf/my_env_mujoco.xml -m src/my_env/my_env_mujoco/meshes -c -j src/my_env/my_env_mujoco/config/config.json -->
 <robot name="my_env" xmlns:xacro="http://ros.org/wiki/xacro">
   <xacro:include filename="$(find my_env_description)/urdf/my_arm_macro.urdf.xacro"/>
   <xacro:include filename="$(find my_env_description)/urdf/my_arm_mujoco_control.urdf.xacro"/>
+  <xacro:include filename="$(find my_env_description)/urdf/len_macro.xacro"/>
   <xacro:macro name="my_env" params="
   arm_A_tf_prefix:=arm_A_
@@ -30,43 +33,271 @@
   gripper_com_port_B:=/dev/ttyUSB1
   ">
-  <!-- 定义材料 -->
-  <material name="wood">
-    <color rgba="0.65 0.5 0.39 1"/>
-  </material>
+  <!-- <material name="aluminum">
+    <color rgba="0.7 0.7 0.7 1.0"/>
+  </material> -->
   <link name="world"/>
-  <!-- 桌子-基座 joint -->
-  <joint name="world_to_table" type="fixed">
+  <!-- platform joint -->
+  <joint name="world_to_platform" type="fixed">
     <parent link="world" />
-    <child link="table" />
-    <origin xyz="0 0 0" rpy="0 0 0" />
-  </joint>
-  <!-- 桌子 link -->
-  <link name="table">
-    <visual>
-      <geometry>
-        <box size="2.0 1.2 0.8"/>
-      </geometry>
-      <origin rpy="0 0 0" xyz="0 0 0.4"/>
-      <material name="wood"/>
-    </visual>
-    <collision>
-      <geometry>
-        <box size="2.0 1.2 0.8"/>
-      </geometry>
-      <origin rpy="0 0 0" xyz="0 0 0.4"/>
-    </collision>
-  </link>
+    <child link="platform_link" />
+    <origin xyz="0 0 1.0" rpy="0 0 0" />
+  </joint>
+  <!-- platform link -->
+  <link name="platform_link">
+    <visual>
+      <geometry>
+        <mesh filename="package://my_env_description/meshes/platform.STL"/>
+      </geometry>
+      <material name="aluminum"/>
+    </visual>
+    <collision><geometry><mesh filename="package://my_env_description/meshes/platform_0.STL"/></geometry></collision>
+    <collision><geometry><mesh filename="package://my_env_description/meshes/platform_1.STL"/></geometry></collision>
+  </link>
+  <!-- basket_A link -->
+  <link name="basket_A_link">
+    <visual>
+      <geometry>
+        <mesh filename="package://my_env_description/meshes/basket.STL"/>
+      </geometry>
+      <material name="aluminum"/>
+    </visual>
+    <collision><geometry><mesh filename="package://my_env_description/meshes/basket_parts/basket_0.stl"/></geometry></collision>
+    <collision><geometry><mesh filename="package://my_env_description/meshes/basket_parts/basket_1.stl"/></geometry></collision>
+    <collision><geometry><mesh filename="package://my_env_description/meshes/basket_parts/basket_2.stl"/></geometry></collision>
+    <collision><geometry><mesh filename="package://my_env_description/meshes/basket_parts/basket_3.stl"/></geometry></collision>
+    <collision><geometry><mesh filename="package://my_env_description/meshes/basket_parts/basket_4.stl"/></geometry></collision>
+    <collision><geometry><mesh filename="package://my_env_description/meshes/basket_parts/basket_5.stl"/></geometry></collision>
+    <collision><geometry><mesh filename="package://my_env_description/meshes/basket_parts/basket_6.stl"/></geometry></collision>
+  </link>
+  <!-- basket_A joint -->
+  <joint name="platform_to_basket_A" type="fixed">
+    <parent link="platform_link"/>
+    <child link="basket_A_link"/>
+    <origin xyz="0 -0.3015 0" rpy="0 0 0" />
+  </joint>
+  <!-- basket_B link -->
+  <link name="basket_B_link">
+    <visual>
+      <geometry>
+        <mesh filename="package://my_env_description/meshes/basket.STL"/>
+      </geometry>
+      <material name="aluminum"/>
+    </visual>
+    <collision><geometry><mesh filename="package://my_env_description/meshes/basket_parts/basket_0.stl"/></geometry></collision>
+    <collision><geometry><mesh filename="package://my_env_description/meshes/basket_parts/basket_1.stl"/></geometry></collision>
+    <collision><geometry><mesh filename="package://my_env_description/meshes/basket_parts/basket_2.stl"/></geometry></collision>
+    <collision><geometry><mesh filename="package://my_env_description/meshes/basket_parts/basket_3.stl"/></geometry></collision>
+    <collision><geometry><mesh filename="package://my_env_description/meshes/basket_parts/basket_4.stl"/></geometry></collision>
+    <collision><geometry><mesh filename="package://my_env_description/meshes/basket_parts/basket_5.stl"/></geometry></collision>
+    <collision><geometry><mesh filename="package://my_env_description/meshes/basket_parts/basket_6.stl"/></geometry></collision>
+  </link>
+  <!-- basket_B joint -->
+  <joint name="platform_to_basket_B" type="fixed">
+    <parent link="platform_link"/>
+    <child link="basket_B_link"/>
+    <origin xyz="0 -0.3015 0" rpy="0 0 ${pi}" />
+  </joint>
+  <!--lens link & joint-->
+  <!-- lens_0 -->
+  <xacro:len_macro
+    link_name="lens_0_link"
+    parent_name="world"
+  >
+    <origin xyz="0.5 -0.3015 1.2" rpy="0 ${pi} ${pi/2}" />
+  </xacro:len_macro>
+  <link name="peg_0_link">
+    <visual>
+      <geometry>
+        <mesh filename="package://my_env_description/meshes/main_body_peg.STL"/>
+      </geometry>
+      <material name="aluminum"/>
+    </visual>
+    <collision><geometry><mesh filename="package://my_env_description/meshes/main_body_peg.STL"/></geometry></collision>
+  </link>
+  <joint name="platform_to_peg_0" type="fixed">
+    <parent link="platform_link"/>
+    <child link="peg_0_link"/>
+    <origin xyz="0 -0.025 0.523" rpy="${pi} 0 0" />
+  </joint>
+  <!-- lens_A1 -->
+  <xacro:len_macro
+    link_name="lens_A1_link"
+    parent_name="world"
+  >
+    <origin xyz="0.551 -0.3015 1.2" rpy="0 ${pi} ${pi/2}" />
+  </xacro:len_macro>
+  <link name="peg_A1_link">
+    <visual>
+      <geometry>
+        <mesh filename="package://my_env_description/meshes/main_body_peg.STL"/>
+      </geometry>
+      <material name="aluminum"/>
+    </visual>
+    <collision><geometry><mesh filename="package://my_env_description/meshes/main_body_peg.STL"/></geometry></collision>
+  </link>
+  <joint name="platform_to_peg_A1" type="fixed">
+    <parent link="platform_link"/>
+    <child link="peg_A1_link"/>
+    <origin xyz="${0.5*0.523} -0.025 ${0.866*0.523}" rpy="${pi} ${pi/6} 0" />
+  </joint>
+  <!-- lens_A2 -->
+  <xacro:len_macro
+    link_name="lens_A2_link"
+    parent_name="world"
+  >
+    <origin xyz="0.602 -0.3015 1.2" rpy="0 ${pi} ${pi/2}" />
+  </xacro:len_macro>
+  <link name="peg_A2_link">
+    <visual>
+      <geometry>
+        <mesh filename="package://my_env_description/meshes/main_body_peg.STL"/>
+      </geometry>
+      <material name="aluminum"/>
+    </visual>
+    <collision><geometry><mesh filename="package://my_env_description/meshes/main_body_peg.STL"/></geometry></collision>
+  </link>
+  <joint name="platform_to_peg_A2" type="fixed">
+    <parent link="platform_link"/>
+    <child link="peg_A2_link"/>
+    <origin xyz="${0.866*0.523} -0.025 ${0.5*0.523}" rpy="${pi} ${2*pi/6} 0" />
+  </joint>
+  <!-- lens_A3 -->
+  <xacro:len_macro
+    link_name="lens_A3_link"
+    parent_name="world"
+  >
+    <origin xyz="0.653 -0.3015 1.2" rpy="0 ${pi} ${pi/2}" />
+  </xacro:len_macro>
+  <link name="peg_A3_link">
+    <visual>
+      <geometry>
+        <mesh filename="package://my_env_description/meshes/main_body_peg.STL"/>
+      </geometry>
+      <material name="aluminum"/>
+    </visual>
+    <collision><geometry><mesh filename="package://my_env_description/meshes/main_body_peg.STL"/></geometry></collision>
+  </link>
+  <joint name="platform_to_peg_A3" type="fixed">
+    <parent link="platform_link"/>
+    <child link="peg_A3_link"/>
+    <origin xyz="${1*0.523} -0.025 ${0*0.523}" rpy="${pi} ${3*pi/6} 0" />
+  </joint>
+  <!-- lens_A4 -->
+  <xacro:len_macro
+    link_name="lens_A4_link"
+    parent_name="world"
+  >
+    <origin xyz="0.704 -0.3015 1.2" rpy="0 ${pi} ${pi/2}" />
+  </xacro:len_macro>
+  <link name="peg_A4_link">
+    <visual>
+      <geometry>
+        <mesh filename="package://my_env_description/meshes/main_body_peg.STL"/>
+      </geometry>
+      <material name="aluminum"/>
+    </visual>
+    <collision><geometry><mesh filename="package://my_env_description/meshes/main_body_peg.STL"/></geometry></collision>
+  </link>
+  <joint name="platform_to_peg_A4" type="fixed">
+    <parent link="platform_link"/>
+    <child link="peg_A4_link"/>
+    <origin xyz="${0.866*0.523} -0.025 ${-0.5*0.523}" rpy="${pi} ${4*pi/6} 0" />
+  </joint>
+  <!-- lens_B1 -->
+  <xacro:len_macro
+    link_name="lens_B1_link"
+    parent_name="world"
+  >
+    <origin xyz="-0.5 -0.3015 1.2" rpy="0 ${pi} ${-pi/2}" />
+  </xacro:len_macro>
+  <link name="peg_B1_link">
+    <visual>
+      <geometry>
+        <mesh filename="package://my_env_description/meshes/main_body_peg.STL"/>
+      </geometry>
+      <material name="aluminum"/>
+    </visual>
+    <collision><geometry><mesh filename="package://my_env_description/meshes/main_body_peg.STL"/></geometry></collision>
+  </link>
+  <joint name="platform_to_peg_B1" type="fixed">
+    <parent link="platform_link"/>
+    <child link="peg_B1_link"/>
+    <origin xyz="${-0.5*0.523} -0.025 ${0.866*0.523}" rpy="${pi} ${-pi/6} 0" />
+  </joint>
+  <!-- lens_B2 -->
+  <xacro:len_macro
+    link_name="lens_B2_link"
+    parent_name="world"
+  >
+    <origin xyz="-0.551 -0.3015 1.2" rpy="0 ${pi} ${-pi/2}" />
+  </xacro:len_macro>
+  <link name="peg_B2_link">
+    <visual>
+      <geometry>
+        <mesh filename="package://my_env_description/meshes/main_body_peg.STL"/>
+      </geometry>
+      <material name="aluminum"/>
+    </visual>
+    <collision><geometry><mesh filename="package://my_env_description/meshes/main_body_peg.STL"/></geometry></collision>
+  </link>
+  <joint name="platform_to_peg_B2" type="fixed">
+    <parent link="platform_link"/>
+    <child link="peg_B2_link"/>
+    <origin xyz="${-0.866*0.523} -0.025 ${0.5*0.523}" rpy="${pi} ${-2*pi/6} 0" />
+  </joint>
+  <!-- lens_B3 -->
+  <xacro:len_macro
+    link_name="lens_B3_link"
+    parent_name="world"
+  >
+    <origin xyz="-0.602 -0.3015 1.2" rpy="0 ${pi} ${-pi/2}" />
+  </xacro:len_macro>
+  <link name="peg_B3_link">
+    <visual>
+      <geometry>
+        <mesh filename="package://my_env_description/meshes/main_body_peg.STL"/>
+      </geometry>
+      <material name="aluminum"/>
+    </visual>
+    <collision><geometry><mesh filename="package://my_env_description/meshes/main_body_peg.STL"/></geometry></collision>
+  </link>
+  <joint name="platform_to_peg_B3" type="fixed">
+    <parent link="platform_link"/>
+    <child link="peg_B3_link"/>
+    <origin xyz="${-1*0.523} -0.025 ${0*0.523}" rpy="${pi} ${-3*pi/6} 0" />
+  </joint>
+  <!-- lens_B4 -->
+  <xacro:len_macro
+    link_name="lens_B4_link"
+    parent_name="world"
+  >
+    <origin xyz="-0.653 -0.3015 1.2" rpy="0 ${pi} ${-pi/2}" />
+  </xacro:len_macro>
+  <link name="peg_B4_link">
+    <visual>
+      <geometry>
+        <mesh filename="package://my_env_description/meshes/main_body_peg.STL"/>
+      </geometry>
+      <material name="aluminum"/>
+    </visual>
+    <collision><geometry><mesh filename="package://my_env_description/meshes/main_body_peg.STL"/></geometry></collision>
+  </link>
+  <joint name="platform_to_peg_B4" type="fixed">
+    <parent link="platform_link"/>
+    <child link="peg_B4_link"/>
+    <origin xyz="${-0.866*0.523} -0.025 ${-0.5*0.523}" rpy="${pi} ${-4*pi/6} 0" />
+  </joint>
   <!-- UR 安装座 link & joint -->
   <link name="ur_mount_A"/>
-  <joint name="table_to_ur_mount_A" type="fixed">
-    <parent link="table"/>
+  <joint name="world_to_ur_mount_A" type="fixed">
+    <parent link="world"/>
     <child link="ur_mount_A"/>
-    <origin xyz="0.4 0.2 0.8" rpy="0 0 ${pi/2}" />
+    <origin xyz="0.6 0.4 0.8" rpy="0 0 0" />
   </joint>
   <link name="ur_mount_B"/>
-  <joint name="table_to_ur_mount_B" type="fixed">
-    <parent link="table"/>
+  <joint name="world_to_ur_mount_B" type="fixed">
+    <parent link="world"/>
     <child link="ur_mount_B"/>
-    <origin xyz="-0.4 0.2 0.8" rpy="0 0 ${-pi/2}" />
+    <origin xyz="-0.6 0.4 0.8" rpy="0 0 ${pi}" />
   </joint>
   <!-- 创建 UR 机器人 -->
@@ -124,5 +355,5 @@
     <ros2_control name="my_env_ros2_mujoco" type="system">
       <hardware>
-        <plugin>mujoco_ros2_simulation/MujocoSystemInterface</plugin>
+        <plugin>mujoco_ros2_control/MujocoSystemInterface</plugin>
         <param name="mujoco_model">${mjcf_file_path}</param>
         <!-- Override the slowdown settings in the Simulate App and run at 3x speed -->
