Commit message: mujoco control for lens assenbly

File: src/my_env/my_env_mujoco/urdf/my_env_mujoco.urdf (robot description, URDF)
Before this commit: robot my_env, 78 links, 77 joints
Links:
- removed link arm_A_realsense_camera_frame
- removed link arm_B_realsense_camera_frame
- removed link table
- added link basket_A_link; collision mesh filename=package://my_env_description/meshes/basket_parts/basket_0.s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; collision mesh filename=package://my_env_description/meshes/basket_parts/basket_1.s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
- added link basket_B_link; collision mesh filename=package://my_env_description/meshes/basket_parts/basket_0.s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; collision mesh filename=package://my_env_description/meshes/basket_parts/basket_1.s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
- added link lens_0_link; collision mesh filename=package://my_env_description/meshes/lens_parts/lens_0.stl; collision mesh filename=package://my_env_description/meshes/lens_parts/lens_1.stl
- added link lens_A1_link; collision mesh filename=package://my_env_description/meshes/lens_parts/lens_0.stl; collision mesh filename=package://my_env_description/meshes/lens_parts/lens_1.stl
- added link lens_A2_link; collision mesh filename=package://my_env_description/meshes/lens_parts/lens_0.stl; collision mesh filename=package://my_env_description/meshes/lens_parts/lens_1.stl
- added link lens_A3_link; collision mesh filename=package://my_env_description/meshes/lens_parts/lens_0.stl; collision mesh filename=package://my_env_description/meshes/lens_parts/lens_1.stl
- added link lens_A4_link; collision mesh filename=package://my_env_description/meshes/lens_parts/lens_0.stl; collision mesh filename=package://my_env_description/meshes/lens_parts/lens_1.stl
- added link lens_B1_link; collision mesh filename=package://my_env_description/meshes/lens_parts/lens_0.stl; collision mesh filename=package://my_env_description/meshes/lens_parts/lens_1.stl
- added link lens_B2_link; collision mesh filename=package://my_env_description/meshes/lens_parts/lens_0.stl; collision mesh filename=package://my_env_description/meshes/lens_parts/lens_1.stl
- added link lens_B3_link; collision mesh filename=package://my_env_description/meshes/lens_parts/lens_0.stl; collision mesh filename=package://my_env_description/meshes/lens_parts/lens_1.stl
- added link lens_B4_link; collision mesh filename=package://my_env_description/meshes/lens_parts/lens_0.stl; collision mesh filename=package://my_env_description/meshes/lens_parts/lens_1.stl
- added link peg_0_link; collision mesh filename=package://my_env_description/meshes/main_body_peg.STL; visual mesh filename=package://my_env_description/meshes/main_body_peg.STL
- added link peg_A1_link; collision mesh filename=package://my_env_description/meshes/main_body_peg.STL; visual mesh filename=package://my_env_description/meshes/main_body_peg.STL
- added link peg_A2_link; collision mesh filename=package://my_env_description/meshes/main_body_peg.STL; visual mesh filename=package://my_env_description/meshes/main_body_peg.STL
- added link peg_A3_link; collision mesh filename=package://my_env_description/meshes/main_body_peg.STL; visual mesh filename=package://my_env_description/meshes/main_body_peg.STL
- added link peg_A4_link; collision mesh filename=package://my_env_description/meshes/main_body_peg.STL; visual mesh filename=package://my_env_description/meshes/main_body_peg.STL
- added link peg_B1_link; collision mesh filename=package://my_env_description/meshes/main_body_peg.STL; visual mesh filename=package://my_env_description/meshes/main_body_peg.STL
- added link peg_B2_link; collision mesh filename=package://my_env_description/meshes/main_body_peg.STL; visual mesh filename=package://my_env_description/meshes/main_body_peg.STL
- added link peg_B3_link; collision mesh filename=package://my_env_description/meshes/main_body_peg.STL; visual mesh filename=package://my_env_description/meshes/main_body_peg.STL
- added link peg_B4_link; collision mesh filename=package://my_env_description/meshes/main_body_peg.STL; visual mesh filename=package://my_env_description/meshes/main_body_peg.STL
- added link platform_link; collision mesh filename=package://my_env_description/meshes/platform_0.STL; collision mesh filename=package://my_env_description/meshes/platform_1.STL
- link arm_A_ur_base_link_inertia: geometry collision mesh filename=package://ur_description/meshes/ur5e/collision/base.stl; visual mesh filename=package://ur_description/meshes/ur5e/visual/base.dae
- link arm_A_ur_forearm_link: mass 2.33 -> 2.846; geometry collision mesh filename=package://ur_description/meshes/ur5e/collision/forearm.stl; visual mesh filename=package://ur_description/meshes/ur5e/visual/forearm.dae
- link arm_A_ur_shoulder_link: mass 3.7 -> 3.761; geometry collision mesh filename=package://ur_description/meshes/ur5e/collision/shoulder.stl; visual mesh filename=package://ur_description/meshes/ur5e/visual/shoulder.dae
- link arm_A_ur_upper_arm_link: mass 8.393 -> 8.058; geometry collision mesh filename=package://ur_description/meshes/ur5e/collision/upperarm.stl; visual mesh filename=package://ur_description/meshes/ur5e/visual/upperarm.dae
- link arm_A_ur_wrist_1_link: mass 1.219 -> 1.37; geometry collision mesh filename=package://ur_description/meshes/ur5e/collision/wrist1.stl; visual mesh filename=package://ur_description/meshes/ur5e/visual/wrist1.dae
- link arm_A_ur_wrist_2_link: mass 1.219 -> 1.3; geometry collision mesh filename=package://ur_description/meshes/ur5e/collision/wrist2.stl; visual mesh filename=package://ur_description/meshes/ur5e/visual/wrist2.dae
- link arm_A_ur_wrist_3_link: mass 0.1879 -> 0.365; geometry collision mesh filename=package://ur_description/meshes/ur5e/collision/wrist3.stl; visual mesh filename=package://ur_description/meshes/ur5e/visual/wrist3.dae
Joints:
- removed joint arm_A_realsense_camera_frame_joint
- removed joint arm_B_realsense_camera_frame_joint
- removed joint table_to_ur_mount_A
- removed joint table_to_ur_mount_B
- removed joint world_to_table
- added joint platform_to_basket_A: type fixed, parent platform_link, child basket_A_link, origin xyz=0 -0.3015 0 rpy=0 0 0
- added joint platform_to_basket_B: type fixed, parent platform_link, child basket_B_link, origin xyz=0 -0.3015 0 rpy=0 0 3.141592653589793
- added joint platform_to_peg_0: type fixed, parent platform_link, child peg_0_link, origin xyz=0 -0.025 0.523 rpy=3.141592653589793 0 0
- added joint platform_to_peg_A1: type fixed, parent platform_link, child peg_A1_link, origin xyz=0.2615 -0.025 0.452918 rpy=3.141592653589793 0.5235987755982988 0
- added joint platform_to_peg_A2: type fixed, parent platform_link, child peg_A2_link, origin xyz=0.452918 -0.025 0.2615 rpy=3.141592653589793 1.0471975511965976 0
- added joint platform_to_peg_A3: type fixed, parent platform_link, child peg_A3_link, origin xyz=0.523 -0.025 0.0 rpy=3.141592653589793 1.5707963267948966 0
- added joint platform_to_peg_A4: type fixed, parent platform_link, child peg_A4_link, origin xyz=0.452918 -0.025 -0.2615 rpy=3.141592653589793 2.0943951023931953 0
- added joint platform_to_peg_B1: type fixed, parent platform_link, child peg_B1_link, origin xyz=-0.2615 -0.025 0.452918 rpy=3.141592653589793 -0.5235987755982988 0
- added joint platform_to_peg_B2: type fixed, parent platform_link, child peg_B2_link, origin xyz=-0.452918 -0.025 0.2615 rpy=3.141592653589793 -1.0471975511965976 0
- added joint platform_to_peg_B3: type fixed, parent platform_link, child peg_B3_link, origin xyz=-0.523 -0.025 0.0 rpy=3.141592653589793 -1.5707963267948966 0
- added joint platform_to_peg_B4: type fixed, parent platform_link, child peg_B4_link, origin xyz=-0.452918 -0.025 -0.2615 rpy=3.141592653589793 -2.0943951023931953 0
- added joint world_to_lens_0_link: type fixed, parent world, child lens_0_link, origin xyz=0.5 -0.3015 1.2 rpy=0 3.141592653589793 1.5707963267948966
- added joint world_to_lens_A1_link: type fixed, parent world, child lens_A1_link, origin xyz=0.551 -0.3015 1.2 rpy=0 3.141592653589793 1.5707963267948966
- added joint world_to_lens_A2_link: type fixed, parent world, child lens_A2_link, origin xyz=0.602 -0.3015 1.2 rpy=0 3.141592653589793 1.5707963267948966
- added joint world_to_lens_A3_link: type fixed, parent world, child lens_A3_link, origin xyz=0.653 -0.3015 1.2 rpy=0 3.141592653589793 1.5707963267948966
- added joint world_to_lens_A4_link: type fixed, parent world, child lens_A4_link, origin xyz=0.704 -0.3015 1.2 rpy=0 3.141592653589793 1.5707963267948966
- added joint world_to_lens_B1_link: type fixed, parent world, child lens_B1_link, origin xyz=-0.5 -0.3015 1.2 rpy=0 3.141592653589793 -1.5707963267948966
- added joint world_to_lens_B2_link: type fixed, parent world, child lens_B2_link, origin xyz=-0.551 -0.3015 1.2 rpy=0 3.141592653589793 -1.5707963267948966
- added joint world_to_lens_B3_link: type fixed, parent world, child lens_B3_link, origin xyz=-0.602 -0.3015 1.2 rpy=0 3.141592653589793 -1.5707963267948966
- added joint world_to_lens_B4_link: type fixed, parent world, child lens_B4_link, origin xyz=-0.653 -0.3015 1.2 rpy=0 3.141592653589793 -1.5707963267948966
- added joint world_to_platform: type fixed, parent world, child platform_link, origin xyz=0 0 1.0 rpy=0 0 0
- added joint world_to_ur_mount_A: type fixed, parent world, child ur_mount_A, origin xyz=0.6 0.4 0.8 rpy=0 0 0
- added joint world_to_ur_mount_B: type fixed, parent world, child ur_mount_B, origin xyz=-0.6 0.4 0.8 rpy=0 0 3.141592653589793
- joint arm_A_ur_shoulder_pan_joint: origin xyz=0 0 0.089159 rpy=0 0 0 -> xyz=0 0 0.1625 rpy=0 0 0
- joint arm_A_ur_wrist_1_joint: origin xyz=-0.39225 0 0.10915 rpy=0 0 0 -> xyz=-0.3922 0 0.1333 rpy=0 0 0
- joint arm_A_ur_wrist_2_joint: origin xyz=0 -0.09465 -1.941303950897609e-11 rpy=1.570796327 0 0 -> xyz=0 -0.0997 -2.044881182297852e-11 rpy=1.570796327 0 0
- joint arm_A_ur_wrist_3_joint: origin xyz=0 0.0823 -1.688001216681175e-11 rpy=1.570796326589793 3.141592653589793 3.141592653589793 -> xyz=0 0.0996 -2.042830148012698e-11 rpy=1.570796326589793 3.141592653589793 3.141592653589793

File: src/my_env/my_env_mujoco/urdf/my_env_mujoco.urdf.xacro (robot description, xacro)
@@ -7,5 +7,5 @@
   <!-- UR_A 机器人参数 -->
   <xacro:arg name="arm_A_tf_prefix" default="arm_A_"/>
-  <xacro:arg name="ur_A_ur_type" default="ur5"/>
+  <xacro:arg name="ur_A_ur_type" default="ur5e"/>
   <!-- UR_B 机器人参数 -->
   <xacro:arg name="arm_B_tf_prefix" default="arm_B_"/>
