Commit message: mujoco control for lens assenbly

File: src/my_env/my_env_mujoco/urdf/my_env_mujoco_fixed.urdf (robot description, URDF)
Before this commit: robot my_env, 78 links, 77 joints
Links:
- removed link arm_A_realsense_camera_frame
- removed link arm_B_realsense_camera_frame
- removed link table
- added link basket_A_link; collision mesh filename=../meshes/basket_0_a307d541.stl; collision mesh filename=../meshes/basket_1_ee7564a5.stl
- added link basket_B_link; collision mesh filename=../meshes/basket_0_a307d541.stl; collision mesh filename=../meshes/basket_1_ee7564a5.stl
- added link lens_0_link; collision mesh filename=../meshes/lens_0_95837269.stl; collision mesh filename=../meshes/lens_1_0ea760e3.stl
- added link lens_A1_link; collision mesh filename=../meshes/lens_0_95837269.stl; collision mesh filename=../meshes/lens_1_0ea760e3.stl
- added link lens_A2_link; collision mesh filename=../meshes/lens_0_95837269.stl; collision mesh filename=../meshes/lens_1_0ea760e3.stl
- added link lens_A3_link; collision mesh filename=../meshes/lens_0_95837269.stl; collision mesh filename=../meshes/lens_1_0ea760e3.stl
- added link lens_A4_link; collision mesh filename=../meshes/lens_0_95837269.stl; collision mesh filename=../meshes/lens_1_0ea760e3.stl
- added link lens_B1_link; collision mesh filename=../meshes/lens_0_95837269.stl; collision mesh filename=../meshes/lens_1_0ea760e3.stl
- added link lens_B2_link; collision mesh filename=../meshes/lens_0_95837269.stl; collision mesh filename=../meshes/lens_1_0ea760e3.stl
- added link lens_B3_link; collision mesh filename=../meshes/lens_0_95837269.stl; collision mesh filename=../meshes/lens_1_0ea760e3.stl
- added link lens_B4_link; collision mesh filename=../meshes/lens_0_95837269.stl; collision mesh filename=../meshes/lens_1_0ea760e3.stl
- added link peg_0_link; collision mesh filename=../meshes/main_body_peg_f2370d47.STL; visual mesh filename=../meshes/main_body_peg_f2370d47.STL
- added link peg_A1_link; collision mesh filename=../meshes/main_body_peg_f2370d47.STL; visual mesh filename=../meshes/main_body_peg_f2370d47.STL
- added link peg_A2_link; collision mesh filename=../meshes/main_body_peg_f2370d47.STL; visual mesh filename=../meshes/main_body_peg_f2370d47.STL
- added link peg_A3_link; collision mesh filename=../meshes/main_body_peg_f2370d47.STL; visual mesh filename=../meshes/main_body_peg_f2370d47.STL
- added link peg_A4_link; collision mesh filename=../meshes/main_body_peg_f2370d47.STL; visual mesh filename=../meshes/main_body_peg_f2370d47.STL
- added link peg_B1_link; collision mesh filename=../meshes/main_body_peg_f2370d47.STL; visual mesh filename=../meshes/main_body_peg_f2370d47.STL
- added link peg_B2_link; collision mesh filename=../meshes/main_body_peg_f2370d47.STL; visual mesh filename=../meshes/main_body_peg_f2370d47.STL
- added link peg_B3_link; collision mesh filename=../meshes/main_body_peg_f2370d47.STL; visual mesh filename=../meshes/main_body_peg_f2370d47.STL
- added link peg_B4_link; collision mesh filename=../meshes/main_body_peg_f2370d47.STL; visual mesh filename=../meshes/main_body_peg_f2370d47.STL
- added link platform_link; collision mesh filename=../meshes/platform_0_0b097b69.STL; collision mesh filename=../meshes/platform_1_191e2908.STL
- link arm_A_realsense_link: geometry collision box size=0.02505 0.09 0.025; visual mesh filename=../meshes/d435_6743a526_0.obj
- link arm_A_realsense_shelf: geometry collision mesh filename=../meshes/RealSense_D435_Shelf_d359ca29.STL; visual mesh filename=../meshes/RealSense_D435_Shelf_d359ca29.STL
- link arm_A_robotiq_85_base_link: geometry collision mesh filename=../meshes/robotiq_base_e14b1363.stl; visual mesh filename=../meshes/robotiq_base_ba4c22e7_0.obj
- link arm_A_robotiq_85_left_finger_link: geometry collision mesh filename=../meshes/left_finger_1b48fede.stl; visual mesh filename=../meshes/left_finger_e1ea88f9_0.obj
- link arm_A_robotiq_85_left_finger_tip_link: geometry collision mesh filename=../meshes/left_finger_tip_c9609174.stl; visual mesh filename=../meshes/left_finger_tip_4c918411_0.obj
- link arm_A_robotiq_85_left_inner_knuckle_link: geometry collision mesh filename=../meshes/left_inner_knuckle_11ecd5a1.stl; visual mesh filename=../meshes/left_inner_knuckle_d6e20ced_0.obj
- link arm_A_robotiq_85_left_knuckle_link: geometry collision mesh filename=../meshes/left_knuckle_51d3a21e.stl; visual mesh filename=../meshes/left_knuckle_ac6d7519_0.obj
- link arm_A_robotiq_85_right_finger_link: geometry collision mesh filename=../meshes/right_finger_df3e86a5.stl; visual mesh filename=../meshes/right_finger_12094dbb_0.obj
- link arm_A_robotiq_85_right_finger_tip_link: geometry collision mesh filename=../meshes/right_finger_tip_8abbbc6d.stl; visual mesh filename=../meshes/right_finger_tip_5aafdc4f_0.obj
- link arm_A_robotiq_85_right_inner_knuckle_link: geometry collision mesh filename=../meshes/right_inner_knuckle_2c3a72a4.stl; visual mesh filename=../meshes/right_inner_knuckle_8d05a49d_0.obj
- link arm_A_robotiq_85_right_knuckle_link: geometry collision mesh filename=../meshes/right_knuckle_8dc62fad.stl; visual mesh filename=../meshes/right_knuckle_922d025b_0.obj
- link arm_A_robotiq_ur_to_robotiq_link: geometry collision mesh filename=../meshes/ur_to_robotiq_adapter_c1f8affd.stl; visual mesh filename=../meshes/ur_to_robotiq_adapter_e07b68cf_0.obj
- link arm_A_ur_base_link_inertia: geometry collision mesh filename=../meshes/base_bd1b2dd6.stl; visual mesh filename=../meshes/base_b81001a2_0.obj
- link arm_A_ur_forearm_link: mass 2.33 -> 2.846; geometry collision mesh filename=../meshes/forearm_98bdcf8e.stl; visual mesh filename=../meshes/forearm_861ccd15_0.obj
- link arm_A_ur_shoulder_link: mass 3.7 -> 3.761; geometry collision mesh filename=../meshes/shoulder_661339ad.stl; visual mesh filename=../meshes/shoulder_0fe2d913_0.obj
- link arm_A_ur_upper_arm_link: mass 8.393 -> 8.058; geometry collision mesh filename=../meshes/upperarm_d0455716.stl; visual mesh filename=../meshes/upperarm_12b51e98_0.obj
- link arm_A_ur_wrist_1_link: mass 1.219 -> 1.37; geometry collision mesh filename=../meshes/wrist1_2df87b9f.stl; visual mesh filename=../meshes/wrist1_1e3ee180_0.obj
- link arm_A_ur_wrist_2_link: mass 1.219 -> 1.3; geometry collision mesh filename=../meshes/wrist2_e6869549.stl; visual mesh filename=../meshes/wrist2_bde41993_0.obj
- link arm_A_ur_wrist_3_link: mass 0.1879 -> 0.365; geometry collision mesh filename=../meshes/wrist3_21abe53b.stl; visual mesh filename=../meshes/wrist3_8e7adc5c_0.obj
- link arm_B_realsense_link: geometry collision box size=0.02505 0.09 0.025; visual mesh filename=../meshes/d435_6743a526_0.obj
- link arm_B_realsense_shelf: geometry collision mesh filename=../meshes/RealSense_D435_Shelf_d359ca29.STL; visual mesh filename=../meshes/RealSense_D435_Shelf_d359ca29.STL
- link arm_B_robotiq_85_base_link: geometry collision mesh filename=../meshes/robotiq_base_e14b1363.stl; visual mesh filename=../meshes/robotiq_base_ba4c22e7_0.obj
- link arm_B_robotiq_85_left_finger_link: geometry collision mesh filename=../meshes/left_finger_1b48fede.stl; visual mesh filename=../meshes/left_finger_e1ea88f9_0.obj
- link arm_B_robotiq_85_left_finger_tip_link: geometry collision mesh filename=../meshes/left_finger_tip_c9609174.stl; visual mesh filename=../meshes/left_finger_tip_4c918411_0.obj
- link arm_B_robotiq_85_left_inner_knuckle_link: geometry collision mesh filename=../meshes/left_inner_knuckle_11ecd5a1.stl; visual mesh filename=../meshes/left_inner_knuckle_d6e20ced_0.obj
- link arm_B_robotiq_85_left_knuckle_link: geometry collision mesh filename=../meshes/left_knuckle_51d3a21e.stl; visual mesh filename=../meshes/left_knuckle_ac6d7519_0.obj
- link arm_B_robotiq_85_right_finger_link: geometry collision mesh filename=../meshes/right_finger_df3e86a5.stl; visual mesh filename=../meshes/right_finger_12094dbb_0.obj
- link arm_B_robotiq_85_right_finger_tip_link: geometry collision mesh filename=../meshes/right_finger_tip_8abbbc6d.stl; visual mesh filename=../meshes/right_finger_tip_5aafdc4f_0.obj
- link arm_B_robotiq_85_right_inner_knuckle_link: geometry collision mesh filename=../meshes/right_inner_knuckle_2c3a72a4.stl; visual mesh filename=../meshes/right_inner_knuckle_8d05a49d_0.obj
- link arm_B_robotiq_85_right_knuckle_link: geometry collision mesh filename=../meshes/right_knuckle_8dc62fad.stl; visual mesh filename=../meshes/right_knuckle_922d025b_0.obj
- link arm_B_robotiq_ur_to_robotiq_link: geometry collision mesh filename=../meshes/ur_to_robotiq_adapter_c1f8affd.stl; visual mesh filename=../meshes/ur_to_robotiq_adapter_e07b68cf_0.obj
- link arm_B_ur_base_link_inertia: geometry collision mesh filename=../meshes/base_bd1b2dd6.stl; visual mesh filename=../meshes/base_b81001a2_0.obj
- link arm_B_ur_forearm_link: geometry collision mesh filename=../meshes/forearm_98bdcf8e.stl; visual mesh filename=../meshes/forearm_861ccd15_0.obj
- link arm_B_ur_shoulder_link: geometry collision mesh filename=../meshes/shoulder_661339ad.stl; visual mesh filename=../meshes/shoulder_0fe2d913_0.obj
- link arm_B_ur_upper_arm_link: geometry collision mesh filename=../meshes/upperarm_d0455716.stl; visual mesh filename=../meshes/upperarm_12b51e98_0.obj
- link arm_B_ur_wrist_1_link: geometry collision mesh filename=../meshes/wrist1_2df87b9f.stl; visual mesh filename=../meshes/wrist1_1e3ee180_0.obj
- link arm_B_ur_wrist_2_link: geometry collision mesh filename=../meshes/wrist2_e6869549.stl; visual mesh filename=../meshes/wrist2_bde41993_0.obj
- link arm_B_ur_wrist_3_link: geometry collision mesh filename=../meshes/wrist3_21abe53b.stl; visual mesh filename=../meshes/wrist3_8e7adc5c_0.obj
Joints:
- removed joint arm_A_realsense_camera_frame_joint
- removed joint arm_B_realsense_camera_frame_joint
- removed joint table_to_ur_mount_A
- removed joint table_to_ur_mount_B
- removed joint world_to_table
- added joint platform_to_basket_A: type fixed, parent platform_link, child basket_A_link, origin xyz=0 -0.3015 0 rpy=0 0 0
- added joint platform_to_basket_B: type fixed, parent platform_link, child basket_B_link, origin xyz=0 -0.3015 0 rpy=0 0 3.141592653589793
- added joint platform_to_peg_0: type fixed, parent platform_link, child peg_0_link, origin xyz=0 -0.025 0.523 rpy=3.141592653589793 0 0
- added joint platform_to_peg_A1: type fixed, parent platform_link, child peg_A1_link, origin xyz=0.2615 -0.025 0.452918 rpy=3.141592653589793 0.5235987755982988 0
- added joint platform_to_peg_A2: type fixed, parent platform_link, child peg_A2_link, origin xyz=0.452918 -0.025 0.2615 rpy=3.141592653589793 1.0471975511965976 0
- added joint platform_to_peg_A3: type fixed, parent platform_link, child peg_A3_link, origin xyz=0.523 -0.025 0.0 rpy=3.141592653589793 1.5707963267948966 0
- added joint platform_to_peg_A4: type fixed, parent platform_link, child peg_A4_link, origin xyz=0.452918 -0.025 -0.2615 rpy=3.141592653589793 2.0943951023931953 0
- added joint platform_to_peg_B1: type fixed, parent platform_link, child peg_B1_link, origin xyz=-0.2615 -0.025 0.452918 rpy=3.141592653589793 -0.5235987755982988 0
- added joint platform_to_peg_B2: type fixed, parent platform_link, child peg_B2_link, origin xyz=-0.452918 -0.025 0.2615 rpy=3.141592653589793 -1.0471975511965976 0
- added joint platform_to_peg_B3: type fixed, parent platform_link, child peg_B3_link, origin xyz=-0.523 -0.025 0.0 rpy=3.141592653589793 -1.5707963267948966 0
- added joint platform_to_peg_B4: type fixed, parent platform_link, child peg_B4_link, origin xyz=-0.452918 -0.025 -0.2615 rpy=3.141592653589793 -2.0943951023931953 0
- added joint world_to_lens_0_link: type fixed, parent world, child lens_0_link, origin xyz=0.5 -0.3015 1.2 rpy=0 3.141592653589793 1.5707963267948966
- added joint world_to_lens_A1_link: type fixed, parent world, child lens_A1_link, origin xyz=0.551 -0.3015 1.2 rpy=0 3.141592653589793 1.5707963267948966
- added joint world_to_lens_A2_link: type fixed, parent world, child lens_A2_link, origin xyz=0.602 -0.3015 1.2 rpy=0 3.141592653589793 1.5707963267948966
- added joint world_to_lens_A3_link: type fixed, parent world, child lens_A3_link, origin xyz=0.653 -0.3015 1.2 rpy=0 3.141592653589793 1.5707963267948966
- added joint world_to_lens_A4_link: type fixed, parent world, child lens_A4_link, origin xyz=0.704 -0.3015 1.2 rpy=0 3.141592653589793 1.5707963267948966
- added joint world_to_lens_B1_link: type fixed, parent world, child lens_B1_link, origin xyz=-0.5 -0.3015 1.2 rpy=0 3.141592653589793 -1.5707963267948966
- added joint world_to_lens_B2_link: type fixed, parent world, child lens_B2_link, origin xyz=-0.551 -0.3015 1.2 rpy=0 3.141592653589793 -1.5707963267948966
- added joint world_to_lens_B3_link: type fixed, parent world, child lens_B3_link, origin xyz=-0.602 -0.3015 1.2 rpy=0 3.141592653589793 -1.5707963267948966
- added joint world_to_lens_B4_link: type fixed, parent world, child lens_B4_link, origin xyz=-0.653 -0.3015 1.2 rpy=0 3.141592653589793 -1.5707963267948966
- added joint world_to_platform: type fixed, parent world, child platform_link, origin xyz=0 0 1.0 rpy=0 0 0
- added joint world_to_ur_mount_A: type fixed, parent world, child ur_mount_A, origin xyz=0.6 0.4 0.8 rpy=0 0 0
- added joint world_to_ur_mount_B: type fixed, parent world, child ur_mount_B, origin xyz=-0.6 0.4 0.8 rpy=0 0 3.141592653589793
- joint arm_A_ur_shoulder_pan_joint: origin xyz=0 0 0.089159 rpy=0 0 0 -> xyz=0 0 0.1625 rpy=0 0 0
- joint arm_A_ur_wrist_1_joint: origin xyz=-0.39225 0 0.10915 rpy=0 0 0 -> xyz=-0.3922 0 0.1333 rpy=0 0 0
- joint arm_A_ur_wrist_2_joint: origin xyz=0 -0.09465 -1.941303950897609e-11 rpy=1.570796327 0 0 -> xyz=0 -0.0997 -2.044881182297852e-11 rpy=1.570796327 0 0
- joint arm_A_ur_wrist_3_joint: origin xyz=0 0.0823 -1.688001216681175e-11 rpy=1.570796326589793 3.141592653589793 3.141592653589793 -> xyz=0 0.0996 -2.042830148012698e-11 rpy=1.570796326589793 3.141592653589793 3.141592653589793
