Commit message: add global camera

File: src/my_env/my_env_description/urdf/my_env.urdf.xacro (robot description, xacro)
@@ -1,4 +1,6 @@
 <?xml version="1.0"?>
 <robot name="my_env" xmlns:xacro="http://ros.org/wiki/xacro">
+<!-- xacro src/my_env/my_env_description/urdf/my_env.urdf.xacro -o src/my_env/my_env_mujoco/urdf/my_env_mujoco.urdf -->
+<!-- urdf2mjcf src/my_env/my_env_mujoco/urdf/my_env_mujoco.urdf -o ./src/my_env/my_env_mujoco/mjcf/my_env_mujoco.xml -m src/my_env/my_env_mujoco/meshes -c -j src/my_env/my_env_mujoco/config/config.json -->
   <!-- 首先包含自定义描述宏 -->
   <xacro:include filename="$(find my_env_description)/urdf/my_env_macro.urdf.xacro"/>

File: src/my_env/my_env_description/urdf/my_env_macro.urdf.xacro (robot description, xacro)
@@ -1,5 +1,3 @@
 <?xml version="1.0"?>
-<!-- xacro src/my_env/my_env_description/urdf/my_env.urdf.xacro -o src/my_env/my_env_mujoco/urdf/my_env_mujoco.urdf -->
-<!-- urdf2mjcf src/my_env/my_env_mujoco/urdf/my_env_mujoco.urdf -o ./src/my_env/my_env_mujoco/mjcf/my_env_mujoco.xml -m src/my_env/my_env_mujoco/meshes -c -j src/my_env/my_env_mujoco/config/config.json -->
 <robot name="my_env" xmlns:xacro="http://ros.org/wiki/xacro">
   <xacro:include filename="$(find my_env_description)/urdf/my_arm_macro.urdf.xacro"/>
@@ -288,4 +286,17 @@
     <origin xyz="${-0.866*0.523} -0.025 ${-0.5*0.523}" rpy="${pi} ${-4*pi/6} 0" />
   </joint>
+  <!-- 全局相机 -->
+  <!-- 创建 RealSense 相机 使用宏定义 -->
+    <!-- params 'name' is actually tf_prefix with '_' -->
+    <xacro:sensor_d435
+      parent="world"
+      name="global_realsense"
+      use_nominal_extrinsics="false"
+      add_plug="false"
+      use_mesh="true"
+    >
+      <!-- RealSense 的基座位于相机底部的1/4螺纹孔，距离后背面10mm，底部平面距离后背2个螺纹孔所在直线12.5mm -->
+      <origin xyz="0 0.2 1.8" rpy="0 ${pi/4} ${-pi/2}"/>
+    </xacro:sensor_d435>
   <!-- UR 安装座 link & joint -->
   <link name="ur_mount_A"/>
@@ -366,4 +377,13 @@
         <param name="lidar_publish_rate">10.0</param>
       </hardware>
+      <!-- 全局相机 -->
+      <!-- ! For cameras, the sensor name _must_ match the camera name in the MJCF -->
+      <sensor name="global_realsense_camera">
+        <!-- Parameters will be used as is -->
+        <param name="frame_name">global_realsense_link</param>
+        <param name="info_topic">/global_realsense_camera/camera_info</param>
+        <param name="image_topic">/global_realsense_camera/color</param>
+        <param name="depth_topic">/global_realsense_camera/depth</param>
+      </sensor>
       <!-- 把两套机械臂的 joint/sensor 接口“塞进同一个 system”里 -->
       <xacro:my_arm_mujoco_control

File: src/my_env/my_env_mujoco/urdf/my_env_mujoco.urdf (robot description, URDF)
Before this commit: robot my_env, 96 links, 95 joints
Links:
- added link global_realsense_bottom_screw_frame
- added link global_realsense_link, mass 0.072; collision box size=0.02505 0.09 0.025; visual mesh filename=file:///opt/ros/humble/share/realsense2_description/meshes/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
Joints:
- added joint global_realsense_joint: type fixed, parent world, child global_realsense_bottom_screw_frame, origin xyz=0 0.8 2.2 rpy=0 0.7853981633974483 -1.5707963267948966
- added joint global_realsense_link_joint: type fixed, parent global_realsense_bottom_screw_frame, child global_realsense_link, origin xyz=0.010600000000000002 0.0175 0.0125 rpy=0 0 0

File: src/my_env/my_env_mujoco/urdf/my_env_mujoco.urdf.xacro (robot description, xacro)
@@ -1,4 +1,6 @@
 <?xml version="1.0"?>
 <robot name="my_env" xmlns:xacro="http://ros.org/wiki/xacro">
+<!-- xacro src/my_env/my_env_description/urdf/my_env.urdf.xacro -o src/my_env/my_env_mujoco/urdf/my_env_mujoco.urdf -->
+<!-- urdf2mjcf src/my_env/my_env_mujoco/urdf/my_env_mujoco.urdf -o ./src/my_env/my_env_mujoco/mjcf/my_env_mujoco.xml -m src/my_env/my_env_mujoco/meshes -c -j src/my_env/my_env_mujoco/config/config.json -->
   <!-- 首先包含自定义描述宏 -->
   <xacro:include filename="$(find my_env_description)/urdf/my_env_macro.urdf.xacro"/>

File: src/my_env/my_env_mujoco/urdf/my_env_mujoco_fixed.urdf (robot description, URDF)
Before this commit: robot my_env, 96 links, 95 joints
Links:
- added link global_realsense_bottom_screw_frame
- added link global_realsense_link, mass 0.072; collision box size=0.02505 0.09 0.025; visual mesh filename=../meshes/d435_6743a526_0.obj
Joints:
- added joint global_realsense_joint: type fixed, parent world, child global_realsense_bottom_screw_frame, origin xyz=0 0.8 2.2 rpy=0 0.7853981633974483 -1.5707963267948966
- added joint global_realsense_link_joint: type fixed, parent global_realsense_bottom_screw_frame, child global_realsense_link, origin xyz=0.010600000000000002 0.0175 0.0125 rpy=0 0 0
