Commit message: add pids controller for mujoco_ros2_control

File: src/my_env/my_env_description/urdf/my_arm_mujoco_control.urdf.xacro (robot description, xacro)
@@ -15,4 +15,5 @@
       <command_interface name="position"/>
       <command_interface name="velocity"/>
+      <command_interface name="effort"/>
       <state_interface name="position">
         <!-- initial position for the FakeSystem and simulation -->
@@ -25,4 +26,5 @@
       <command_interface name="position"/>
       <command_interface name="velocity"/>
+      <command_interface name="effort"/>
       <state_interface name="position">
         <!-- initial position for the FakeSystem and simulation -->
@@ -35,4 +37,5 @@
       <command_interface name="position"/>
       <command_interface name="velocity"/>
+      <command_interface name="effort"/>
       <state_interface name="position">
         <!-- initial position for the FakeSystem and simulation -->
@@ -45,4 +48,5 @@
       <command_interface name="position"/>
       <command_interface name="velocity"/>
+      <command_interface name="effort"/>
       <state_interface name="position">
         <!-- initial position for the FakeSystem and simulation -->
@@ -55,4 +59,5 @@
       <command_interface name="position"/>
       <command_interface name="velocity"/>
+      <command_interface name="effort"/>
       <state_interface name="position">
         <!-- initial position for the FakeSystem and simulation -->
@@ -65,4 +70,5 @@
       <command_interface name="position"/>
       <command_interface name="velocity"/>
+      <command_interface name="effort"/>
       <state_interface name="position">
         <!-- initial position for the FakeSystem and simulation -->

File: src/my_env/my_env_description/urdf/my_env.urdf.xacro (robot description, xacro)
@@ -28,4 +28,5 @@
     generate_ros2_control="$(arg generate_ros2_control)"
     mjcf_file_path=""
+    pids_config_file_path=""
     ur_A_ur_type="$(arg ur_A_ur_type)"
     ur_B_ur_type="$(arg ur_B_ur_type)"

File: src/my_env/my_env_description/urdf/my_env_macro.urdf.xacro (robot description, xacro)
@@ -12,4 +12,5 @@
   use_sim_mujoco:=false
   mjcf_file_path
+  pids_config_file_path
   generate_ros2_control:=false
   ur_reverse_ip:=0.0.0.0
@@ -297,5 +298,5 @@
     >
       <!-- RealSense 的基座位于相机底部的1/4螺纹孔，距离后背面10mm，底部平面距离后背2个螺纹孔所在直线12.5mm -->
-      <origin xyz="0 0.2 1.8" rpy="0 ${pi/4} ${-pi/2}"/>
+      <origin xyz="0 0.4 2.2" rpy="0 ${pi/4} ${-pi/2}"/>
     </xacro:sensor_d435>
   <!-- UR 安装座 link & joint -->
@@ -368,4 +369,5 @@
         <plugin>mujoco_ros2_control/MujocoSystemInterface</plugin>
         <param name="mujoco_model">${mjcf_file_path}</param>
+        <param name="pids_config_file">${pids_config_file_path}</param>
         <!-- Override the slowdown settings in the Simulate App and run at 3x speed -->
         <param name="sim_speed_factor">1.0</param>

File: src/my_env/my_env_mujoco/urdf/my_env_mujoco.urdf.xacro (robot description, xacro)
@@ -18,4 +18,5 @@
   <xacro:arg name="use_sim_mujoco" default="true" />
   <xacro:arg name="mjcf_file_path" default="$(find my_env_mujoco)/urdf/my_env_mujoco.xml"/>
+  <xacro:arg name="pids_config_file_path" default="$(find my_env_control)/config/mujoco_pids_config.yaml"/>
   <xacro:arg name="generate_ros2_control" default="false" />
   <!-- 夹爪和相机参数 -->
@@ -29,4 +30,5 @@
     use_sim_mujoco="$(arg use_sim_mujoco)"
     mjcf_file_path="$(arg mjcf_file_path)"
+    pids_config_file_path="$(arg pids_config_file_path)"
     generate_ros2_control="$(arg generate_ros2_control)"
     ur_A_ur_type="$(arg ur_A_ur_type)"
