Commit message: backup

File: src/my_env/my_env_description/urdf/len_macro.xacro (robot description, xacro)
@@ -7,4 +7,9 @@
   ">
   <link name="${link_name}">
+    <inertial>
+      <origin xyz="0 0 0.205" rpy="0 0 0"/>
+      <mass value="0.438"/>
+      <inertia ixx="0.003246" ixy="0.0" ixz="0.0" iyy="0.006287" iyz="0.0" izz="0.003223"/>
+    </inertial>
     <visual>
       <geometry>

File: src/my_env/my_env_description/urdf/my_arm_mujoco_control.urdf.xacro (robot description, xacro)
@@ -5,7 +5,8 @@
     realsense_tf_prefix
     g2f85_tf_prefix
+    ur_initial_positions:=${dict(shoulder_pan_joint=0.0,shoulder_lift_joint=-1.57,elbow_joint=0.0,wrist_1_joint=-1.57,wrist_2_joint=0.0,wrist_3_joint=0.0)}
   ">
     <xacro:property name="_ur_tf_prefix" value="${ur_tf_prefix}"/>
-    <xacro:property name="_ur_initial_positions" value="${dict(shoulder_pan_joint=0.0,shoulder_lift_joint=-1.57,elbow_joint=0.0,wrist_1_joint=-1.57,wrist_2_joint=0.0,wrist_3_joint=0.0)}"/>
+    <xacro:property name="_ur_initial_positions" value="${ur_initial_positions}"/>
     <xacro:property name="_realsense_tf_prefix" value="${realsense_tf_prefix}"/>
     <xacro:property name="_g2f85_tf_prefix" value="${g2f85_tf_prefix}"/>

File: src/my_env/my_env_description/urdf/my_env.urdf.xacro (robot description, xacro)
@@ -10,7 +10,9 @@
   <xacro:arg name="arm_A_tf_prefix" default="arm_A_"/>
   <xacro:arg name="ur_A_ur_type" default="ur5e"/>
+  <!-- <xacro:arg name="ur_A_initial_positions" default="${dict(shoulder_pan_joint=0.0,shoulder_lift_joint=-1.57,elbow_joint=0.0,wrist_1_joint=-1.57,wrist_2_joint=0.0,wrist_3_joint=0.0)}"/> -->
   <!-- UR_B 机器人参数 -->
   <xacro:arg name="arm_B_tf_prefix" default="arm_B_"/>
   <xacro:arg name="ur_B_ur_type" default="ur5e"/>
+  <!-- <xacro:arg name="ur_B_initial_positions" default="${dict(shoulder_pan_joint=0.0,shoulder_lift_joint=-1.57,elbow_joint=0.0,wrist_1_joint=-1.57,wrist_2_joint=0.0,wrist_3_joint=0.0)}"/> -->
   <!-- 控制参数 -->
   <xacro:arg name="use_fake_hardware" default="true" />

File: src/my_env/my_env_description/urdf/my_env_macro.urdf.xacro (robot description, xacro)
@@ -1,4 +1,6 @@
 <?xml version="1.0"?>
 <robot name="my_env" xmlns:xacro="http://ros.org/wiki/xacro">
+<!-- xacro src/my_env/my_env_description/urdf/my_env.urdf.xacro -o src/my_env/my_env_mujoco/urdf/my_env_mujoco.urdf -->
+<!-- urdf2mjcf src/my_env/my_env_mujoco/urdf/my_env_mujoco.urdf -o ./src/my_env/my_env_mujoco/mjcf/my_env_mujoco.xml -m src/my_env/my_env_mujoco/meshes -c -j src/my_env/my_env_mujoco/config/config.json -->
   <xacro:include filename="$(find my_env_description)/urdf/my_arm_macro.urdf.xacro"/>
   <xacro:include filename="$(find my_env_description)/urdf/my_arm_mujoco_control.urdf.xacro"/>
@@ -14,4 +16,6 @@
   pids_config_file_path
   generate_ros2_control:=false
+  ur_A_initial_positions:=${dict(shoulder_pan_joint=0.0,shoulder_lift_joint=-1.57,elbow_joint=0.0,wrist_1_joint=-1.57,wrist_2_joint=0.0,wrist_3_joint=0.0)}
+  ur_B_initial_positions:=${dict(shoulder_pan_joint=0.0,shoulder_lift_joint=-1.57,elbow_joint=0.0,wrist_1_joint=-1.57,wrist_2_joint=0.0,wrist_3_joint=0.0)}
   ur_reverse_ip:=0.0.0.0
   ur_headless_mode:=false
@@ -305,5 +309,5 @@
     <parent link="world"/>
     <child link="ur_mount_A"/>
-    <origin xyz="0.6 0.4 0.8" rpy="0 0 0" />
+    <origin xyz="0.6 0.3 0.8" rpy="0 0 0" />
   </joint>
   <link name="ur_mount_B"/>
@@ -311,5 +315,5 @@
     <parent link="world"/>
     <child link="ur_mount_B"/>
-    <origin xyz="-0.6 0.4 0.8" rpy="0 0 ${pi}" />
+    <origin xyz="-0.6 0.3 0.8" rpy="0 0 ${pi}" />
   </joint>
   <!-- 创建 UR 机器人 -->
@@ -365,4 +369,6 @@
     <xacro:property name="arm_A_g2f85_prefix" value="${arm_A_tf_prefix}"/> <!-- ! Match the prefix in my_arm_macro.urdf.xacro -->
     <xacro:property name="arm_B_g2f85_prefix" value="${arm_B_tf_prefix}"/> <!-- ! Match the prefix in my_arm_macro.urdf.xacro -->
+    <xacro:property name="arm_A_ur_initial_positions" value="${ur_A_initial_positions}"/>
+    <xacro:property name="arm_B_ur_initial_positions" value="${ur_B_initial_positions}"/>
     <ros2_control name="my_env_ros2_mujoco" type="system">
       <hardware>
@@ -392,9 +398,13 @@
           ur_tf_prefix="${arm_A_ur_prefix}"
           realsense_tf_prefix="${arm_A_realsense_prefix}"
-          g2f85_tf_prefix="${arm_A_g2f85_prefix}"/>
+          g2f85_tf_prefix="${arm_A_g2f85_prefix}"
+          ur_initial_positions="${arm_A_ur_initial_positions}"
+      />
       <xacro:my_arm_mujoco_control
           ur_tf_prefix="${arm_B_ur_prefix}"
           realsense_tf_prefix="${arm_B_realsense_prefix}"
-          g2f85_tf_prefix="${arm_B_g2f85_prefix}"/>
+          g2f85_tf_prefix="${arm_B_g2f85_prefix}"
+          ur_initial_positions="${arm_B_ur_initial_positions}"
+      />
     </ros2_control>
   </xacro:if>

File: src/my_env/my_env_mujoco/urdf/my_env_mujoco.urdf (robot description, URDF)
Before this commit: robot my_env, 98 links, 97 joints
Links:
- link lens_0_link: mass None -> 0.438
- link lens_A1_link: mass None -> 0.438
- link lens_A2_link: mass None -> 0.438
- link lens_A3_link: mass None -> 0.438
- link lens_A4_link: mass None -> 0.438
- link lens_B1_link: mass None -> 0.438
- link lens_B2_link: mass None -> 0.438
- link lens_B3_link: mass None -> 0.438
- link lens_B4_link: mass None -> 0.438
Joints:
- joint global_realsense_joint: origin xyz=0 0.8 2.2 rpy=0 0.7853981633974483 -1.5707963267948966 -> xyz=0 0.4 2.2 rpy=0 0.7853981633974483 -1.5707963267948966
- joint world_to_ur_mount_A: origin xyz=0.6 0.4 0.8 rpy=0 0 0 -> xyz=0.6 0.3 0.8 rpy=0 0 0
- joint world_to_ur_mount_B: origin xyz=-0.6 0.4 0.8 rpy=0 0 3.141592653589793 -> xyz=-0.6 0.3 0.8 rpy=0 0 3.141592653589793

File: src/my_env/my_env_mujoco/urdf/my_env_mujoco.urdf.xacro (robot description, xacro)
@@ -1,5 +1,5 @@
 <?xml version="1.0"?>
 <robot name="my_env" xmlns:xacro="http://ros.org/wiki/xacro">
-<!-- xacro src/my_env/my_env_description/urdf/my_env.urdf.xacro -o src/my_env/my_env_mujoco/urdf/my_env_mujoco.urdf -->
+<!-- xacro src/my_env/my_env_mujoco/urdf/my_env_mujoco.urdf.xacro -o src/my_env/my_env_mujoco/urdf/my_env_mujoco.urdf -->
 <!-- urdf2mjcf src/my_env/my_env_mujoco/urdf/my_env_mujoco.urdf -o ./src/my_env/my_env_mujoco/mjcf/my_env_mujoco.xml -m src/my_env/my_env_mujoco/meshes -c -j src/my_env/my_env_mujoco/config/config.json -->
   <!-- 首先包含自定义描述宏 -->
@@ -20,6 +20,10 @@
   <xacro:arg name="pids_config_file_path" default="$(find my_env_control)/config/mujoco_pids_config.yaml"/>
   <xacro:arg name="generate_ros2_control" default="false" />
+  <!-- <xacro:arg name="ur_A_initial_positions" default="{shoulder_pan_joint=0.0,shoulder_lift_joint=-1.57,elbow_joint=0.0,wrist_1_joint=-1.57,wrist_2_joint=0.0,wrist_3_joint=0.0}"/> -->
+  <!-- <xacro:arg name="ur_B_initial_positions" default="{shoulder_pan_joint=0.0,shoulder_lift_joint=-1.57,elbow_joint=0.0,wrist_1_joint=-1.57,wrist_2_joint=0.0,wrist_3_joint=0.0}"/> -->
   <!-- 夹爪和相机参数 -->
   <xacro:arg name="camera_use_nominal_extrinsics" default="true"/>
+  <xacro:property name="ur_A_initial_positions" value="${dict(shoulder_pan_joint=-1.57,shoulder_lift_joint=-1.27,elbow_joint=1.0,wrist_1_joint=-1.3,wrist_2_joint=-1.57,wrist_3_joint=-1.57)}"/>
+  <xacro:property name="ur_B_initial_positions" value="${dict(shoulder_pan_joint=-1.57,shoulder_lift_joint=-2.27,elbow_joint=-0.2,wrist_1_joint=-2.24,wrist_2_joint=1.57,wrist_3_joint=1.57)}"/>
   <!-- 创建包含机器人的场景描述 - 传递my_env宏需要的所有参数 -->
   <xacro:my_env
@@ -34,4 +38,6 @@
     ur_A_ur_type="$(arg ur_A_ur_type)"
     ur_B_ur_type="$(arg ur_B_ur_type)"
+    ur_A_initial_positions="${ur_A_initial_positions}"
+    ur_B_initial_positions="${ur_B_initial_positions}"
     camera_use_nominal_extrinsics="$(arg camera_use_nominal_extrinsics)"
   />

File: src/my_env/my_env_mujoco/urdf/my_env_mujoco_fixed.urdf (robot description, URDF)
Before this commit: robot my_env, 98 links, 97 joints
Links:
- link lens_0_link: mass None -> 0.438
- link lens_A1_link: mass None -> 0.438
- link lens_A2_link: mass None -> 0.438
- link lens_A3_link: mass None -> 0.438
- link lens_A4_link: mass None -> 0.438
- link lens_B1_link: mass None -> 0.438
- link lens_B2_link: mass None -> 0.438
- link lens_B3_link: mass None -> 0.438
- link lens_B4_link: mass None -> 0.438
Joints:
- joint global_realsense_joint: origin xyz=0 0.8 2.2 rpy=0 0.7853981633974483 -1.5707963267948966 -> xyz=0 0.4 2.2 rpy=0 0.7853981633974483 -1.5707963267948966
- joint world_to_ur_mount_A: origin xyz=0.6 0.4 0.8 rpy=0 0 0 -> xyz=0.6 0.3 0.8 rpy=0 0 0
- joint world_to_ur_mount_B: origin xyz=-0.6 0.4 0.8 rpy=0 0 3.141592653589793 -> xyz=-0.6 0.3 0.8 rpy=0 0 3.141592653589793
