Commit message: add car servo demo

File: src/my_env/my_env_description/urdf/my_env_macro.urdf.xacro (robot description, xacro)
@@ -23,5 +23,5 @@
     <parent link="world" />
     <child link="table" />
-    <origin xyz="0 ${0.863 + 0.05} 0" rpy="0 0 0" />
+    <origin xyz="${0.863 + 0.05} 0 0" rpy="0 0 0" />
   </joint>
   <!-- world2arm_shelf joint -->
@@ -29,5 +29,5 @@
     <parent link="world" />
     <child link="arm_shelf" />
-    <origin xyz="0 0 0.15" rpy="0 0 0" />
+    <origin xyz="0 0 0.15" rpy="0 0 ${-pi/2}" />
   </joint>
   <!-- 桌子 link -->
@@ -35,5 +35,5 @@
     <visual>
       <geometry>
-        <box size="2.7 1.0 0.765"/> # L*W*H=2.7*1.0*0.765m
+        <box size="1.0 2.7 0.765"/> # L*W*H=2.7*1.0*0.765m
       </geometry>
       <origin rpy="0 0 0" xyz="0 0 ${0.765/2}" />
@@ -42,5 +42,5 @@
     <collision>
       <geometry>
-        <box size="2.7 1.0 0.765"/> # L*W*H=2.7*1.0*0.765m
+        <box size="1.0 2.7 0.765"/> # L*W*H=2.7*1.0*0.765m
       </geometry>
       <origin rpy="0 0 0" xyz="0 0 ${0.765/2}" />

Commit message: 删除moveit servo 没用的参数，修复moveit servo的测试。修改home 关节角

File: src/my_env/my_env_description/urdf/my_env_macro.urdf.xacro (robot description, xacro)
@@ -23,5 +23,5 @@
     <parent link="world" />
     <child link="table" />
-    <origin xyz="${0.863 + 0.05} 0 0" rpy="0 0 0" />
+    <origin xyz="${0.863 + 0.02} 0 0" rpy="0 0 0" />
   </joint>
   <!-- world2arm_shelf joint -->

Commit message: 增加了 osc2 arm control

File: src/my_env/my_env_description/urdf/my_env_macro.urdf.xacro (robot description, xacro)
@@ -62,4 +62,13 @@
       <origin rpy="0 0 0" xyz="0 0 ${1.353/2}" />
     </collision>
+    <inertial>
+      <mass value="50.0"/>
+      <!-- 箱体惯性: Ixx = m/12*(y²+z²), Iyy = m/12*(x²+z²), Izz = m/12*(x²+y²) -->
+      <inertia ixx="${50.0/12.0 * (0.613*0.613 + 1.353*1.353)}"
+               ixy="0.0" ixz="0.0"
+               iyy="${50.0/12.0 * (0.726*0.726 + 1.353*1.353)}"
+               iyz="0.0"
+               izz="${50.0/12.0 * (0.726*0.726 + 0.613*0.613)}"/>
+    </inertial>
   </link>
   <!-- UR 安装座 link & joint -->

Commit message: 实现了 ocs2 控制机械臂

File: src/my_env/my_env_description/urdf/my_env_macro.urdf.xacro (robot description, xacro)
@@ -19,15 +19,20 @@
   </material>
   <link name="world"/>
+  <link name="base_link"/>
+  <joint name="world_to_base_link" type="fixed">
+    <parent link="world" />
+    <child link="base_link" />
+  </joint>
   <!-- world2tabel joint -->
   <joint name="world_to_table" type="fixed">
-    <parent link="world" />
+    <parent link="base_link" />
     <child link="table" />
-    <origin xyz="${0.863 + 0.02} 0 0" rpy="0 0 0" />
+    <origin xyz="0 ${0.863 + 0.02} 0" rpy="0 0 0" />
   </joint>
   <!-- world2arm_shelf joint -->
   <joint name="world_to_arm_shelf" type="fixed">
-    <parent link="world" />
+    <parent link="base_link" />
     <child link="arm_shelf" />
-    <origin xyz="0 0 0.15" rpy="0 0 ${-pi/2}" />
+    <origin xyz="0 0 0" rpy="0 0 0" />
   </joint>
   <!-- 桌子 link -->
@@ -35,5 +40,5 @@
     <visual>
       <geometry>
-        <box size="1.0 2.7 0.765"/> # L*W*H=2.7*1.0*0.765m
+        <box size="2.7 1.0 0.765"/> # L*W*H=2.7*1.0*0.765m
       </geometry>
       <origin rpy="0 0 0" xyz="0 0 ${0.765/2}" />
@@ -42,5 +47,5 @@
     <collision>
       <geometry>
-        <box size="1.0 2.7 0.765"/> # L*W*H=2.7*1.0*0.765m
+        <box size="2.7 1.0 0.765"/> # L*W*H=2.7*1.0*0.765m
       </geometry>
       <origin rpy="0 0 0" xyz="0 0 ${0.765/2}" />
@@ -53,5 +58,5 @@
         <mesh filename="package://my_env_description/meshes/arm_shelf.STL"/> # L*W*H=0.613*0.726*1.353m
       </geometry>
-      <origin rpy="0 0 0" xyz="0 0 0" />
+      <origin rpy="0 0 0" xyz="0 0 0.15" />
       <material name="arm_shelf_material"/>
     </visual>
@@ -60,5 +65,5 @@
         <box size="0.726 0.613 1.353"/> # L*W*H=0.726*0.613*1.353m
       </geometry>
-      <origin rpy="0 0 0" xyz="0 0 ${1.353/2}" />
+      <origin rpy="0 0 0" xyz="0 0 ${1.353/2+0.15}" />
     </collision>
     <inertial>

Commit message: 修复：修复夹爪无法接入 rviz 中夹爪控制 panel 的问题；修复 ocs2 marker 的 left 和 right 与实际机械臂左右臂相反的问题。 变更：现在控制器的初始关节位置参数不再由 launch 文件参数传入， xacro 读取默认的初始位置参数；

File: src/my_env/my_env_description/urdf/my_env_macro.urdf.xacro (robot description, xacro)
@@ -82,5 +82,5 @@
     <parent link="arm_shelf"/>
     <child link="ur_mount_A"/>
-    <origin xyz="0.431 0.1875 1.0575" rpy="0 ${pi/2} 0" />
+    <origin xyz="0.431 0.1875 1.2075" rpy="0 ${pi/2} 0" />
   </joint>
   <link name="ur_mount_B"/>
@@ -88,5 +88,5 @@
     <parent link="arm_shelf"/>
     <child link="ur_mount_B"/>
-    <origin xyz="-0.363 0.1875 1.0575" rpy="0 ${-pi/2} 0" />
+    <origin xyz="-0.363 0.1875 1.2075" rpy="0 ${-pi/2} 0" />
   </joint>
   <!-- 创建 UR 机器人 (Jazzy: 仅传几何相关参数) -->
