Commit message: 将assembly环境独立为一个文件夹，并重命名其相关文件名

File: src/my_env/my_env_description/urdf/assembly_env/assembly_env.urdf.xacro (robot description, xacro)
@@ -1,8 +1,8 @@
 <?xml version="1.0"?>
-<robot name="my_env" xmlns:xacro="http://ros.org/wiki/xacro">
-<!-- xacro src/my_env/my_env_description/urdf/my_env.urdf.xacro -o src/my_env/my_env_mujoco/urdf/my_env_mujoco.urdf -->
-<!-- urdf2mjcf src/my_env/my_env_mujoco/urdf/my_env_mujoco.urdf -o ./src/my_env/my_env_mujoco/mjcf/my_env_mujoco.xml -m src/my_env/my_env_mujoco/meshes -c -j src/my_env/my_env_mujoco/config/config.json -->
+<robot name="assembly_env" xmlns:xacro="http://ros.org/wiki/xacro">
+<!-- xacro src/my_env/my_env_description/urdf/assembly_env/assembly_env.urdf.xacro -o src/my_env/my_env_mujoco/urdf/assembly_env_mujoco.urdf -->
+<!-- urdf2mjcf src/my_env/my_env_mujoco/urdf/assembly_env_mujoco.urdf -o ./src/my_env/my_env_mujoco/mjcf/assembly_env_mujoco.xml -m src/my_env/my_env_mujoco/meshes -c -j src/my_env/my_env_mujoco/config/config.json -->
   <!-- 首先包含自定义描述宏 -->
-  <xacro:include filename="$(find my_env_description)/urdf/my_env_macro.urdf.xacro"/>
+  <xacro:include filename="$(find my_env_description)/urdf/assenmly_env/assembly_env_macro.urdf.xacro"/>
   <!-- 我们需要指定用于参数化描述的参数 -->
   <!-- 为所需的ur_type创建一个文件夹，并从ur_description包中复制文件到那里 -->
@@ -22,6 +22,6 @@
   <!-- 夹爪和相机参数 -->
   <xacro:arg name="camera_use_nominal_extrinsics" default="true"/>
-  <!-- 创建包含机器人的场景描述 - 传递my_env宏需要的所有参数 -->
-  <xacro:my_env
+  <!-- 创建包含机器人的场景描述 - 传递assembly_env宏需要的所有参数 -->
+  <xacro:assembly_env
     arm_A_tf_prefix="$(arg arm_A_tf_prefix)"
     arm_B_tf_prefix="$(arg arm_B_tf_prefix)"

File: src/my_env/my_env_description/urdf/assembly_env/assembly_env_macro.urdf.xacro (robot description, xacro)
@@ -1,10 +1,10 @@
 <?xml version="1.0"?>
-<robot name="my_env" xmlns:xacro="http://ros.org/wiki/xacro">
-<!-- xacro src/my_env/my_env_description/urdf/my_env.urdf.xacro -o src/my_env/my_env_mujoco/urdf/my_env_mujoco.urdf -->
-<!-- urdf2mjcf src/my_env/my_env_mujoco/urdf/my_env_mujoco.urdf -o ./src/my_env/my_env_mujoco/mjcf/my_env_mujoco.xml -m src/my_env/my_env_mujoco/meshes -c -j src/my_env/my_env_mujoco/config/config.json -->
+<robot name="assembly_env" xmlns:xacro="http://ros.org/wiki/xacro">
+<!-- xacro src/my_env/my_env_description/urdf/assembly_env/assembly_env.urdf.xacro -o src/my_env/my_env_mujoco/urdf/assembly_env_mujoco.urdf -->
+<!-- urdf2mjcf src/my_env/my_env_mujoco/urdf/assembly_env_mujoco.urdf -o ./src/my_env/my_env_mujoco/mjcf/assembly_env_mujoco.xml -m src/my_env/my_env_mujoco/meshes -c -j src/my_env/my_env_mujoco/config/config.json -->
   <xacro:include filename="$(find my_env_description)/urdf/my_arm_macro.urdf.xacro"/>
   <xacro:include filename="$(find my_env_description)/urdf/my_arm_mujoco_control.urdf.xacro"/>
-  <xacro:include filename="$(find my_env_description)/urdf/len_macro.xacro"/>
-  <xacro:macro name="my_env" params="
+  <xacro:include filename="$(find my_env_description)/urdf/assembly_env/len_macro.xacro"/>
+  <xacro:macro name="assembly_env" params="
   arm_A_tf_prefix:=arm_A_
   arm_B_tf_prefix:=arm_B_

File: src/my_env/my_env_mujoco/urdf/assembly_env/assembly_env_mujoco.urdf.xacro (robot description, xacro)
@@ -1,8 +1,8 @@
 <?xml version="1.0"?>
-<robot name="my_env" xmlns:xacro="http://ros.org/wiki/xacro">
-<!-- xacro src/my_env/my_env_mujoco/urdf/my_env_mujoco.urdf.xacro -o src/my_env/my_env_mujoco/urdf/my_env_mujoco.urdf -->
-<!-- urdf2mjcf src/my_env/my_env_mujoco/urdf/my_env_mujoco.urdf -o ./src/my_env/my_env_mujoco/mjcf/my_env_mujoco.xml -m src/my_env/my_env_mujoco/meshes -c -j src/my_env/my_env_mujoco/config/config.json -->
+<robot name="assembly_env_mujoco" xmlns:xacro="http://ros.org/wiki/xacro">
+<!-- xacro src/my_env/my_env_mujoco/urdf/assembly_env/assembly_env_mujoco.urdf.xacro -o src/my_env/my_env_mujoco/urdf/assembly_env/assembly_env_mujoco.urdf -->
+<!-- urdf2mjcf src/my_env/my_env_mujoco/urdf/assembly_env/assembly_env_mujoco.urdf -o ./src/my_env/my_env_mujoco/mjcf/assembly_env_mujoco.xml -m src/my_env/my_env_mujoco/meshes -c -j src/my_env/my_env_mujoco/config/assembly_config.json -->
   <!-- 首先包含自定义描述宏 -->
-  <xacro:include filename="$(find my_env_description)/urdf/my_env_macro.urdf.xacro"/>
+  <xacro:include filename="$(find my_env_description)/urdf/assembly_env/assembly_env_macro.urdf.xacro"/>
   <!-- 我们需要指定用于参数化描述的参数 -->
   <!-- 为所需的ur_type创建一个文件夹，并从ur_description包中复制文件到那里 -->
@@ -26,6 +26,6 @@
   <xacro:property name="ur_A_initial_positions" value="${dict(shoulder_pan_joint=-1.57,shoulder_lift_joint=-1.27,elbow_joint=1.0,wrist_1_joint=-1.3,wrist_2_joint=-1.57,wrist_3_joint=-1.57)}"/>
   <xacro:property name="ur_B_initial_positions" value="${dict(shoulder_pan_joint=-1.57,shoulder_lift_joint=-2.27,elbow_joint=-0.2,wrist_1_joint=-2.24,wrist_2_joint=1.57,wrist_3_joint=1.57)}"/>
-  <!-- 创建包含机器人的场景描述 - 传递my_env宏需要的所有参数 -->
-  <xacro:my_env
+  <!-- 创建包含机器人的场景描述 - 传递assembly_env宏需要的所有参数 -->
+  <xacro:assembly_env
     arm_A_tf_prefix="$(arg arm_A_tf_prefix)"
     arm_B_tf_prefix="$(arg arm_B_tf_prefix)"

File: src/my_env/my_env_mujoco/urdf/assembly_env/assembly_env_mujoco_fixed.urdf (robot description, URDF)
Before this commit: robot my_env, 98 links, 97 joints
Links:
- link arm_A_realsense_link: geometry collision box size=0.02505 0.09 0.025; visual mesh filename=../../meshes/d435_6743a526_0.obj
- link arm_A_realsense_shelf: geometry collision mesh filename=../../meshes/RealSense_D435_Shelf_d359ca29.STL; visual mesh filename=../../meshes/RealSense_D435_Shelf_d359ca29.STL
- link arm_A_robotiq_85_base_link: geometry collision mesh filename=../../meshes/robotiq_base_e14b1363.stl; visual mesh filename=../../meshes/robotiq_base_ba4c22e7_0.obj
- link arm_A_robotiq_85_left_finger_link: geometry collision mesh filename=../../meshes/left_finger_1b48fede.stl; visual mesh filename=../../meshes/left_finger_e1ea88f9_0.obj
- link arm_A_robotiq_85_left_finger_tip_link: geometry collision mesh filename=../../meshes/left_finger_tip_c9609174.stl; visual mesh filename=../../meshes/left_finger_tip_4c918411_0.obj
- link arm_A_robotiq_85_left_inner_knuckle_link: geometry collision mesh filename=../../meshes/left_inner_knuckle_11ecd5a1.stl; visual mesh filename=../../meshes/left_inner_knuckle_d6e20ced_0.obj
- link arm_A_robotiq_85_left_knuckle_link: geometry collision mesh filename=../../meshes/left_knuckle_51d3a21e.stl; visual mesh filename=../../meshes/left_knuckle_ac6d7519_0.obj
- link arm_A_robotiq_85_right_finger_link: geometry collision mesh filename=../../meshes/right_finger_df3e86a5.stl; visual mesh filename=../../meshes/right_finger_12094dbb_0.obj
- link arm_A_robotiq_85_right_finger_tip_link: geometry collision mesh filename=../../meshes/right_finger_tip_8abbbc6d.stl; visual mesh filename=../../meshes/right_finger_tip_5aafdc4f_0.obj
- link arm_A_robotiq_85_right_inner_knuckle_link: geometry collision mesh filename=../../meshes/right_inner_knuckle_2c3a72a4.stl; visual mesh filename=../../meshes/right_inner_knuckle_8d05a49d_0.obj
- link arm_A_robotiq_85_right_knuckle_link: geometry collision mesh filename=../../meshes/right_knuckle_8dc62fad.stl; visual mesh filename=../../meshes/right_knuckle_922d025b_0.obj
- link arm_A_robotiq_ur_to_robotiq_link: geometry collision mesh filename=../../meshes/ur_to_robotiq_adapter_c1f8affd.stl; visual mesh filename=../../meshes/ur_to_robotiq_adapter_e07b68cf_0.obj
- link arm_A_ur_base_link_inertia: geometry collision mesh filename=../../meshes/base_bd1b2dd6.stl; visual mesh filename=../../meshes/base_b81001a2_0.obj
- link arm_A_ur_forearm_link: geometry collision mesh filename=../../meshes/forearm_98bdcf8e.stl; visual mesh filename=../../meshes/forearm_861ccd15_0.obj
- link arm_A_ur_shoulder_link: geometry collision mesh filename=../../meshes/shoulder_661339ad.stl; visual mesh filename=../../meshes/shoulder_0fe2d913_0.obj
- link arm_A_ur_upper_arm_link: geometry collision mesh filename=../../meshes/upperarm_d0455716.stl; visual mesh filename=../../meshes/upperarm_12b51e98_0.obj
- link arm_A_ur_wrist_1_link: geometry collision mesh filename=../../meshes/wrist1_2df87b9f.stl; visual mesh filename=../../meshes/wrist1_1e3ee180_0.obj
- link arm_A_ur_wrist_2_link: geometry collision mesh filename=../../meshes/wrist2_e6869549.stl; visual mesh filename=../../meshes/wrist2_bde41993_0.obj
- link arm_A_ur_wrist_3_link: geometry collision mesh filename=../../meshes/wrist3_21abe53b.stl; visual mesh filename=../../meshes/wrist3_8e7adc5c_0.obj
- link arm_B_realsense_link: geometry collision box size=0.02505 0.09 0.025; visual mesh filename=../../meshes/d435_6743a526_0.obj
- link arm_B_realsense_shelf: geometry collision mesh filename=../../meshes/RealSense_D435_Shelf_d359ca29.STL; visual mesh filename=../../meshes/RealSense_D435_Shelf_d359ca29.STL
- link arm_B_robotiq_85_base_link: geometry collision mesh filename=../../meshes/robotiq_base_e14b1363.stl; visual mesh filename=../../meshes/robotiq_base_ba4c22e7_0.obj
- link arm_B_robotiq_85_left_finger_link: geometry collision mesh filename=../../meshes/left_finger_1b48fede.stl; visual mesh filename=../../meshes/left_finger_e1ea88f9_0.obj
- link arm_B_robotiq_85_left_finger_tip_link: geometry collision mesh filename=../../meshes/left_finger_tip_c9609174.stl; visual mesh filename=../../meshes/left_finger_tip_4c918411_0.obj
- link arm_B_robotiq_85_left_inner_knuckle_link: geometry collision mesh filename=../../meshes/left_inner_knuckle_11ecd5a1.stl; visual mesh filename=../../meshes/left_inner_knuckle_d6e20ced_0.obj
- link arm_B_robotiq_85_left_knuckle_link: geometry collision mesh filename=../../meshes/left_knuckle_51d3a21e.stl; visual mesh filename=../../meshes/left_knuckle_ac6d7519_0.obj
- link arm_B_robotiq_85_right_finger_link: geometry collision mesh filename=../../meshes/right_finger_df3e86a5.stl; visual mesh filename=../../meshes/right_finger_12094dbb_0.obj
- link arm_B_robotiq_85_right_finger_tip_link: geometry collision mesh filename=../../meshes/right_finger_tip_8abbbc6d.stl; visual mesh filename=../../meshes/right_finger_tip_5aafdc4f_0.obj
- link arm_B_robotiq_85_right_inner_knuckle_link: geometry collision mesh filename=../../meshes/right_inner_knuckle_2c3a72a4.stl; visual mesh filename=../../meshes/right_inner_knuckle_8d05a49d_0.obj
- link arm_B_robotiq_85_right_knuckle_link: geometry collision mesh filename=../../meshes/right_knuckle_8dc62fad.stl; visual mesh filename=../../meshes/right_knuckle_922d025b_0.obj
- link arm_B_robotiq_ur_to_robotiq_link: geometry collision mesh filename=../../meshes/ur_to_robotiq_adapter_c1f8affd.stl; visual mesh filename=../../meshes/ur_to_robotiq_adapter_e07b68cf_0.obj
- link arm_B_ur_base_link_inertia: geometry collision mesh filename=../../meshes/base_bd1b2dd6.stl; visual mesh filename=../../meshes/base_b81001a2_0.obj
- link arm_B_ur_forearm_link: geometry collision mesh filename=../../meshes/forearm_98bdcf8e.stl; visual mesh filename=../../meshes/forearm_861ccd15_0.obj
- link arm_B_ur_shoulder_link: geometry collision mesh filename=../../meshes/shoulder_661339ad.stl; visual mesh filename=../../meshes/shoulder_0fe2d913_0.obj
- link arm_B_ur_upper_arm_link: geometry collision mesh filename=../../meshes/upperarm_d0455716.stl; visual mesh filename=../../meshes/upperarm_12b51e98_0.obj
- link arm_B_ur_wrist_1_link: geometry collision mesh filename=../../meshes/wrist1_2df87b9f.stl; visual mesh filename=../../meshes/wrist1_1e3ee180_0.obj
- link arm_B_ur_wrist_2_link: geometry collision mesh filename=../../meshes/wrist2_e6869549.stl; visual mesh filename=../../meshes/wrist2_bde41993_0.obj
- link arm_B_ur_wrist_3_link: geometry collision mesh filename=../../meshes/wrist3_21abe53b.stl; visual mesh filename=../../meshes/wrist3_8e7adc5c_0.obj
- link basket_A_link: geometry collision mesh filename=../../meshes/basket_0_a307d541.stl; collision mesh filename=../../meshes/basket_1_ee7564a5.stl
- link basket_B_link: geometry collision mesh filename=../../meshes/basket_0_a307d541.stl; collision mesh filename=../../meshes/basket_1_ee7564a5.stl
- link global_realsense_link: geometry collision box size=0.02505 0.09 0.025; visual mesh filename=../../meshes/d435_6743a526_0.obj
- link lens_0_link: geometry collision mesh filename=../../meshes/lens_0_95837269.stl; collision mesh filename=../../meshes/lens_1_0ea760e3.stl
- link lens_A1_link: geometry collision mesh filename=../../meshes/lens_0_95837269.stl; collision mesh filename=../../meshes/lens_1_0ea760e3.stl
- link lens_A2_link: geometry collision mesh filename=../../meshes/lens_0_95837269.stl; collision mesh filename=../../meshes/lens_1_0ea760e3.stl
- link lens_A3_link: geometry collision mesh filename=../../meshes/lens_0_95837269.stl; collision mesh filename=../../meshes/lens_1_0ea760e3.stl
- link lens_A4_link: geometry collision mesh filename=../../meshes/lens_0_95837269.stl; collision mesh filename=../../meshes/lens_1_0ea760e3.stl
- link lens_B1_link: geometry collision mesh filename=../../meshes/lens_0_95837269.stl; collision mesh filename=../../meshes/lens_1_0ea760e3.stl
- link lens_B2_link: geometry collision mesh filename=../../meshes/lens_0_95837269.stl; collision mesh filename=../../meshes/lens_1_0ea760e3.stl
- link lens_B3_link: geometry collision mesh filename=../../meshes/lens_0_95837269.stl; collision mesh filename=../../meshes/lens_1_0ea760e3.stl
- link lens_B4_link: geometry collision mesh filename=../../meshes/lens_0_95837269.stl; collision mesh filename=../../meshes/lens_1_0ea760e3.stl
- link peg_0_link: geometry collision mesh filename=../../meshes/main_body_peg_f2370d47.STL; visual mesh filename=../../meshes/main_body_peg_f2370d47.STL
- link peg_A1_link: geometry collision mesh filename=../../meshes/main_body_peg_f2370d47.STL; visual mesh filename=../../meshes/main_body_peg_f2370d47.STL
- link peg_A2_link: geometry collision mesh filename=../../meshes/main_body_peg_f2370d47.STL; visual mesh filename=../../meshes/main_body_peg_f2370d47.STL
- link peg_A3_link: geometry collision mesh filename=../../meshes/main_body_peg_f2370d47.STL; visual mesh filename=../../meshes/main_body_peg_f2370d47.STL
- link peg_A4_link: geometry collision mesh filename=../../meshes/main_body_peg_f2370d47.STL; visual mesh filename=../../meshes/main_body_peg_f2370d47.STL
- link peg_B1_link: geometry collision mesh filename=../../meshes/main_body_peg_f2370d47.STL; visual mesh filename=../../meshes/main_body_peg_f2370d47.STL
- link peg_B2_link: geometry collision mesh filename=../../meshes/main_body_peg_f2370d47.STL; visual mesh filename=../../meshes/main_body_peg_f2370d47.STL
- link peg_B3_link: geometry collision mesh filename=../../meshes/main_body_peg_f2370d47.STL; visual mesh filename=../../meshes/main_body_peg_f2370d47.STL
- link peg_B4_link: geometry collision mesh filename=../../meshes/main_body_peg_f2370d47.STL; visual mesh filename=../../meshes/main_body_peg_f2370d47.STL
- link platform_link: geometry collision mesh filename=../../meshes/platform_0_0b097b69.STL; collision mesh filename=../../meshes/platform_1_191e2908.STL
