Commit message: fixed missing files; 现在ros2 control 启动文件可以选择xacro和mjcf文件

File: src/my_env/my_env_mujoco/urdf/assembly_env/assembly_env_mujoco.urdf.xacro (robot description, xacro)
@@ -17,5 +17,5 @@
   <xacro:arg name="fake_sensor_commands" default="true" />
   <xacro:arg name="use_sim_mujoco" default="true" />
-  <xacro:arg name="mjcf_file_path" default="$(find my_env_mujoco)/urdf/my_env_mujoco.xml"/>
+  <xacro:arg name="mjcf_file_path" default="$(find my_env_mujoco)/mjcf/assembly_env_mujoco.xml"/>
   <xacro:arg name="pids_config_file_path" default="$(find my_env_control)/config/mujoco_pids_config.yaml"/>
   <xacro:arg name="generate_ros2_control" default="false" />

File: src/my_env/my_env_mujoco/urdf/my_env_mujoco.urdf.xacro (robot description, xacro)
@@ -15,8 +15,12 @@
   <xacro:arg name="fake_sensor_commands" default="true" />
   <xacro:arg name="use_sim_mujoco" default="true" />
-  <xacro:arg name="mjcf_file_path" default="$(find my_env_mujoco)/urdf/my_env_mujoco.xml"/>
+  <xacro:arg name="mjcf_file_path" default="$(find my_env_mujoco)/mjcf/my_env_mujoco.xml"/>
   <xacro:arg name="generate_ros2_control" default="false" />
+  <!-- <xacro:arg name="ur_A_initial_positions" default="{shoulder_pan_joint=0.0,shoulder_lift_joint=-1.57,elbow_joint=0.0,wrist_1_joint=-1.57,wrist_2_joint=0.0,wrist_3_joint=0.0}"/> -->
+  <!-- <xacro:arg name="ur_B_initial_positions" default="{shoulder_pan_joint=0.0,shoulder_lift_joint=-1.57,elbow_joint=0.0,wrist_1_joint=-1.57,wrist_2_joint=0.0,wrist_3_joint=0.0}"/> -->
   <!-- 夹爪和相机参数 -->
   <xacro:arg name="camera_use_nominal_extrinsics" default="true"/>
+  <xacro:property name="ur_A_initial_positions" value="${dict(shoulder_pan_joint=-1.57,shoulder_lift_joint=-1.27,elbow_joint=1.0,wrist_1_joint=-1.3,wrist_2_joint=-1.57,wrist_3_joint=-1.57)}"/>
+  <xacro:property name="ur_B_initial_positions" value="${dict(shoulder_pan_joint=-1.57,shoulder_lift_joint=-2.27,elbow_joint=-0.2,wrist_1_joint=-2.24,wrist_2_joint=1.57,wrist_3_joint=1.57)}"/>
   <!-- 创建包含机器人的场景描述 - 传递my_env宏需要的所有参数 -->
   <xacro:my_env
