Commit message: 机械臂关节名前缀和机械臂类型不再能通过参数设置，而是作为属性写入my_evn_macro

File: src/my_env/my_env_control/urdf/assembly_env_control.urdf.xacro (robot description, xacro)
@@ -5,7 +5,7 @@
   <!-- 我们需要指定用于参数化描述的参数 -->
   <!-- 为所需的ur_type创建一个文件夹，并从ur_description包中复制文件到那里 -->
-  <!-- 总体参数 -->
-  <xacro:arg name="arm_A_tf_prefix" default="arm_A_"/>
-  <xacro:arg name="arm_B_tf_prefix" default="arm_B_"/>
+  <!-- 总体参数 (前缀和型号固定为 property) -->
+  <xacro:property name="arm_A_tf_prefix" value="arm_A_"/>
+  <xacro:property name="arm_B_tf_prefix" value="arm_B_"/>
   <xacro:arg name="use_fake_hardware" default="true" />
   <xacro:arg name="use_fake_sensor_commands" default="true" />
@@ -17,5 +17,5 @@
   <xacro:arg name="ur_headless_mode" default="false"/>
   <!-- UR_A 机器人参数 -->
-  <xacro:arg name="ur_A_ur_type" default="ur5"/>
+  <xacro:property name="ur_A_ur_type" value="ur5"/>
   <xacro:arg name="ur_A_robot_ip" default="192.168.1.101"/>
   <xacro:arg name="ur_A_reverse_port" default="50001"/>
@@ -24,5 +24,5 @@
   <xacro:arg name="ur_A_trajectory_port" default="50004"/>
   <!-- UR_B 机器人参数 -->
-  <xacro:arg name="ur_B_ur_type" default="ur5e"/>
+  <xacro:property name="ur_B_ur_type" value="ur5e"/>
   <xacro:arg name="ur_B_robot_ip" default="192.168.1.102"/>
   <xacro:arg name="ur_B_reverse_port" default="50011"/>
@@ -36,6 +36,6 @@
   <!-- 创建包含机器人的场景描述 - 传递assembly_env宏需要的所有参数 -->
   <xacro:assembly_env
-    arm_A_tf_prefix="$(arg arm_A_tf_prefix)"
-    arm_B_tf_prefix="$(arg arm_B_tf_prefix)"
+    arm_A_tf_prefix="${arm_A_tf_prefix}"
+    arm_B_tf_prefix="${arm_B_tf_prefix}"
     use_fake_hardware="$(arg use_fake_hardware)"
     use_fake_sensor_commands="$(arg use_fake_sensor_commands)"
@@ -45,6 +45,6 @@
     ur_reverse_ip="$(arg ur_reverse_ip)"
     ur_headless_mode="$(arg ur_headless_mode)"
-    ur_A_ur_type="$(arg ur_A_ur_type)"
-    ur_B_ur_type="$(arg ur_B_ur_type)"
+    ur_A_ur_type="${ur_A_ur_type}"
+    ur_B_ur_type="${ur_B_ur_type}"
     ur_A_robot_ip="$(arg ur_A_robot_ip)"
     ur_B_robot_ip="$(arg ur_B_robot_ip)"

File: src/my_env/my_env_control/urdf/my_env_control.urdf.xacro (robot description, xacro)
@@ -9,6 +9,4 @@
   <!-- 为所需的ur_type创建一个文件夹，并从ur_description包中复制文件到那里 -->
   <!-- 总体参数 -->
-  <xacro:arg name="arm_A_tf_prefix" default="arm_A_"/>
-  <xacro:arg name="arm_B_tf_prefix" default="arm_B_"/>
   <xacro:arg name="use_fake_hardware" default="true" />
   <xacro:arg name="use_fake_sensor_commands" default="true" />
@@ -16,6 +14,5 @@
   <xacro:arg name="ur_reverse_ip" default="0.0.0.0"/>
   <xacro:arg name="ur_headless_mode" default="false"/>
-  <!-- UR_A 机器人参数 -->
-  <xacro:arg name="ur_A_ur_type" default="ur5"/>
+  <!-- UR_A 机器人参数 (前缀和型号固定为 property) -->
   <xacro:arg name="ur_A_robot_ip" default="192.168.1.101"/>
   <xacro:arg name="ur_A_reverse_port" default="50001"/>
@@ -24,7 +21,6 @@
   <xacro:arg name="ur_A_trajectory_port" default="50004"/>
   <xacro:arg name="ur_A_rw_rate" default="0"/>
-  <xacro:arg name="ur_A_kinematics_parameters_file" default="$(find ur_description)/config/$(arg ur_A_ur_type)/default_kinematics.yaml"/>
-  <!-- UR_B 机器人参数 -->
-  <xacro:arg name="ur_B_ur_type" default="ur5e"/>
+  <xacro:arg name="ur_A_kinematics_parameters_file" default="$(find ur_description)/config/${ur_A_ur_type}/default_kinematics.yaml"/>
+  <!-- UR_B 机器人参数 (前缀和型号固定为 property) -->
   <xacro:arg name="ur_B_robot_ip" default="192.168.1.102"/>
   <xacro:arg name="ur_B_reverse_port" default="50011"/>
@@ -33,5 +29,5 @@
   <xacro:arg name="ur_B_trajectory_port" default="50014"/>
   <xacro:arg name="ur_B_rw_rate" default="0"/>
-  <xacro:arg name="ur_B_kinematics_parameters_file" default="$(find ur_description)/config/$(arg ur_B_ur_type)/default_kinematics.yaml"/>
+  <xacro:arg name="ur_B_kinematics_parameters_file" default="$(find ur_description)/config/${ur_B_ur_type}/default_kinematics.yaml"/>
   <!-- 夹爪和相机参数 -->
   <xacro:arg name="g2f85_A_com_port" default="/dev/ttyUSB0"/>
@@ -76,8 +72,4 @@
   <!-- Jazzy: 纯几何描述（仅传几何参数给 my_env） -->
   <xacro:my_env
-    arm_A_tf_prefix="$(arg arm_A_tf_prefix)"
-    arm_B_tf_prefix="$(arg arm_B_tf_prefix)"
-    ur_A_ur_type="$(arg ur_A_ur_type)"
-    ur_B_ur_type="$(arg ur_B_ur_type)"
     camera_use_nominal_extrinsics="$(arg camera_use_nominal_extrinsics)"
     safety_limits="$(arg safety_limits)"
@@ -92,6 +84,6 @@
   <xacro:ur_ros2_control
     name="ur_A"
-    tf_prefix="$(arg arm_A_tf_prefix)ur_"
-    kinematics_parameters_file="$(find ur_description)/config/$(arg ur_A_ur_type)/default_kinematics.yaml"
+    tf_prefix="${arm_A_tf_prefix}ur_"
+    kinematics_parameters_file="$(find ur_description)/config/${ur_A_ur_type}/default_kinematics.yaml"
     robot_ip="$(arg ur_A_robot_ip)"
     script_filename="$(arg script_filename)"
@@ -124,6 +116,6 @@
   <xacro:ur_ros2_control
     name="ur_B"
-    tf_prefix="$(arg arm_B_tf_prefix)ur_"
-    kinematics_parameters_file="$(find ur_description)/config/$(arg ur_B_ur_type)/default_kinematics.yaml"
+    tf_prefix="${arm_B_tf_prefix}ur_"
+    kinematics_parameters_file="$(find ur_description)/config/${ur_B_ur_type}/default_kinematics.yaml"
     robot_ip="$(arg ur_B_robot_ip)"
     script_filename="$(arg script_filename)"
@@ -159,5 +151,5 @@
   <xacro:robotiq_gripper_ros2_control
     name="arm_A_g2f85"
-    prefix="$(arg arm_A_tf_prefix)"
+    prefix="${arm_A_tf_prefix}"
     use_fake_hardware="True"
     mock_sensor_commands="$(arg use_fake_sensor_commands)"
@@ -176,5 +168,5 @@
   <xacro:robotiq_gripper_ros2_control
     name="arm_B_g2f85"
-    prefix="$(arg arm_B_tf_prefix)"
+    prefix="${arm_B_tf_prefix}"
     use_fake_hardware="True"
     mock_sensor_commands="$(arg use_fake_sensor_commands)"

File: src/my_env/my_env_description/urdf/my_env.urdf.xacro (robot description, xacro)
@@ -5,10 +5,4 @@
   <!-- 我们需要指定用于参数化描述的参数 -->
   <!-- 为所需的ur_type创建一个文件夹，并从ur_description包中复制文件到那里 -->
-  <!-- UR_A 机器人参数 -->
-  <xacro:arg name="arm_A_tf_prefix" default="arm_A_"/>
-  <xacro:arg name="ur_A_ur_type" default="ur5"/>
-  <!-- UR_B 机器人参数 -->
-  <xacro:arg name="arm_B_tf_prefix" default="arm_B_"/>
-  <xacro:arg name="ur_B_ur_type" default="ur5e"/>
   <!-- 夹爪和相机参数 -->
   <xacro:arg name="camera_use_nominal_extrinsics" default="true"/>
@@ -20,8 +14,4 @@
   <!-- Jazzy: 纯描述入口，用于 RViz/MoveIt，不包含 ros2_control -->
   <xacro:my_env
-    arm_A_tf_prefix="$(arg arm_A_tf_prefix)"
-    arm_B_tf_prefix="$(arg arm_B_tf_prefix)"
-    ur_A_ur_type="$(arg ur_A_ur_type)"
-    ur_B_ur_type="$(arg ur_B_ur_type)"
     camera_use_nominal_extrinsics="$(arg camera_use_nominal_extrinsics)"
     safety_limits="$(arg safety_limits)"

File: src/my_env/my_env_description/urdf/my_env_macro.urdf.xacro (robot description, xacro)
@@ -4,8 +4,4 @@
   <!-- Jazzy: 纯几何描述，不包含 ros2_control -->
   <xacro:macro name="my_env" params="
-  arm_A_tf_prefix:=arm_A_
-  arm_B_tf_prefix:=arm_B_
-  ur_A_ur_type:=ur5
-  ur_B_ur_type:=ur5e
   camera_use_nominal_extrinsics:=true
   safety_limits:=false
@@ -14,4 +10,8 @@
   force_abs_paths:=false
   ">
+  <xacro:property name="arm_A_tf_prefix" value="arm_A_"/>
+  <xacro:property name="ur_A_ur_type" value="ur5"/>
+  <xacro:property name="arm_B_tf_prefix" value="arm_B_"/>
+  <xacro:property name="ur_B_ur_type" value="ur5e"/>
   <!-- 定义材料 -->
   <material name="table_material">

File: src/my_env/my_env_mujoco/urdf/my_env_mujoco.urdf.xacro (robot description, xacro)
@@ -7,10 +7,10 @@
   <!-- 我们需要指定用于参数化描述的参数 -->
   <!-- 为所需的ur_type创建一个文件夹，并从ur_description包中复制文件到那里 -->
-  <!-- UR_A 机器人参数 -->
-  <xacro:arg name="arm_A_tf_prefix" default="arm_A_"/>
-  <xacro:arg name="ur_A_ur_type" default="ur5"/>
-  <!-- UR_B 机器人参数 -->
-  <xacro:arg name="arm_B_tf_prefix" default="arm_B_"/>
-  <xacro:arg name="ur_B_ur_type" default="ur5e"/>
+  <!-- UR_A 机器人参数 (固定为 property) -->
+  <xacro:property name="arm_A_tf_prefix" value="arm_A_"/>
+  <xacro:property name="ur_A_ur_type" value="ur5"/>
+  <!-- UR_B 机器人参数 (固定为 property) -->
+  <xacro:property name="arm_B_tf_prefix" value="arm_B_"/>
+  <xacro:property name="ur_B_ur_type" value="ur5e"/>
   <!-- 控制参数 -->
   <xacro:arg name="use_fake_hardware" default="true" />
@@ -40,8 +40,8 @@
   <!-- Jazzy: 纯几何描述（仅传几何参数给 my_env） -->
   <xacro:my_env
-    arm_A_tf_prefix="$(arg arm_A_tf_prefix)"
-    arm_B_tf_prefix="$(arg arm_B_tf_prefix)"
-    ur_A_ur_type="$(arg ur_A_ur_type)"
-    ur_B_ur_type="$(arg ur_B_ur_type)"
+    arm_A_tf_prefix="${arm_A_tf_prefix}"
+    arm_B_tf_prefix="${arm_B_tf_prefix}"
+    ur_A_ur_type="${ur_A_ur_type}"
+    ur_B_ur_type="${ur_B_ur_type}"
     camera_use_nominal_extrinsics="$(arg camera_use_nominal_extrinsics)"
     safety_limits="$(arg safety_limits)"
@@ -55,10 +55,10 @@
   <!-- ============================================ -->
   <xacro:if value="$(arg use_sim_mujoco)">
-    <xacro:property name="arm_A_ur_prefix" value="$(arg arm_A_tf_prefix)ur_"/> <!-- ! Match the prefix in my_arm_macro.urdf.xacro -->
-    <xacro:property name="arm_B_ur_prefix" value="$(arg arm_B_tf_prefix)ur_"/> <!-- ! Match the prefix in my_arm_macro.urdf.xacro -->
-    <xacro:property name="arm_A_realsense_prefix" value="$(arg arm_A_tf_prefix)realsense_"/> <!-- ! append the '_' in the prefix -->
-    <xacro:property name="arm_B_realsense_prefix" value="$(arg arm_B_tf_prefix)realsense_"/> <!-- ! append the '_' in the prefix -->
-    <xacro:property name="arm_A_g2f85_prefix" value="$(arg arm_A_tf_prefix)"/> <!-- ! Match the prefix in my_arm_macro.urdf.xacro -->
-    <xacro:property name="arm_B_g2f85_prefix" value="$(arg arm_B_tf_prefix)"/> <!-- ! Match the prefix in my_arm_macro.urdf.xacro -->
+    <xacro:property name="arm_A_ur_prefix" value="${arm_A_tf_prefix}ur_"/> <!-- ! Match the prefix in my_arm_macro.urdf.xacro -->
+    <xacro:property name="arm_B_ur_prefix" value="${arm_B_tf_prefix}ur_"/> <!-- ! Match the prefix in my_arm_macro.urdf.xacro -->
+    <xacro:property name="arm_A_realsense_prefix" value="${arm_A_tf_prefix}realsense_"/> <!-- ! append the '_' in the prefix -->
+    <xacro:property name="arm_B_realsense_prefix" value="${arm_B_tf_prefix}realsense_"/> <!-- ! append the '_' in the prefix -->
+    <xacro:property name="arm_A_g2f85_prefix" value="${arm_A_tf_prefix}"/> <!-- ! Match the prefix in my_arm_macro.urdf.xacro -->
+    <xacro:property name="arm_B_g2f85_prefix" value="${arm_B_tf_prefix}"/> <!-- ! Match the prefix in my_arm_macro.urdf.xacro -->
     <ros2_control name="my_env_ros2_mujoco" type="system">
       <hardware>
