Commit message: added mujoco ros2 control

File: src/my_env/my_env_control/urdf/my_env_control.urdf.xacro (robot description, xacro)
@@ -11,4 +11,5 @@
   <xacro:arg name="use_fake_sensor_commands" default="true" />
   <xacro:arg name="use_sim_gazebo" default="false" />
+  <xacro:arg name="use_sim_mujoco" default="false" />
   <xacro:arg name="generate_ros2_control" default="true" />
   <!-- UR 机器人其他参数 -->
@@ -40,4 +41,5 @@
     use_fake_sensor_commands="$(arg use_fake_sensor_commands)"
     use_sim_gazebo="$(arg use_sim_gazebo)"
+    use_sim_mujoco="$(arg use_sim_mujoco)"
     generate_ros2_control="$(arg generate_ros2_control)"
     ur_reverse_ip="$(arg ur_reverse_ip)"

File: src/my_env/my_env_description/urdf/my_arm_macro.urdf.xacro (robot description, xacro)
@@ -22,5 +22,5 @@
     ur_trajectory_port:=50004
     ur_headless_mode:=false
-    robotiq_com_port:=/dev/ttyUSB0
+    g2f85_com_port:=/dev/ttyUSB0
     realsense_use_nominal_extrinsics:=false
     *origin
@@ -28,5 +28,5 @@
     <!-- UR parameters -->
     <xacro:property name="_ur_name" value="${name}_ur"/>
-    <xacro:property name="_ur_tf_prefix" value="${tf_prefix}ur_"/>
+    <xacro:property name="_ur_tf_prefix" value="${tf_prefix}ur_"/> <!-- ! Match the prefix in my_env_macro.urdf.xacro -->
     <xacro:property name="_ur_parent" value="${parent}"/>
     <xacro:property name="_ur_joint_limits_parameters_file" value="$(find ur_description)/config/${ur_type}/joint_limits.yaml"/>
@@ -65,22 +65,22 @@
     <!-- RealSense parameters -->
     <xacro:property name="_realsense_name" value="${tf_prefix}realsense" />
-    <xacro:property name="_realsense_prefix" value="${tf_prefix}realsense" />
+    <xacro:property name="_realsense_prefix" value="${tf_prefix}realsense" /> <!-- ! Match the prefix in my_env_macro.urdf.xacro -->
     <xacro:property name="_realsense_use_nominal_extrinsics" value="${realsense_use_nominal_extrinsics}" />
     <xacro:property name="_realsense_add_plug" value="false" />
     <xacro:property name="_realsense_use_mesh" value="true" />
-    <!-- Robotiq parameters -->
-    <xacro:property name="_robotiq_name" value="${name}_robotiq" />
-    <xacro:property name="_robotiq_prefix" value="${tf_prefix}" />
-    <xacro:property name="_robotiq_sim_gazebo" value="${use_sim_gazebo}" />
-    <xacro:property name="_robotiq_sim_isaac" value="false" />
-    <xacro:property name="_robotiq_use_fake_hardware" value="${use_fake_hardware}" />
-    <xacro:property name="_robotiq_mock_sensor_commands" value="${use_fake_sensor_commands}" />
-    <xacro:property name="_robotiq_include_ros2_control" value="${generate_ros2_control}" />
-    <xacro:property name="_robotiq_com_port" value="${robotiq_com_port}  " />
-    <xacro:property name="_robotiq_gripper_speed_multiplier" value="1.0" />
-    <xacro:property name="_robotiq_gripper_force_multiplier" value="0.5" />
-    <xacro:property name="_robotiq_gripper_max_speed" value="0.150" />
-    <xacro:property name="_robotiq_gripper_max_force" value="235.0" />
-    <xacro:property name="_robotiq_gripper_closed_position" value="0.7929" />
+    <!-- Robotiq 2f85 gripper parameters -->
+    <xacro:property name="_g2f85_name" value="${name}_g2f85" />
+    <xacro:property name="_g2f85_prefix" value="${tf_prefix}" /> <!-- ! Match the prefix in my_env_macro.urdf.xacro -->
+    <xacro:property name="_g2f85_sim_gazebo" value="${use_sim_gazebo}" />
+    <xacro:property name="_g2f85_sim_isaac" value="false" />
+    <xacro:property name="_g2f85_use_fake_hardware" value="${use_fake_hardware}" />
+    <xacro:property name="_g2f85_mock_sensor_commands" value="${use_fake_sensor_commands}" />
+    <xacro:property name="_g2f85_include_ros2_control" value="${generate_ros2_control}" />
+    <xacro:property name="_g2f85_com_port" value="${g2f85_com_port}" />
+    <xacro:property name="_g2f85_gripper_speed_multiplier" value="1.0" />
+    <xacro:property name="_g2f85_gripper_force_multiplier" value="0.5" />
+    <xacro:property name="_g2f85_gripper_max_speed" value="0.150" />
+    <xacro:property name="_g2f85_gripper_max_force" value="235.0" />
+    <xacro:property name="_g2f85_gripper_closed_position" value="0.7929" />
     <!-- 创建 UR 机器人 使用宏定义 -->
     <xacro:ur_robot
@@ -167,27 +167,36 @@
       <origin xyz="0 0.0875 0.013" rpy="0 ${-pi/2} ${-pi/2}"/>
     </xacro:sensor_d435>
+    <!-- Fuck you, Mujoco ROS2 plugin. The parameters of the sensor camera are invalid -->
+    <!-- The default frame_name of the camera in mujoco ROS2 plugin is ${sensor name}_frame. -->
+    <!-- I have to add this link to fix the problem. -->
+    <link name="${_realsense_prefix}_camera_frame"/>
+    <joint name="${_realsense_prefix}_camera_frame_joint" type="fixed">
+      <parent link="${_realsense_prefix}_link"/>
+      <child link="${_realsense_prefix}_camera_frame"/>
+      <origin xyz="0 0 0" rpy="0 0 0" />
+    </joint>
     <!-- 创建 robotiq 夹爪底座 使用宏定义 -->
     <xacro:ur_to_robotiq
-      prefix="${_robotiq_prefix}robotiq_"
+      prefix="${_g2f85_prefix}robotiq_"
       parent="${_realsense_prefix}_shelf_child_side"
-      child="${_robotiq_prefix}robotiq_ur_to_robotiq_child_side"
+      child="${_g2f85_prefix}robotiq_ur_to_g2f85_child_side"
     >
     </xacro:ur_to_robotiq>
     <!-- 创建 robotiq 夹爪 使用宏定义 -->
     <xacro:robotiq_gripper
-      name="${_robotiq_name}"
-      prefix="${_robotiq_prefix}"
-      parent="${_robotiq_prefix}robotiq_ur_to_robotiq_child_side"
-      sim_gazebo="${_robotiq_sim_gazebo}"
-      sim_isaac="${_robotiq_sim_isaac}"
-      use_fake_hardware="${_robotiq_use_fake_hardware}"
-      mock_sensor_commands="${_robotiq_mock_sensor_commands}"
-      include_ros2_control="${_robotiq_include_ros2_control}"
-      com_port="${_robotiq_com_port}"
-      gripper_speed_multiplier="${_robotiq_gripper_speed_multiplier}"
-      gripper_force_multiplier="${_robotiq_gripper_force_multiplier}"
-      gripper_max_speed="${_robotiq_gripper_max_speed}"
-      gripper_max_force="${_robotiq_gripper_max_force}"
-      gripper_closed_position="${_robotiq_gripper_closed_position}"
+      name="${_g2f85_name}"
+      prefix="${_g2f85_prefix}"
+      parent="${_g2f85_prefix}robotiq_ur_to_g2f85_child_side"
+      sim_gazebo="${_g2f85_sim_gazebo}"
+      sim_isaac="${_g2f85_sim_isaac}"
+      use_fake_hardware="${_g2f85_use_fake_hardware}"
+      mock_sensor_commands="${_g2f85_mock_sensor_commands}"
+      include_ros2_control="${_g2f85_include_ros2_control}"
+      com_port="${_g2f85_com_port}"
+      gripper_speed_multiplier="${_g2f85_gripper_speed_multiplier}"
+      gripper_force_multiplier="${_g2f85_gripper_force_multiplier}"
+      gripper_max_speed="${_g2f85_gripper_max_speed}"
+      gripper_max_force="${_g2f85_gripper_max_force}"
+      gripper_closed_position="${_g2f85_gripper_closed_position}"
     >
       <origin xyz="0 0 0" rpy="0 0 0" />
@@ -197,5 +206,5 @@
     <joint name="${tf_prefix}_tcp_joint" type="fixed">
         <origin xyz="0 0 0.14" rpy="0 0 0"/>
-        <parent link="${_robotiq_prefix}robotiq_85_base_link"/>
+        <parent link="${_g2f85_prefix}robotiq_85_base_link"/>
         <child link="${tf_prefix}_tcp"/>
     </joint>

File: src/my_env/my_env_description/urdf/my_env_macro.urdf.xacro (robot description, xacro)
@@ -1,5 +1,6 @@
 <?xml version="1.0"?>
 <robot name="my_env" xmlns:xacro="http://ros.org/wiki/xacro">
-  <xacro:include filename="$(find my_env_description)/urdf/my_ur_macro.urdf.xacro"/>
+  <xacro:include filename="$(find my_env_description)/urdf/my_arm_macro.urdf.xacro"/>
+  <xacro:include filename="$(find my_env_description)/urdf/my_arm_mujoco_control.urdf.xacro"/>
   <xacro:macro name="my_env" params="
   arm_A_tf_prefix:=arm_A_
@@ -8,4 +9,6 @@
   use_fake_sensor_commands:=false
   use_sim_gazebo:=false
+  use_sim_mujoco:=false
+  mjcf_file_path
   generate_ros2_control:=false
   ur_reverse_ip:=0.0.0.0
@@ -84,5 +87,5 @@
     ur_trajectory_port = "${ur_A_trajectory_port}"
     ur_headless_mode = "${ur_headless_mode}"
-    robotiq_com_port = "${gripper_com_port_A}"
+    g2f85_com_port = "${gripper_com_port_A}"
     realsense_use_nominal_extrinsics = "${camera_use_nominal_extrinsics}"
   >
@@ -105,9 +108,42 @@
     ur_trajectory_port = "${ur_B_trajectory_port}"
     ur_headless_mode = "${ur_headless_mode}"
-    robotiq_com_port = "${gripper_com_port_B}"
+    g2f85_com_port = "${gripper_com_port_B}"
     realsense_use_nominal_extrinsics = "${camera_use_nominal_extrinsics}"
   >
     <origin xyz="0 0 0" rpy="0 0 0" />
   </xacro:my_arm>
+  <!-- 创建 mujoco ros2 control 相关 -->
+  <!-- 只保留一个 ros2_control system：只启动一次 MujocoSystemInterface -->
+  <xacro:if value="${use_sim_mujoco}">
+    <xacro:property name="arm_A_ur_prefix" value="${arm_A_tf_prefix}ur_"/> <!-- ! Match the prefix in my_arm_macro.urdf.xacro -->
+    <xacro:property name="arm_B_ur_prefix" value="${arm_B_tf_prefix}ur_"/> <!-- ! Match the prefix in my_arm_macro.urdf.xacro -->
+    <xacro:property name="arm_A_realsense_prefix" value="${arm_A_tf_prefix}realsense"/> <!-- ! Match the prefix in my_arm_macro.urdf.xacro -->
+    <xacro:property name="arm_B_realsense_prefix" value="${arm_B_tf_prefix}realsense"/> <!-- ! Match the prefix in my_arm_macro.urdf.xacro -->
+    <xacro:property name="arm_A_g2f85_prefix" value="${arm_A_tf_prefix}"/> <!-- ! Match the prefix in my_arm_macro.urdf.xacro -->
+    <xacro:property name="arm_B_g2f85_prefix" value="${arm_B_tf_prefix}"/> <!-- ! Match the prefix in my_arm_macro.urdf.xacro -->
+    <ros2_control name="my_env_ros2_mujoco" type="system">
+      <hardware>
+        <plugin>mujoco_ros2_simulation/MujocoSystemInterface</plugin>
+        <param name="mujoco_model">${mjcf_file_path}</param>
+        <!-- Override the slowdown settings in the Simulate App and run at 3x speed -->
+        <param name="sim_speed_factor">1.0</param>
+        <!-- If set to true, will not launch the Simulate App window -->
+        <param name="headless">false</param>
+        <!-- Publish camera images -->
+        <param name="camera_publish_rate">30.0</param>
+        <!-- Publish lidar scans at 10 hz -->
+        <param name="lidar_publish_rate">10.0</param>
+      </hardware>
+      <!-- 把两套机械臂的 joint/sensor 接口“塞进同一个 system”里 -->
+      <xacro:my_arm_mujoco_control
+          ur_tf_prefix="${arm_A_ur_prefix}"
+          realsense_tf_prefix="${arm_A_realsense_prefix}"
+          g2f85_tf_prefix="${arm_A_g2f85_prefix}"/>
+      <xacro:my_arm_mujoco_control
+          ur_tf_prefix="${arm_B_ur_prefix}"
+          realsense_tf_prefix="${arm_B_realsense_prefix}"
+          g2f85_tf_prefix="${arm_B_g2f85_prefix}"/>
+    </ros2_control>
+  </xacro:if>
   </xacro:macro>
 </robot>
