Commit message: 修改 xacro 文件为description和ros2 control分离的形式（Jazzy升级）

File: src/my_env/my_env_control/urdf/my_env_control.urdf.xacro (robot description, xacro)
@@ -3,4 +3,7 @@
   <!-- 首先包含自定义描述宏 -->
   <xacro:include filename="$(find my_env_description)/urdf/my_env_macro.urdf.xacro"/>
+  <!-- Jazzy: ros2_control 宏分别来自 ur_robot_driver 和 robotiq_description -->
+  <xacro:include filename="$(find ur_robot_driver)/urdf/ur.ros2_control.xacro" />
+  <xacro:include filename="$(find robotiq_description)/urdf/2f_85.ros2_control.xacro" />
   <!-- 我们需要指定用于参数化描述的参数 -->
   <!-- 为所需的ur_type创建一个文件夹，并从ur_description包中复制文件到那里 -->
@@ -10,7 +13,4 @@
   <xacro:arg name="use_fake_hardware" default="true" />
   <xacro:arg name="use_fake_sensor_commands" default="true" />
-  <xacro:arg name="use_sim_gazebo" default="false" />
-  <xacro:arg name="use_sim_mujoco" default="false" />
-  <xacro:arg name="generate_ros2_control" default="true" />
   <!-- UR 机器人其他参数 -->
   <xacro:arg name="ur_reverse_ip" default="0.0.0.0"/>
@@ -23,4 +23,5 @@
   <xacro:arg name="ur_A_script_command_port" default="50003"/>
   <xacro:arg name="ur_A_trajectory_port" default="50004"/>
+  <xacro:arg name="ur_A_rw_rate" default="0"/>
   <!-- UR_B 机器人参数 -->
   <xacro:arg name="ur_B_ur_type" default="ur5e"/>
@@ -30,34 +31,160 @@
   <xacro:arg name="ur_B_script_command_port" default="50013"/>
   <xacro:arg name="ur_B_trajectory_port" default="50014"/>
+  <xacro:arg name="ur_B_rw_rate" default="0"/>
   <!-- 夹爪和相机参数 -->
-  <xacro:arg name="gripper_com_port_A" default="/dev/ttyUSB0"/>
-  <xacro:arg name="gripper_com_port_B" default="/dev/ttyUSB1"/>
+  <xacro:arg name="g2f85_A_com_port" default="/dev/ttyUSB0"/>
+  <xacro:arg name="g2f85_B_com_port" default="/dev/ttyUSB1"/>
   <xacro:arg name="camera_use_nominal_extrinsics" default="true"/>
-  <!-- 创建包含机器人的场景描述 - 传递my_env宏需要的所有参数 -->
+  <!-- UR 安全限位和路径参数（几何用） -->
+  <xacro:arg name="safety_limits" default="false"/>
+  <xacro:arg name="safety_pos_margin" default="0.15"/>
+  <xacro:arg name="safety_k_position" default="20"/>
+  <xacro:arg name="force_abs_paths" default="false"/>
+  <!-- UR ros2_control recipe 文件 -->
+  <xacro:arg name="script_filename" default="$(find ur_client_library)/resources/external_control.urscript"/>
+  <xacro:arg name="output_recipe_filename" default="$(find ur_robot_driver)/resources/rtde_output_recipe.txt"/>
+  <xacro:arg name="input_recipe_filename" default="$(find ur_robot_driver)/resources/rtde_input_recipe.txt"/>
+  <!-- 初始位置文件 -->
+  <xacro:arg name="initial_positions_file" default="$(find ur_description)/config/initial_positions.yaml"/>
+  <!-- ============================================ -->
+  <!-- UR ros2_control 可选参数（两臂共享）           -->
+  <!-- ============================================ -->
+  <xacro:arg name="ur_transmission_hw_interface" default="hardware_interface/PositionJointInterface"/>
+  <xacro:arg name="ur_use_tool_communication" default="false"/>
+  <xacro:arg name="ur_tool_voltage" default="0"/>
+  <xacro:arg name="ur_tool_parity" default="0"/>
+  <xacro:arg name="ur_tool_baud_rate" default="115200"/>
+  <xacro:arg name="ur_tool_stop_bits" default="1"/>
+  <xacro:arg name="ur_tool_rx_idle_chars" default="1.5"/>
+  <xacro:arg name="ur_tool_tx_idle_chars" default="3.5"/>
+  <xacro:arg name="ur_tool_device_name" default="/tmp/ttyUR"/>
+  <xacro:arg name="ur_tool_tcp_port" default="54321"/>
+  <xacro:arg name="ur_non_blocking_read" default="true"/>
+  <xacro:arg name="ur_robot_receive_timeout" default="0.04"/>
+  <!-- ============================================ -->
+  <!-- Robotiq 夹爪 ros2_control 可选参数（两臂共享） -->
+  <!-- ============================================ -->
+  <xacro:arg name="g2f85_gripper_speed_multiplier" default="1.0"/>
+  <xacro:arg name="g2f85_gripper_force_multiplier" default="0.5"/>
+  <xacro:arg name="g2f85_gripper_max_speed" default="0.150"/>
+  <xacro:arg name="g2f85_gripper_max_force" default="235.0"/>
+  <xacro:arg name="g2f85_gripper_closed_position" default="0.7929"/>
+  <!-- 转换为 property 以便在调用中使用 substitution -->
+  <xacro:property name="initial_positions_file" default="$(arg initial_positions_file)"/>
+  <!-- Jazzy: 纯几何描述（仅传几何参数给 my_env） -->
   <xacro:my_env
     arm_A_tf_prefix="$(arg arm_A_tf_prefix)"
     arm_B_tf_prefix="$(arg arm_B_tf_prefix)"
-    use_fake_hardware="$(arg use_fake_hardware)"
-    use_fake_sensor_commands="$(arg use_fake_sensor_commands)"
-    use_sim_gazebo="$(arg use_sim_gazebo)"
-    use_sim_mujoco="$(arg use_sim_mujoco)"
-    generate_ros2_control="$(arg generate_ros2_control)"
-    ur_reverse_ip="$(arg ur_reverse_ip)"
-    ur_headless_mode="$(arg ur_headless_mode)"
     ur_A_ur_type="$(arg ur_A_ur_type)"
     ur_B_ur_type="$(arg ur_B_ur_type)"
-    ur_A_robot_ip="$(arg ur_A_robot_ip)"
-    ur_B_robot_ip="$(arg ur_B_robot_ip)"
-    ur_A_reverse_port="$(arg ur_A_reverse_port)"
-    ur_A_script_sender_port="$(arg ur_A_script_sender_port)"
-    ur_A_script_command_port="$(arg ur_A_script_command_port)"
-    ur_A_trajectory_port="$(arg ur_A_trajectory_port)"
-    ur_B_reverse_port="$(arg ur_B_reverse_port)"
-    ur_B_script_sender_port="$(arg ur_B_script_sender_port)"
-    ur_B_script_command_port="$(arg ur_B_script_command_port)"
-    ur_B_trajectory_port="$(arg ur_B_trajectory_port)"
     camera_use_nominal_extrinsics="$(arg camera_use_nominal_extrinsics)"
-    gripper_com_port_A="$(arg gripper_com_port_A)"
-    gripper_com_port_B="$(arg gripper_com_port_B)"
+    safety_limits="$(arg safety_limits)"
+    safety_pos_margin="$(arg safety_pos_margin)"
+    safety_k_position="$(arg safety_k_position)"
+    force_abs_paths="$(arg force_abs_paths)"
+  />
+  <!-- ============================================ -->
+  <!-- Jazzy: UR ros2_control (独立于几何描述)       -->
+  <!-- ============================================ -->
+  <!-- arm_A UR ros2_control -->
+  <xacro:ur_ros2_control
+    name="ur_A"
+    tf_prefix="$(arg arm_A_tf_prefix)ur_"
+    kinematics_parameters_file="$(find ur_description)/config/$(arg ur_A_ur_type)/default_kinematics.yaml"
+    robot_ip="$(arg ur_A_robot_ip)"
+    script_filename="$(arg script_filename)"
+    output_recipe_filename="$(arg output_recipe_filename)"
+    input_recipe_filename="$(arg input_recipe_filename)"
+    reverse_ip="$(arg ur_reverse_ip)"
+    reverse_port="$(arg ur_A_reverse_port)"
+    script_sender_port="$(arg ur_A_script_sender_port)"
+    script_command_port="$(arg ur_A_script_command_port)"
+    trajectory_port="$(arg ur_A_trajectory_port)"
+    use_mock_hardware="$(arg use_fake_hardware)"
+    mock_sensor_commands="$(arg use_fake_sensor_commands)"
+    headless_mode="$(arg ur_headless_mode)"
+    initial_positions="${xacro.load_yaml(initial_positions_file)}"
+    transmission_hw_interface="$(arg ur_transmission_hw_interface)"
+    use_tool_communication="$(arg ur_use_tool_communication)"
+    tool_voltage="$(arg ur_tool_voltage)"
+    tool_parity="$(arg ur_tool_parity)"
+    tool_baud_rate="$(arg ur_tool_baud_rate)"
+    tool_stop_bits="$(arg ur_tool_stop_bits)"
+    tool_rx_idle_chars="$(arg ur_tool_rx_idle_chars)"
+    tool_tx_idle_chars="$(arg ur_tool_tx_idle_chars)"
+    tool_device_name="$(arg ur_tool_device_name)"
+    tool_tcp_port="$(arg ur_tool_tcp_port)"
+    non_blocking_read="$(arg ur_non_blocking_read)"
+    robot_receive_timeout="$(arg ur_robot_receive_timeout)"
+    rw_rate="$(arg ur_A_rw_rate)"
+  />
+  <!-- arm_B UR ros2_control -->
+  <xacro:ur_ros2_control
+    name="ur_B"
+    tf_prefix="$(arg arm_B_tf_prefix)ur_"
+    kinematics_parameters_file="$(find ur_description)/config/$(arg ur_B_ur_type)/default_kinematics.yaml"
+    robot_ip="$(arg ur_B_robot_ip)"
+    script_filename="$(arg script_filename)"
+    output_recipe_filename="$(arg output_recipe_filename)"
+    input_recipe_filename="$(arg input_recipe_filename)"
+    reverse_ip="$(arg ur_reverse_ip)"
+    reverse_port="$(arg ur_B_reverse_port)"
+    script_sender_port="$(arg ur_B_script_sender_port)"
+    script_command_port="$(arg ur_B_script_command_port)"
+    trajectory_port="$(arg ur_B_trajectory_port)"
+    use_mock_hardware="$(arg use_fake_hardware)"
+    mock_sensor_commands="$(arg use_fake_sensor_commands)"
+    headless_mode="$(arg ur_headless_mode)"
+    initial_positions="${xacro.load_yaml(initial_positions_file)}"
+    transmission_hw_interface="$(arg ur_transmission_hw_interface)"
+    use_tool_communication="$(arg ur_use_tool_communication)"
+    tool_voltage="$(arg ur_tool_voltage)"
+    tool_parity="$(arg ur_tool_parity)"
+    tool_baud_rate="$(arg ur_tool_baud_rate)"
+    tool_stop_bits="$(arg ur_tool_stop_bits)"
+    tool_rx_idle_chars="$(arg ur_tool_rx_idle_chars)"
+    tool_tx_idle_chars="$(arg ur_tool_tx_idle_chars)"
+    tool_device_name="$(arg ur_tool_device_name)"
+    tool_tcp_port="$(arg ur_tool_tcp_port)"
+    non_blocking_read="$(arg ur_non_blocking_read)"
+    robot_receive_timeout="$(arg ur_robot_receive_timeout)"
+    rw_rate="$(arg ur_B_rw_rate)"
+  />
+  <!-- ============================================ -->
+  <!-- Jazzy: Robotiq 夹爪 ros2_control             -->
+  <!-- ============================================ -->
+  <!-- arm_A 夹爪 ros2_control -->
+  <xacro:robotiq_gripper_ros2_control
+    name="arm_A_g2f85"
+    prefix="$(arg arm_A_tf_prefix)"
+    use_fake_hardware="$(arg use_fake_hardware)"
+    mock_sensor_commands="$(arg use_fake_sensor_commands)"
+    com_port="$(arg g2f85_A_com_port)"
+    sim_gazebo="False"
+    sim_isaac="False"
+    isaac_joint_commands="/isaac_joint_commands"
+    isaac_joint_states="/isaac_joint_states"
+    gripper_speed_multiplier="$(arg g2f85_gripper_speed_multiplier)"
+    gripper_force_multiplier="$(arg g2f85_gripper_force_multiplier)"
+    gripper_max_speed="$(arg g2f85_gripper_max_speed)"
+    gripper_max_force="$(arg g2f85_gripper_max_force)"
+    gripper_closed_position="$(arg g2f85_gripper_closed_position)"
+  />
+  <!-- arm_B 夹爪 ros2_control -->
+  <xacro:robotiq_gripper_ros2_control
+    name="arm_B_g2f85"
+    prefix="$(arg arm_B_tf_prefix)"
+    use_fake_hardware="$(arg use_fake_hardware)"
+    mock_sensor_commands="$(arg use_fake_sensor_commands)"
+    com_port="$(arg g2f85_B_com_port)"
+    sim_gazebo="False"
+    sim_isaac="False"
+    isaac_joint_commands="/isaac_joint_commands"
+    isaac_joint_states="/isaac_joint_states"
+    gripper_speed_multiplier="$(arg g2f85_gripper_speed_multiplier)"
+    gripper_force_multiplier="$(arg g2f85_gripper_force_multiplier)"
+    gripper_max_speed="$(arg g2f85_gripper_max_speed)"
+    gripper_max_force="$(arg g2f85_gripper_max_force)"
+    gripper_closed_position="$(arg g2f85_gripper_closed_position)"
   />
 </robot>

File: src/my_env/my_env_description/urdf/my_arm_macro.urdf.xacro (robot description, xacro)
@@ -6,25 +6,18 @@
   <xacro:include filename="$(find realsense2_description)/urdf/_d435.urdf.xacro" />
   <!-- 宏定义自己的机械臂结构 UR+Robotiq+RealSense -->
+  <!-- Jazzy: 仅纯几何描述，不包含任何 ros2_control -->
   <xacro:macro name="my_arm" params="
     name:=my_arm
     tf_prefix:=my_arm
     parent:=world
-    use_fake_hardware:=false
-    use_fake_sensor_commands:=false
-    use_sim_gazebo:=false
-    generate_ros2_control:=false
     ur_type:=ur5e
-    ur_reverse_ip:=0.0.0.0
-    ur_reverse_port:=50001
-    ur_robot_ip
-    ur_script_sender_port:=50002
-    ur_script_command_port:=50003
-    ur_trajectory_port:=50004
-    ur_headless_mode:=false
-    g2f85_com_port:=/dev/ttyUSB0
     realsense_use_nominal_extrinsics:=false
+    safety_limits:=false
+    safety_pos_margin:=0.15
+    safety_k_position:=20
+    force_abs_paths:=false
     *origin
     ">
-    <!-- UR parameters -->
+    <!-- UR parameters (Jazzy: 仅 yaml 配置文件路径) -->
     <xacro:property name="_ur_name" value="${name}_ur"/>
     <xacro:property name="_ur_tf_prefix" value="${tf_prefix}ur_"/> <!-- ! Match the prefix in my_env_macro.urdf.xacro -->
@@ -34,33 +27,4 @@
     <xacro:property name="_ur_physical_parameters_file" value="$(find ur_description)/config/${ur_type}/physical_parameters.yaml"/>
     <xacro:property name="_ur_visual_parameters_file" value="$(find ur_description)/config/${ur_type}/visual_parameters.yaml"/>
-    <!-- UR Simulation parameters -->
-    <xacro:property name="_ur_use_fake_hardware" value="${use_fake_hardware}" />
-    <xacro:property name="_ur_fake_sensor_commands" value="${use_fake_sensor_commands}" />
-    <xacro:property name="_ur_sim_gazebo" value="${use_sim_gazebo}" />
-    <xacro:property name="_ur_sim_ignition" value="false" />
-    <!-- UR tool communication related parameters-->
-    <xacro:property name="_ur_use_tool_communication" value="false" />
-    <xacro:property name="_ur_tool_voltage" value="0" />
-    <xacro:property name="_ur_tool_parity" value="0" />
-    <xacro:property name="_ur_tool_baud_rate" value="115200" />
-    <xacro:property name="_ur_tool_stop_bits" value="1" />
-    <xacro:property name="_ur_tool_rx_idle_chars" value="1.5" />
-    <xacro:property name="_ur_tool_tx_idle_chars" value="3.5" />
-    <xacro:property name="_ur_tool_device_name" value="/tmp/ttyUR" />
-    <xacro:property name="_ur_tool_tcp_port" value="54321" />
-    <!-- UR ros2_control related parameters -->
-    <xacro:property name="_ur_generate_ros2_control" value="${generate_ros2_control}" />
-    <xacro:property name="_ur_initial_positions_file" value="$(find ur_description)/config/initial_positions.yaml" />
-    <xacro:property name="_ur_initial_positions" value="${xacro.load_yaml(_ur_initial_positions_file)}" />
-    <xacro:property name="_ur_headless_mode" value="${ur_headless_mode}" />
-    <xacro:property name="_ur_script_filename" value="$(find ur_client_library)/resources/external_control.urscript" />
-    <xacro:property name="_ur_output_recipe_filename" value="$(find ur_robot_driver)/resources/rtde_output_recipe.txt" />
-    <xacro:property name="_ur_input_recipe_filename" value="$(find ur_robot_driver)/resources/rtde_input_recipe.txt" />
-    <xacro:property name="_ur_reverse_ip" value="${ur_reverse_ip}" />
-    <xacro:property name="_ur_reverse_port" value="${ur_reverse_port}" />
-    <xacro:property name="_ur_robot_ip" value="${ur_robot_ip}" />
-    <xacro:property name="_ur_script_sender_port" value="${ur_script_sender_port}" />
-    <xacro:property name="_ur_script_command_port" value="${ur_script_command_port}" />
-    <xacro:property name="_ur_trajectory_port" value="${ur_trajectory_port}" />
     <!-- RealSense parameters -->
     <xacro:property name="_realsense_name" value="${tf_prefix}realsense" />
@@ -69,19 +33,8 @@
     <xacro:property name="_realsense_add_plug" value="false" />
     <xacro:property name="_realsense_use_mesh" value="true" />
-    <!-- Robotiq 2f85 gripper parameters -->
+    <!-- Robotiq 2f85 gripper parameters (Jazzy: 纯几何，不含 ros2_control) -->
     <xacro:property name="_g2f85_name" value="${name}_g2f85" />
     <xacro:property name="_g2f85_prefix" value="${tf_prefix}" /> <!-- ! Match the prefix in my_env_macro.urdf.xacro -->
-    <xacro:property name="_g2f85_sim_gazebo" value="${use_sim_gazebo}" />
-    <xacro:property name="_g2f85_sim_isaac" value="false" />
-    <xacro:property name="_g2f85_use_fake_hardware" value="${use_fake_hardware}" />
-    <xacro:property name="_g2f85_mock_sensor_commands" value="${use_fake_sensor_commands}" />
-    <xacro:property name="_g2f85_include_ros2_control" value="${generate_ros2_control}" />
-    <xacro:property name="_g2f85_com_port" value="${g2f85_com_port}" />
-    <xacro:property name="_g2f85_gripper_speed_multiplier" value="1.0" />
-    <xacro:property name="_g2f85_gripper_force_multiplier" value="0.5" />
-    <xacro:property name="_g2f85_gripper_max_speed" value="0.150" />
-    <xacro:property name="_g2f85_gripper_max_force" value="235.0" />
-    <xacro:property name="_g2f85_gripper_closed_position" value="0.7929" />
-    <!-- 创建 UR 机器人 使用宏定义 -->
+    <!-- 创建 UR 机器人 使用宏定义 (Jazzy: 纯描述，无 ros2_control 参数) -->
     <xacro:ur_robot
       name="${_ur_name}"
@@ -92,29 +45,8 @@
       physical_parameters_file="${_ur_physical_parameters_file}"
       visual_parameters_file="${_ur_visual_parameters_file}"
-      generate_ros2_control_tag="${_ur_generate_ros2_control}"
-      use_fake_hardware="${_ur_use_fake_hardware}"
-      fake_sensor_commands="${_ur_fake_sensor_commands}"
-      sim_gazebo="${_ur_sim_gazebo}"
-      sim_ignition="${_ur_sim_ignition}"
-      headless_mode="${_ur_headless_mode}"
-      initial_positions="${_ur_initial_positions}"
-      use_tool_communication="${_ur_use_tool_communication}"
-      tool_voltage="${_ur_tool_voltage}"
-      tool_parity="${_ur_tool_parity}"
-      tool_baud_rate="${_ur_tool_baud_rate}"
-      tool_stop_bits="${_ur_tool_stop_bits}"
-      tool_rx_idle_chars="${_ur_tool_rx_idle_chars}"
-      tool_tx_idle_chars="${_ur_tool_tx_idle_chars}"
-      tool_device_name="${_ur_tool_device_name}"
-      tool_tcp_port="${_ur_tool_tcp_port}"
-      robot_ip="${_ur_robot_ip}"
-      script_filename="${_ur_script_filename}"
-      output_recipe_filename="${_ur_output_recipe_filename}"
-      input_recipe_filename="${_ur_input_recipe_filename}"
-      reverse_ip="${_ur_reverse_ip}"
-      reverse_port="${_ur_reverse_port}"
-      script_sender_port="${_ur_script_sender_port}"
-      script_command_port="${_ur_script_command_port}"
-      trajectory_port="${_ur_trajectory_port}"
+      safety_limits="${safety_limits}"
+      safety_pos_margin="${safety_pos_margin}"
+      safety_k_position="${safety_k_position}"
+      force_abs_paths="${force_abs_paths}"
     >
       <xacro:insert_block name="origin" />
@@ -174,20 +106,10 @@
     >
     </xacro:ur_to_robotiq>
-    <!-- 创建 robotiq 夹爪 使用宏定义 -->
+    <!-- 创建 robotiq 夹爪 使用宏定义 (Jazzy: 纯几何，禁用 ros2_control) -->
     <xacro:robotiq_gripper
       name="${_g2f85_name}"
       prefix="${_g2f85_prefix}"
       parent="${_g2f85_prefix}robotiq_ur_to_g2f85_child_side"
-      sim_gazebo="${_g2f85_sim_gazebo}"
-      sim_isaac="${_g2f85_sim_isaac}"
-      use_fake_hardware="${_g2f85_use_fake_hardware}"
-      mock_sensor_commands="${_g2f85_mock_sensor_commands}"
-      include_ros2_control="${_g2f85_include_ros2_control}"
-      com_port="${_g2f85_com_port}"
-      gripper_speed_multiplier="${_g2f85_gripper_speed_multiplier}"
-      gripper_force_multiplier="${_g2f85_gripper_force_multiplier}"
-      gripper_max_speed="${_g2f85_gripper_max_speed}"
-      gripper_max_force="${_g2f85_gripper_max_force}"
-      gripper_closed_position="${_g2f85_gripper_closed_position}"
+      include_ros2_control="false"
     >
       <origin xyz="0 0 0" rpy="0 0 0" />

File: src/my_env/my_env_description/urdf/my_env.urdf.xacro (robot description, xacro)
@@ -11,22 +11,22 @@
   <xacro:arg name="arm_B_tf_prefix" default="arm_B_"/>
   <xacro:arg name="ur_B_ur_type" default="ur5e"/>
-  <!-- 控制参数 -->
-  <xacro:arg name="use_fake_hardware" default="true" />
-  <xacro:arg name="fake_sensor_commands" default="true" />
-  <xacro:arg name="use_sim_gazebo" default="false" />
-  <xacro:arg name="generate_ros2_control" default="false" />
   <!-- 夹爪和相机参数 -->
   <xacro:arg name="camera_use_nominal_extrinsics" default="true"/>
-  <!-- 创建包含机器人的场景描述 - 传递my_env宏需要的所有参数 -->
+  <!-- UR 安全限位和路径参数 -->
+  <xacro:arg name="safety_limits" default="false"/>
+  <xacro:arg name="safety_pos_margin" default="0.15"/>
+  <xacro:arg name="safety_k_position" default="20"/>
+  <xacro:arg name="force_abs_paths" default="false"/>
+  <!-- Jazzy: 纯描述入口，用于 RViz/MoveIt，不包含 ros2_control -->
   <xacro:my_env
     arm_A_tf_prefix="$(arg arm_A_tf_prefix)"
     arm_B_tf_prefix="$(arg arm_B_tf_prefix)"
-    use_fake_hardware="$(arg use_fake_hardware)"
-    use_fake_sensor_commands="$(arg fake_sensor_commands)"
-    generate_ros2_control="$(arg generate_ros2_control)"
-    mjcf_file_path=""
     ur_A_ur_type="$(arg ur_A_ur_type)"
     ur_B_ur_type="$(arg ur_B_ur_type)"
     camera_use_nominal_extrinsics="$(arg camera_use_nominal_extrinsics)"
+    safety_limits="$(arg safety_limits)"
+    safety_pos_margin="$(arg safety_pos_margin)"
+    safety_k_position="$(arg safety_k_position)"
+    force_abs_paths="$(arg force_abs_paths)"
   />
 </robot>
