Commit message: everything working

File: src/my_env/my_env_control/urdf/my_env_control.urdf.xacro (robot description, xacro)
@@ -3,9 +3,10 @@
   <!-- 首先包含自定义描述宏 -->
   <xacro:include filename="$(find my_env_description)/urdf/my_env_macro.urdf.xacro"/>
-  <!-- Jazzy: ros2_control 宏分别来自 ur_robot_driver 和 robotiq_description -->
+  <!-- Jazzy: ros2_control 宏分别来自 ur_robot_driver、robotiq_description 和 dh_ag95_description -->
   <xacro:include filename="$(find ur_robot_driver)/urdf/ur.ros2_control.xacro" />
   <xacro:include filename="$(find robotiq_description)/urdf/2f_85.ros2_control.xacro" />
+  <xacro:include filename="$(find dh_ag95_description)/urdf/dh_ag95.ros2_control.xacro" />
   <!-- 我们需要指定用于参数化描述的参数 -->
-  <!-- 为所需的ur_type创建一个文件夹，并从ur_description包中复制文件到那里 -->
+  <!-- 双臂前缀/型号等属性现在统一由 dual_arm_config.xacro 提供（通过 my_env_macro.urdf.xacro 间接 include） -->
   <!-- 总体参数 -->
   <xacro:arg name="use_fake_hardware" default="true" />
@@ -43,4 +44,24 @@
   <xacro:arg name="output_recipe_filename" default="$(find ur_robot_driver)/resources/rtde_output_recipe.txt"/>
   <xacro:arg name="input_recipe_filename" default="$(find ur_robot_driver)/resources/rtde_input_recipe.txt"/>
+  <!-- DH-Robotics AG-95 夹爪 共享参数（前缀 ag95_gripper_）-->
+  <xacro:arg name="ag95_gripper_transport_type" default="official_serial"/>
+  <xacro:arg name="ag95_gripper_serial_baudrate" default="115200"/>
+  <xacro:arg name="ag95_gripper_can_bitrate" default="500000"/>
+  <xacro:arg name="ag95_gripper_pcan_bitrate" default="500000"/>
+  <xacro:arg name="ag95_gripper_gripper_model" default="ag-160-95"/>
+  <xacro:arg name="ag95_gripper_default_force_percent" default="30"/>
+  <xacro:arg name="ag95_gripper_auto_initialize" default="true"/>
+  <xacro:arg name="ag95_gripper_rw_rate" default="25"/>
+  <xacro:arg name="ag95_gripper_command_interval_ms" default="10"/>
+  <!-- DH-Robotics AG-95 臂A 独立参数（前缀 ag95_A_）-->
+  <xacro:arg name="ag95_A_serial_port" default="/dev/ttyAG95_A"/>
+  <xacro:arg name="ag95_A_can_interface" default="can0"/>
+  <xacro:arg name="ag95_A_pcan_channel" default="PCAN_USBBUS1"/>
+  <xacro:arg name="ag95_A_gripper_id" default="1"/>
+  <!-- DH-Robotics AG-95 臂B 独立参数（前缀 ag95_B_）-->
+  <xacro:arg name="ag95_B_serial_port" default="/dev/ttyAG95_B"/>
+  <xacro:arg name="ag95_B_can_interface" default="can0"/>
+  <xacro:arg name="ag95_B_pcan_channel" default="PCAN_USBBUS1"/>
+  <xacro:arg name="ag95_B_gripper_id" default="2"/>
   <!-- 初始位置文件 -->
   <xacro:arg name="initial_positions_file" default="$(find ur_description)/config/initial_positions.yaml"/>
@@ -148,9 +169,10 @@
   <!-- Jazzy: Robotiq 夹爪 ros2_control             -->
   <!-- ============================================ -->
+  <xacro:if value="${gripper_type == 'robotiq_2f85'}">
   <!-- arm_A 夹爪 ros2_control -->
   <xacro:robotiq_gripper_ros2_control
     name="arm_A_g2f85"
     prefix="${arm_A_tf_prefix}"
-    use_fake_hardware="True"
+    use_fake_hardware="$(arg use_fake_hardware)"
     mock_sensor_commands="$(arg use_fake_sensor_commands)"
     com_port="$(arg g2f85_A_com_port)"
@@ -169,5 +191,5 @@
     name="arm_B_g2f85"
     prefix="${arm_B_tf_prefix}"
-    use_fake_hardware="True"
+    use_fake_hardware="$(arg use_fake_hardware)"
     mock_sensor_commands="$(arg use_fake_sensor_commands)"
     com_port="$(arg g2f85_B_com_port)"
@@ -182,3 +204,47 @@
     gripper_closed_position="$(arg g2f85_gripper_closed_position)"
   />
+  </xacro:if>
+  <!-- ============================================ -->
+  <!-- Jazzy: DH-Robotics AG-95 夹爪 ros2_control   -->
+  <!-- ============================================ -->
+  <xacro:if value="${gripper_type == 'dh_ag95'}">
+  <!-- arm_A AG-95 夹爪 ros2_control -->
+  <xacro:dh_ag95_ros2_control
+    prefix="${arm_A_tf_prefix}"
+    name="arm_A_ag95_hardware"
+    use_fake_hardware="$(arg use_fake_hardware)"
+    transport_type="$(arg ag95_gripper_transport_type)"
+    serial_port="$(arg ag95_A_serial_port)"
+    serial_baudrate="$(arg ag95_gripper_serial_baudrate)"
+    can_interface="$(arg ag95_A_can_interface)"
+    can_bitrate="$(arg ag95_gripper_can_bitrate)"
+    pcan_channel="$(arg ag95_A_pcan_channel)"
+    pcan_bitrate="$(arg ag95_gripper_pcan_bitrate)"
+    gripper_id="$(arg ag95_A_gripper_id)"
+    gripper_model="$(arg ag95_gripper_gripper_model)"
+    default_force_percent="$(arg ag95_gripper_default_force_percent)"
+    auto_initialize="$(arg ag95_gripper_auto_initialize)"
+    rw_rate="$(arg ag95_gripper_rw_rate)"
+    command_interval_ms="$(arg ag95_gripper_command_interval_ms)"
+  />
+  <!-- arm_B AG-95 夹爪 ros2_control -->
+  <xacro:dh_ag95_ros2_control
+    prefix="${arm_B_tf_prefix}"
+    name="arm_B_ag95_hardware"
+    use_fake_hardware="$(arg use_fake_hardware)"
+    transport_type="$(arg ag95_gripper_transport_type)"
+    serial_port="$(arg ag95_B_serial_port)"
+    serial_baudrate="$(arg ag95_gripper_serial_baudrate)"
+    can_interface="$(arg ag95_B_can_interface)"
+    can_bitrate="$(arg ag95_gripper_can_bitrate)"
+    pcan_channel="$(arg ag95_B_pcan_channel)"
+    pcan_bitrate="$(arg ag95_gripper_pcan_bitrate)"
+    gripper_id="$(arg ag95_B_gripper_id)"
+    gripper_model="$(arg ag95_gripper_gripper_model)"
+    default_force_percent="$(arg ag95_gripper_default_force_percent)"
+    auto_initialize="$(arg ag95_gripper_auto_initialize)"
+    rw_rate="$(arg ag95_gripper_rw_rate)"
+    command_interval_ms="$(arg ag95_gripper_command_interval_ms)"
+  />
+  </xacro:if>
 </robot>

File: src/my_env/my_env_description/urdf/my_arm_macro.urdf.xacro (robot description, xacro)
@@ -1,9 +1,20 @@
 <?xml version="1.0"?>
 <robot xmlns:xacro="http://ros.org/wiki/xacro">
+  <!-- ============================================ -->
+  <!-- 通用依赖（所有夹爪类型都需要）               -->
+  <!-- ============================================ -->
   <xacro:include filename="$(find ur_description)/urdf/ur_macro.xacro"/>
-  <xacro:include filename="$(find robotiq_description)/urdf/robotiq_2f_85_macro.urdf.xacro" />
-  <xacro:include filename="$(find robotiq_description)/urdf/ur_to_robotiq_adapter.urdf.xacro" />
   <xacro:include filename="$(find realsense2_description)/urdf/_d435.urdf.xacro" />
-  <!-- 宏定义自己的机械臂结构 UR+Robotiq+RealSense -->
+  <!-- ============================================ -->
+  <!-- 夹爪类型条件依赖                             -->
+  <!-- ============================================ -->
+  <xacro:if value="${gripper_type == 'robotiq_2f85'}">
+    <xacro:include filename="$(find robotiq_description)/urdf/robotiq_2f_85_macro.urdf.xacro" />
+    <xacro:include filename="$(find robotiq_description)/urdf/ur_to_robotiq_adapter.urdf.xacro" />
+  </xacro:if>
+  <xacro:if value="${gripper_type == 'dh_ag95'}">
+    <xacro:include filename="$(find dh_ag95_description)/urdf/dh_ag95_macro.urdf.xacro" />
+  </xacro:if>
+  <!-- 宏定义自己的机械臂结构 UR+Gripper+RealSense -->
   <!-- Jazzy: 仅纯几何描述，不包含任何 ros2_control -->
   <xacro:macro name="my_arm" params="
@@ -12,4 +23,5 @@
     parent:=world
     ur_type:=ur5e
+    gripper_type:=dh_ag95
     realsense_use_nominal_extrinsics:=false
     safety_limits:=false
@@ -33,7 +45,15 @@
     <xacro:property name="_realsense_add_plug" value="false" />
     <xacro:property name="_realsense_use_mesh" value="true" />
-    <!-- Robotiq 2f85 gripper parameters (Jazzy: 纯几何，不含 ros2_control) -->
-    <xacro:property name="_g2f85_name" value="${name}_g2f85" />
-    <xacro:property name="_g2f85_prefix" value="${tf_prefix}" /> <!-- ! Match the prefix in my_env_macro.urdf.xacro -->
+    <!-- 夹爪参数 —— 根据 gripper_type 分别设置 -->
+    <xacro:if value="${gripper_type == 'robotiq_2f85'}">
+      <!-- Robotiq 2f85 gripper parameters (Jazzy: 纯几何，不含 ros2_control) -->
+      <xacro:property name="_g2f85_name" value="${name}_g2f85" />
+      <xacro:property name="_g2f85_prefix" value="${tf_prefix}" /> <!-- ! Match the prefix in my_env_macro.urdf.xacro -->
+    </xacro:if>
+    <xacro:if value="${gripper_type == 'dh_ag95'}">
+      <!-- DH-Robotics AG-95 gripper parameters -->
+      <xacro:property name="_ag95_prefix" value="${tf_prefix}" />
+      <xacro:property name="_ag95_gripper_base_link" value="${_ag95_prefix}gripper_base_link" />
+    </xacro:if>
     <!-- 创建 UR 机器人 使用宏定义 (Jazzy: 纯描述，无 ros2_control 参数) -->
     <xacro:ur_robot
@@ -99,27 +119,59 @@
       <origin xyz="0 0.0875 0.013" rpy="0 ${-pi/2} ${-pi/2}"/>
     </xacro:sensor_d435>
-    <!-- 创建 robotiq 夹爪底座 使用宏定义 -->
-    <xacro:ur_to_robotiq
-      prefix="${_g2f85_prefix}robotiq_"
-      parent="${_realsense_prefix}_shelf_child_side"
-      child="${_g2f85_prefix}robotiq_ur_to_g2f85_child_side"
-    >
-    </xacro:ur_to_robotiq>
-    <!-- 创建 robotiq 夹爪 使用宏定义 (Jazzy: 纯几何，禁用 ros2_control) -->
-    <xacro:robotiq_gripper
-      name="${_g2f85_name}"
-      prefix="${_g2f85_prefix}"
-      parent="${_g2f85_prefix}robotiq_ur_to_g2f85_child_side"
-      include_ros2_control="false"
-    >
-      <origin xyz="0 0 0" rpy="0 0 0" />
-    </xacro:robotiq_gripper>
-    <!-- 创建 tcp  -->
-    <link name="${tf_prefix}_tcp"/>
-    <joint name="${tf_prefix}_tcp_joint" type="fixed">
-        <origin xyz="0 0 0.14" rpy="0 0 0"/>
-        <parent link="${_g2f85_prefix}robotiq_85_base_link"/>
-        <child link="${tf_prefix}_tcp"/>
-    </joint>
+    <!-- ============================================ -->
+    <!-- Robotiq 2F-85 夹爪 几何                      -->
+    <!-- ============================================ -->
+    <xacro:if value="${gripper_type == 'robotiq_2f85'}">
+      <!-- 创建 robotiq 夹爪底座 使用宏定义 -->
+      <xacro:ur_to_robotiq
+        prefix="${_g2f85_prefix}robotiq_"
+        parent="${_realsense_prefix}_shelf_child_side"
+        child="${_g2f85_prefix}robotiq_ur_to_g2f85_child_side"
+      >
+      </xacro:ur_to_robotiq>
+      <!-- 创建 robotiq 夹爪 使用宏定义 (Jazzy: 纯几何，禁用 ros2_control) -->
+      <xacro:robotiq_gripper
+        name="${_g2f85_name}"
+        prefix="${_g2f85_prefix}"
+        parent="${_g2f85_prefix}robotiq_ur_to_g2f85_child_side"
+        include_ros2_control="false"
+      >
+        <origin xyz="0 0 0" rpy="0 0 0" />
+      </xacro:robotiq_gripper>
+      <!-- 创建 TCP (Robotiq 末端) -->
+      <link name="${tf_prefix}_tcp"/>
+      <joint name="${tf_prefix}_tcp_joint" type="fixed">
+          <origin xyz="0 0 0.14" rpy="0 0 0"/>
+          <parent link="${_g2f85_prefix}robotiq_85_base_link"/>
+          <child link="${tf_prefix}_tcp"/>
+      </joint>
+    </xacro:if>
+    <!-- ============================================ -->
+    <!-- DH-Robotics AG-95 夹爪 几何                  -->
+    <!-- ============================================ -->
+    <xacro:if value="${gripper_type == 'dh_ag95'}">
+      <!-- 创建 dh_ag95 夹爪 使用宏定义 (Jazzy: 纯几何) -->
+      <!--
+        use_flange: 是否启用转接法兰。
+        法兰 mesh 文件需手动放入:
+          dh_ag95_description/meshes/visual/flange.STL
+        启用后会在 realsense_shelf_child_side 与 gripper_base_link 之间
+        插入一个 flange_link fixed joint。
+      -->
+      <xacro:dh_ag95_gripper
+        prefix="${_ag95_prefix}"
+        parent="${_realsense_prefix}_shelf_child_side"
+      >
+        <origin xyz="0 0 -0.0035" rpy="0 0 0" />
+      </xacro:dh_ag95_gripper>
+      <!-- 创建 TCP (AG-95 末端) -->
+      <!-- TODO: 请根据实际 AG-95 尺寸调整 origin xyz 偏移 -->
+      <link name="${tf_prefix}_tcp"/>
+      <joint name="${tf_prefix}_tcp_joint" type="fixed">
+          <origin xyz="0 0 0.14" rpy="0 0 0"/>
+          <parent link="${_ag95_gripper_base_link}"/>
+          <child link="${tf_prefix}_tcp"/>
+      </joint>
+    </xacro:if>
   </xacro:macro>
 </robot>

File: src/my_env/my_env_description/urdf/my_env.urdf.xacro (robot description, xacro)
@@ -6,4 +6,7 @@
   <!-- 为所需的ur_type创建一个文件夹，并从ur_description包中复制文件到那里 -->
   <!-- 夹爪和相机参数 -->
+  <!-- gripper_type 默认在 dual_arm_config.xacro 中配置，此处可通过命令行覆盖 -->
+  <xacro:arg name="gripper_type" default="dh_ag95"/>
+  <xacro:property name="gripper_type" value="$(arg gripper_type)"/>
   <xacro:arg name="camera_use_nominal_extrinsics" default="true"/>
   <!-- UR 安全限位和路径参数 -->

File: src/my_env/my_env_description/urdf/my_env_macro.urdf.xacro (robot description, xacro)
@@ -1,4 +1,5 @@
 <?xml version="1.0"?>
 <robot name="my_env" xmlns:xacro="http://ros.org/wiki/xacro">
+  <xacro:include filename="$(find my_env_description)/urdf/dual_arm_config.xacro"/>
   <xacro:include filename="$(find my_env_description)/urdf/my_arm_macro.urdf.xacro"/>
   <!-- Jazzy: 纯几何描述，不包含 ros2_control -->
@@ -10,8 +11,4 @@
   force_abs_paths:=false
   ">
-  <xacro:property name="arm_A_tf_prefix" value="arm_A_"/>
-  <xacro:property name="ur_A_ur_type" value="ur5"/>
-  <xacro:property name="arm_B_tf_prefix" value="arm_B_"/>
-  <xacro:property name="ur_B_ur_type" value="ur5e"/>
   <!-- 定义材料 -->
   <material name="table_material">
@@ -85,4 +82,5 @@
     parent = "ur_mount_A"
     ur_type = "${ur_A_ur_type}"
+    gripper_type = "${gripper_type}"
     realsense_use_nominal_extrinsics = "${camera_use_nominal_extrinsics}"
     safety_limits = "${safety_limits}"
@@ -98,4 +96,5 @@
     parent = "ur_mount_B"
     ur_type = "${ur_B_ur_type}"
+    gripper_type = "${gripper_type}"
     realsense_use_nominal_extrinsics = "${camera_use_nominal_extrinsics}"
     safety_limits = "${safety_limits}"

Commit message: add arm_shelf mesh ; change arm_shelf frame

File: src/my_env/my_env_control/urdf/my_env_control.urdf.xacro (robot description, xacro)
@@ -34,5 +34,5 @@
   <xacro:arg name="g2f85_A_com_port" default="/dev/ttyUSB0"/>
   <xacro:arg name="g2f85_B_com_port" default="/dev/ttyUSB1"/>
-  <xacro:arg name="camera_use_nominal_extrinsics" default="true"/>
+  <xacro:arg name="camera_use_nominal_extrinsics" default="false"/>
   <!-- UR 安全限位和路径参数（几何用） -->
   <xacro:arg name="safety_limits" default="false"/>

File: src/my_env/my_env_description/urdf/my_env.urdf.xacro (robot description, xacro)
@@ -9,5 +9,5 @@
   <xacro:arg name="gripper_type" default="dh_ag95"/>
   <xacro:property name="gripper_type" value="$(arg gripper_type)"/>
-  <xacro:arg name="camera_use_nominal_extrinsics" default="true"/>
+  <xacro:arg name="camera_use_nominal_extrinsics" default="false"/>
   <!-- UR 安全限位和路径参数 -->
   <xacro:arg name="safety_limits" default="false"/>

File: src/my_env/my_env_description/urdf/my_env_macro.urdf.xacro (robot description, xacro)
@@ -5,5 +5,5 @@
   <!-- Jazzy: 纯几何描述，不包含 ros2_control -->
   <xacro:macro name="my_env" params="
-  camera_use_nominal_extrinsics:=true
+  camera_use_nominal_extrinsics:=false
   safety_limits:=false
   safety_pos_margin:=0.15
@@ -23,5 +23,5 @@
     <parent link="world" />
     <child link="table" />
-    <origin xyz="0 ${1.0/2 + 0.05} 0" rpy="0 0 0" />
+    <origin xyz="0 ${0.863 + 0.05} 0" rpy="0 0 0" />
   </joint>
   <!-- world2arm_shelf joint -->
@@ -29,5 +29,5 @@
     <parent link="world" />
     <child link="arm_shelf" />
-    <origin xyz="0 ${-0.728/2} 0" rpy="0 0 0" />
+    <origin xyz="0 0 0.15" rpy="0 0 0" />
   </joint>
   <!-- 桌子 link -->
@@ -51,12 +51,12 @@
     <visual>
       <geometry>
-        <box size="0.615 0.728 1.353"/> # L*W*H=0.615*0.728*1.353m
+        <mesh filename="package://my_env_description/meshes/arm_shelf.STL"/> # L*W*H=0.613*0.726*1.353m
       </geometry>
-      <origin rpy="0 0 0" xyz="0 0 ${1.353/2}" />
+      <origin rpy="0 0 0" xyz="0 0 0" />
       <material name="arm_shelf_material"/>
     </visual>
     <collision>
       <geometry>
-        <box size="0.615 0.728 1.353"/> # L*W*H=0.615*0.728*1.353m
+        <box size="0.726 0.613 1.353"/> # L*W*H=0.726*0.613*1.353m
       </geometry>
       <origin rpy="0 0 0" xyz="0 0 ${1.353/2}" />
@@ -68,5 +68,5 @@
     <parent link="arm_shelf"/>
     <child link="ur_mount_A"/>
-    <origin xyz="${0.615/2 + 0.068} ${0.728/2 - 0.13} ${1.353 - 0.13}" rpy="0 ${pi/2} 0" />
+    <origin xyz="0.431 0.1875 1.0575" rpy="0 ${pi/2} 0" />
   </joint>
   <link name="ur_mount_B"/>
@@ -74,5 +74,5 @@
     <parent link="arm_shelf"/>
     <child link="ur_mount_B"/>
-    <origin xyz="${-0.615/2} ${0.728/2 - 0.13} ${1.353 - 0.13}" rpy="0 ${-pi/2} 0" />
+    <origin xyz="-0.363 0.1875 1.0575" rpy="0 ${-pi/2} 0" />
   </joint>
   <!-- 创建 UR 机器人 (Jazzy: 仅传几何相关参数) -->
