Commit message: 引出校准参数，设置初始关节角

File: src/my_env/my_env_control/urdf/my_env_control.urdf.xacro (robot description, xacro)
@@ -5,6 +5,10 @@
   <!-- Jazzy: ros2_control 宏分别来自 ur_robot_driver、robotiq_description 和 dh_ag95_description -->
   <xacro:include filename="$(find ur_robot_driver)/urdf/ur.ros2_control.xacro" />
-  <xacro:include filename="$(find robotiq_description)/urdf/2f_85.ros2_control.xacro" />
-  <xacro:include filename="$(find dh_ag95_description)/urdf/dh_ag95.ros2_control.xacro" />
+  <xacro:if value="${gripper_type == 'robotiq_2f85'}">
+    <xacro:include filename="$(find robotiq_description)/urdf/2f_85.ros2_control.xacro" />
+  </xacro:if>
+  <xacro:if value="${gripper_type == 'dh_ag95'}">
+    <xacro:include filename="$(find dh_ag95_description)/urdf/dh_ag95.ros2_control.xacro" />
+  </xacro:if>
   <!-- 我们需要指定用于参数化描述的参数 -->
   <!-- 双臂前缀/型号等属性现在统一由 dual_arm_config.xacro 提供（通过 my_env_macro.urdf.xacro 间接 include） -->
@@ -22,5 +26,4 @@
   <xacro:arg name="ur_A_trajectory_port" default="50004"/>
   <xacro:arg name="ur_A_rw_rate" default="0"/>
-  <xacro:arg name="ur_A_kinematics_parameters_file" default="$(find ur_description)/config/${ur_A_ur_type}/default_kinematics.yaml"/>
   <!-- UR_B 机器人参数 (前缀和型号固定为 property) -->
   <xacro:arg name="ur_B_robot_ip" default="192.168.1.102"/>
@@ -30,5 +33,4 @@
   <xacro:arg name="ur_B_trajectory_port" default="50014"/>
   <xacro:arg name="ur_B_rw_rate" default="0"/>
-  <xacro:arg name="ur_B_kinematics_parameters_file" default="$(find ur_description)/config/${ur_B_ur_type}/default_kinematics.yaml"/>
   <!-- 夹爪和相机参数 -->
   <xacro:arg name="g2f85_A_com_port" default="/dev/ttyUSB0"/>
@@ -65,5 +67,6 @@
   <xacro:arg name="ag95_B_gripper_id" default="2"/>
   <!-- 初始位置文件 -->
-  <xacro:arg name="initial_positions_file" default="$(find ur_description)/config/initial_positions.yaml"/>
+  <xacro:arg name="ur_A_initial_positions_file" default="$(find my_env_control)/config/ur_A_initial_positions.yaml"/>
+  <xacro:arg name="ur_B_initial_positions_file" default="$(find my_env_control)/config/ur_B_initial_positions.yaml"/>
   <!-- ============================================ -->
   <!-- UR ros2_control 可选参数（两臂共享）           -->
@@ -90,5 +93,6 @@
   <xacro:arg name="g2f85_gripper_closed_position" default="0.7929"/>
   <!-- 转换为 property 以便在调用中使用 substitution -->
-  <xacro:property name="initial_positions_file" default="$(arg initial_positions_file)"/>
+  <xacro:property name="ur_A_initial_positions_file" value="$(arg ur_A_initial_positions_file)"/>
+  <xacro:property name="ur_B_initial_positions_file" value="$(arg ur_B_initial_positions_file)"/>
   <!-- Jazzy: 纯几何描述（仅传几何参数给 my_env） -->
   <xacro:my_env
@@ -106,5 +110,5 @@
     name="ur_A"
     tf_prefix="${arm_A_tf_prefix}ur_"
-    kinematics_parameters_file="$(find ur_description)/config/${ur_A_ur_type}/default_kinematics.yaml"
+    kinematics_parameters_file="${ur_A_kinematics_parameters_file}"
     robot_ip="$(arg ur_A_robot_ip)"
     script_filename="$(arg script_filename)"
@@ -119,5 +123,5 @@
     mock_sensor_commands="$(arg use_fake_sensor_commands)"
     headless_mode="$(arg ur_headless_mode)"
-    initial_positions="${xacro.load_yaml(initial_positions_file)}"
+    initial_positions="${xacro.load_yaml(ur_A_initial_positions_file)}"
     transmission_hw_interface="$(arg ur_transmission_hw_interface)"
     use_tool_communication="$(arg ur_use_tool_communication)"
@@ -138,5 +142,5 @@
     name="ur_B"
     tf_prefix="${arm_B_tf_prefix}ur_"
-    kinematics_parameters_file="$(find ur_description)/config/${ur_B_ur_type}/default_kinematics.yaml"
+    kinematics_parameters_file="${ur_B_kinematics_parameters_file}"
     robot_ip="$(arg ur_B_robot_ip)"
     script_filename="$(arg script_filename)"
@@ -151,5 +155,5 @@
     mock_sensor_commands="$(arg use_fake_sensor_commands)"
     headless_mode="$(arg ur_headless_mode)"
-    initial_positions="${xacro.load_yaml(initial_positions_file)}"
+    initial_positions="${xacro.load_yaml(ur_B_initial_positions_file)}"
     transmission_hw_interface="$(arg ur_transmission_hw_interface)"
     use_tool_communication="$(arg ur_use_tool_communication)"

File: src/my_env/my_env_description/urdf/dual_arm_config.xacro (robot description, xacro)
@@ -13,4 +13,5 @@
   <xacro:property name="arm_A_tf_prefix" value="arm_A_"/>
   <xacro:property name="ur_A_ur_type" value="ur5"/>
+  <xacro:property name="ur_A_kinematics_parameters_file" value="$(find my_env_control)/config/ur_A_kinematics_calibration.yaml"/>
   <!-- ============================================ -->
   <!-- 臂 B 配置                                   -->
@@ -18,4 +19,5 @@
   <xacro:property name="arm_B_tf_prefix" value="arm_B_"/>
   <xacro:property name="ur_B_ur_type" value="ur5e"/>
+  <xacro:property name="ur_B_kinematics_parameters_file" value="$(find my_env_control)/config/ur_B_kinematics_calibration.yaml"/>
   <!-- ============================================ -->
   <!-- 夹爪类型选择                                -->

File: src/my_env/my_env_description/urdf/my_arm_macro.urdf.xacro (robot description, xacro)
@@ -23,4 +23,5 @@
     parent:=world
     ur_type:=ur5e
+    kinematics_parameters_file:=''
     gripper_type:=dh_ag95
     realsense_use_nominal_extrinsics:=false
@@ -36,5 +37,10 @@
     <xacro:property name="_ur_parent" value="${parent}"/>
     <xacro:property name="_ur_joint_limits_parameters_file" value="$(find ur_description)/config/${ur_type}/joint_limits.yaml"/>
-    <xacro:property name="_ur_kinematics_parameters_file" value="$(find ur_description)/config/${ur_type}/default_kinematics.yaml"/>
+    <xacro:if value="${kinematics_parameters_file == ''}">
+      <xacro:property name="_ur_kinematics_parameters_file" value="$(find ur_description)/config/${ur_type}/default_kinematics.yaml"/>
+    </xacro:if>
+    <xacro:unless value="${kinematics_parameters_file == ''}">
+      <xacro:property name="_ur_kinematics_parameters_file" value="${kinematics_parameters_file}"/>
+    </xacro:unless>
     <xacro:property name="_ur_physical_parameters_file" value="$(find ur_description)/config/${ur_type}/physical_parameters.yaml"/>
     <xacro:property name="_ur_visual_parameters_file" value="$(find ur_description)/config/${ur_type}/visual_parameters.yaml"/>

File: src/my_env/my_env_description/urdf/my_env.urdf.xacro (robot description, xacro)
@@ -5,8 +5,5 @@
   <!-- 我们需要指定用于参数化描述的参数 -->
   <!-- 为所需的ur_type创建一个文件夹，并从ur_description包中复制文件到那里 -->
-  <!-- 夹爪和相机参数 -->
-  <!-- gripper_type 默认在 dual_arm_config.xacro 中配置，此处可通过命令行覆盖 -->
-  <xacro:arg name="gripper_type" default="dh_ag95"/>
-  <xacro:property name="gripper_type" value="$(arg gripper_type)"/>
+  <!-- 夹爪类型统一由 dual_arm_config.xacro 配置 -->
   <xacro:arg name="camera_use_nominal_extrinsics" default="false"/>
   <!-- UR 安全限位和路径参数 -->

File: src/my_env/my_env_description/urdf/my_env_macro.urdf.xacro (robot description, xacro)
@@ -82,4 +82,5 @@
     parent = "ur_mount_A"
     ur_type = "${ur_A_ur_type}"
+    kinematics_parameters_file = "${ur_A_kinematics_parameters_file}"
     gripper_type = "${gripper_type}"
     realsense_use_nominal_extrinsics = "${camera_use_nominal_extrinsics}"
@@ -96,4 +97,5 @@
     parent = "ur_mount_B"
     ur_type = "${ur_B_ur_type}"
+    kinematics_parameters_file = "${ur_B_kinematics_parameters_file}"
     gripper_type = "${gripper_type}"
     realsense_use_nominal_extrinsics = "${camera_use_nominal_extrinsics}"
