Commit message: 修复了dhag95夹爪的命名，跑通了 mujoco control 的 forward_position_controller ， joint_trajectory_controller 暂时不可用

File: src/my_env/my_env_control/urdf/my_env_control.urdf.xacro (robot description, xacro)
@@ -215,5 +215,5 @@
   <!-- arm_A AG-95 夹爪 ros2_control -->
   <xacro:dh_ag95_ros2_control
-    prefix="${arm_A_tf_prefix}"
+    prefix="${arm_A_tf_prefix}dhag95_"
     name="arm_A_ag95_hardware"
     use_fake_hardware="$(arg use_fake_hardware)"
@@ -234,5 +234,5 @@
   <!-- arm_B AG-95 夹爪 ros2_control -->
   <xacro:dh_ag95_ros2_control
-    prefix="${arm_B_tf_prefix}"
+    prefix="${arm_B_tf_prefix}dhag95_"
     name="arm_B_ag95_hardware"
     use_fake_hardware="$(arg use_fake_hardware)"

File: src/my_env/my_env_description/urdf/my_arm_macro.urdf.xacro (robot description, xacro)
@@ -59,5 +59,5 @@
     <xacro:if value="${gripper_type == 'dh_ag95'}">
       <!-- DH-Robotics AG-95 gripper parameters -->
-      <xacro:property name="_ag95_prefix" value="${tf_prefix}" />
+      <xacro:property name="_ag95_prefix" value="${tf_prefix}dhag95_" />
       <xacro:property name="_ag95_gripper_base_link" value="${_ag95_prefix}gripper_base_link" />
     </xacro:if>

File: src/my_env/my_env_mujoco/urdf/my_env_mujoco.urdf (robot description, URDF)
Before this commit: robot my_env, 73 links, 72 joints
Links:
- removed link arm_A_gripper_base_link
- removed link arm_A_gripper_finger1_finger_link
- removed link arm_A_gripper_finger1_finger_tip_link
- removed link arm_A_gripper_finger1_inner_knuckle_link
- removed link arm_A_gripper_finger1_knuckle_link
- removed link arm_A_gripper_finger2_finger_link
- removed link arm_A_gripper_finger2_finger_tip_link
- removed link arm_A_gripper_finger2_inner_knuckle_link
- removed link arm_A_gripper_finger2_knuckle_link
- removed link arm_A_realsense_color_frame
- removed link arm_A_realsense_color_optical_frame
- removed link arm_A_realsense_depth_frame
- removed link arm_A_realsense_depth_optical_frame
- removed link arm_A_realsense_infra1_frame
- removed link arm_A_realsense_infra1_optical_frame
- removed link arm_A_realsense_infra2_frame
- removed link arm_A_realsense_infra2_optical_frame
- removed link arm_B_gripper_base_link
- removed link arm_B_gripper_finger1_finger_link
- removed link arm_B_gripper_finger1_finger_tip_link
- removed link arm_B_gripper_finger1_inner_knuckle_link
- removed link arm_B_gripper_finger1_knuckle_link
- removed link arm_B_gripper_finger2_finger_link
- removed link arm_B_gripper_finger2_finger_tip_link
- removed link arm_B_gripper_finger2_inner_knuckle_link
- removed link arm_B_gripper_finger2_knuckle_link
- removed link arm_B_realsense_color_frame
- removed link arm_B_realsense_color_optical_frame
- removed link arm_B_realsense_depth_frame
- removed link arm_B_realsense_depth_optical_frame
- removed link arm_B_realsense_infra1_frame
- removed link arm_B_realsense_infra1_optical_frame
- removed link arm_B_realsense_infra2_frame
- removed link arm_B_realsense_infra2_optical_frame
- added link arm_A_dhag95_gripper_base_link, mass 0.83416; collision mesh filename=package://dh_ag95_description/meshes/visual/base_link.STL scale=0.001 0.001 0.001; visual mesh filename=package://dh_ag95_description/meshes/visual/base_link.STL scale=0.001 0.001 0.001
- added link arm_A_dhag95_gripper_finger1_finger_link, mass 0.0222871; collision mesh filename=package://dh_ag95_description/meshes/visual/rod_Link.STL scale=0.001 0.001 0.001; visual mesh filename=package://dh_ag95_description/meshes/visual/rod_Link.STL scale=0.001 0.001 0.001
- added link arm_A_dhag95_gripper_finger1_finger_tip_link, mass 0.0124305; collision mesh filename=package://dh_ag95_description/meshes/visual/distal_phalanx_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 scale=0.001 0.001 0.001; visual mesh filename=package://dh_ag95_description/meshes/visual/distal_phalanx_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 scale=0.001 0.001 0.001
- added link arm_A_dhag95_gripper_finger1_inner_knuckle_link, mass 0.0318004; collision mesh filename=package://dh_ag95_description/meshes/visual/proximal_phalan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 scale=0.001 0.001 0.001; visual mesh filename=package://dh_ag95_description/meshes/visual/proximal_phalan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 scale=0.001 0.001 0.001
- added link arm_A_dhag95_gripper_finger1_knuckle_link, mass 0.011111; collision mesh filename=package://dh_ag95_description/meshes/visual/crank_Link.STL scale=0.001 0.001 0.001; visual mesh filename=package://dh_ag95_description/meshes/visual/crank_Link.STL scale=0.001 0.001 0.001
- added link arm_A_dhag95_gripper_finger2_finger_link, mass 0.0222871; collision mesh filename=package://dh_ag95_description/meshes/visual/rod_Link.STL scale=0.001 0.001 0.001; visual mesh filename=package://dh_ag95_description/meshes/visual/rod_Link.STL scale=0.001 0.001 0.001
- added link arm_A_dhag95_gripper_finger2_finger_tip_link, mass 0.0124305; collision mesh filename=package://dh_ag95_description/meshes/visual/distal_phalanx_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 scale=0.001 0.001 0.001; visual mesh filename=package://dh_ag95_description/meshes/visual/distal_phalanx_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 scale=0.001 0.001 0.001
- added link arm_A_dhag95_gripper_finger2_inner_knuckle_link, mass 0.0318004; collision mesh filename=package://dh_ag95_description/meshes/visual/proximal_phalan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 scale=0.001 0.001 0.001; visual mesh filename=package://dh_ag95_description/meshes/visual/proximal_phalan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 scale=0.001 0.001 0.001
- added link arm_A_dhag95_gripper_finger2_knuckle_link, mass 0.011111; collision mesh filename=package://dh_ag95_description/meshes/visual/crank_Link.STL scale=0.001 0.001 0.001; visual mesh filename=package://dh_ag95_description/meshes/visual/crank_Link.STL scale=0.001 0.001 0.001
- added link arm_B_dhag95_gripper_base_link, mass 0.83416; collision mesh filename=package://dh_ag95_description/meshes/visual/base_link.STL scale=0.001 0.001 0.001; visual mesh filename=package://dh_ag95_description/meshes/visual/base_link.STL scale=0.001 0.001 0.001
- added link arm_B_dhag95_gripper_finger1_finger_link, mass 0.0222871; collision mesh filename=package://dh_ag95_description/meshes/visual/rod_Link.STL scale=0.001 0.001 0.001; visual mesh filename=package://dh_ag95_description/meshes/visual/rod_Link.STL scale=0.001 0.001 0.001
- added link arm_B_dhag95_gripper_finger1_finger_tip_link, mass 0.0124305; collision mesh filename=package://dh_ag95_description/meshes/visual/distal_phalanx_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 scale=0.001 0.001 0.001; visual mesh filename=package://dh_ag95_description/meshes/visual/distal_phalanx_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 scale=0.001 0.001 0.001
- added link arm_B_dhag95_gripper_finger1_inner_knuckle_link, mass 0.0318004; collision mesh filename=package://dh_ag95_description/meshes/visual/proximal_phalan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 scale=0.001 0.001 0.001; visual mesh filename=package://dh_ag95_description/meshes/visual/proximal_phalan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 scale=0.001 0.001 0.001
- added link arm_B_dhag95_gripper_finger1_knuckle_link, mass 0.011111; collision mesh filename=package://dh_ag95_description/meshes/visual/crank_Link.STL scale=0.001 0.001 0.001; visual mesh filename=package://dh_ag95_description/meshes/visual/crank_Link.STL scale=0.001 0.001 0.001
- added link arm_B_dhag95_gripper_finger2_finger_link, mass 0.0222871; collision mesh filename=package://dh_ag95_description/meshes/visual/rod_Link.STL scale=0.001 0.001 0.001; visual mesh filename=package://dh_ag95_description/meshes/visual/rod_Link.STL scale=0.001 0.001 0.001
- added link arm_B_dhag95_gripper_finger2_finger_tip_link, mass 0.0124305; collision mesh filename=package://dh_ag95_description/meshes/visual/distal_phalanx_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 scale=0.001 0.001 0.001; visual mesh filename=package://dh_ag95_description/meshes/visual/distal_phalanx_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 scale=0.001 0.001 0.001
- added link arm_B_dhag95_gripper_finger2_inner_knuckle_link, mass 0.0318004; collision mesh filename=package://dh_ag95_description/meshes/visual/proximal_phalan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 scale=0.001 0.001 0.001; visual mesh filename=package://dh_ag95_description/meshes/visual/proximal_phalan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 scale=0.001 0.001 0.001
- added link arm_B_dhag95_gripper_finger2_knuckle_link, mass 0.011111; collision mesh filename=package://dh_ag95_description/meshes/visual/crank_Link.STL scale=0.001 0.001 0.001; visual mesh filename=package://dh_ag95_description/meshes/visual/crank_Link.STL scale=0.001 0.001 0.001
Joints:
- removed joint arm_A_gripper_base_joint
- removed joint arm_A_gripper_finger1_finger_joint
- removed joint arm_A_gripper_finger1_finger_tip_joint
- removed joint arm_A_gripper_finger1_inner_knuckle_joint
- removed joint arm_A_gripper_finger1_joint
- removed joint arm_A_gripper_finger2_finger_joint
- removed joint arm_A_gripper_finger2_finger_tip_joint
- removed joint arm_A_gripper_finger2_inner_knuckle_joint
- removed joint arm_A_gripper_finger2_joint
- removed joint arm_A_realsense_color_joint
- removed joint arm_A_realsense_color_optical_joint
- removed joint arm_A_realsense_depth_joint
- removed joint arm_A_realsense_depth_optical_joint
- removed joint arm_A_realsense_infra1_joint
- removed joint arm_A_realsense_infra1_optical_joint
- removed joint arm_A_realsense_infra2_joint
- removed joint arm_A_realsense_infra2_optical_joint
- removed joint arm_B_gripper_base_joint
- removed joint arm_B_gripper_finger1_finger_joint
- removed joint arm_B_gripper_finger1_finger_tip_joint
- removed joint arm_B_gripper_finger1_inner_knuckle_joint
- removed joint arm_B_gripper_finger1_joint
- removed joint arm_B_gripper_finger2_finger_joint
- removed joint arm_B_gripper_finger2_finger_tip_joint
- removed joint arm_B_gripper_finger2_inner_knuckle_joint
- removed joint arm_B_gripper_finger2_joint
- removed joint arm_B_realsense_color_joint
- removed joint arm_B_realsense_color_optical_joint
- removed joint arm_B_realsense_depth_joint
- removed joint arm_B_realsense_depth_optical_joint
- removed joint arm_B_realsense_infra1_joint
- removed joint arm_B_realsense_infra1_optical_joint
- removed joint arm_B_realsense_infra2_joint
- removed joint arm_B_realsense_infra2_optical_joint
- added joint arm_A_dhag95_gripper_base_joint: type fixed, parent arm_A_realsense_shelf_child_side, child arm_A_dhag95_gripper_base_link, origin xyz=0 0 -0.0035 rpy=0 0 0
- added joint arm_A_dhag95_gripper_finger1_finger_joint: type continuous, parent arm_A_dhag95_gripper_finger1_knuckle_link, child arm_A_dhag95_gripper_finger1_finger_link, origin xyz=0.0292080077784 0 -0.0227132622407 rpy=0 0 0, axis 0 -1 0, limit lower=-3.14 upper=3.14 effort=0.1 velocity=100.0, mimic joint=arm_A_dhag95_gripper_finger1_joint multiplier=0.4563942 offset=0
- added joint arm_A_dhag95_gripper_finger1_finger_tip_joint: type continuous, parent arm_A_dhag95_gripper_finger1_inner_knuckle_link, child arm_A_dhag95_gripper_finger1_finger_tip_link, origin xyz=0.0394969463769 0 0.0382752038125 rpy=0 0 0, axis 0 1 0, limit lower=-3.14 upper=3.14 effort=0.1 velocity=100.0, mimic joint=arm_A_dhag95_gripper_finger1_joint multiplier=1.49462955 offset=0
- added joint arm_A_dhag95_gripper_finger1_inner_knuckle_joint: type continuous, parent arm_A_dhag95_gripper_base_link, child arm_A_dhag95_gripper_finger1_inner_knuckle_link, origin xyz=-0.016 0 0.10586 rpy=0 0 3.141592653589793, axis 0 -1 0, limit lower=-3.14 upper=3.14 effort=0.1 velocity=100.0, mimic joint=arm_A_dhag95_gripper_finger1_joint multiplier=1.49462955 offset=0
- added joint arm_A_dhag95_gripper_finger1_joint: type revolute, parent arm_A_dhag95_gripper_base_link, child arm_A_dhag95_gripper_finger1_knuckle_link, origin xyz=-0.016 0 0.10586 rpy=0 0 3.141592653589793, axis 0 -1 0, limit lower=0.0 upper=0.65 effort=1000 velocity=2.0
- added joint arm_A_dhag95_gripper_finger2_finger_joint: type continuous, parent arm_A_dhag95_gripper_finger2_knuckle_link, child arm_A_dhag95_gripper_finger2_finger_link, origin xyz=0.0292080077784 0 -0.0227132622407 rpy=0 0 0, axis 0 -1 0, limit lower=-3.14 upper=3.14 effort=0.1 velocity=100.0, mimic joint=arm_A_dhag95_gripper_finger1_joint multiplier=0.4563942 offset=0
- added joint arm_A_dhag95_gripper_finger2_finger_tip_joint: type continuous, parent arm_A_dhag95_gripper_finger2_inner_knuckle_link, child arm_A_dhag95_gripper_finger2_finger_tip_link, origin xyz=0.0394969463769 0 0.0382752038125 rpy=0 0 0, axis 0 1 0, limit lower=-3.14 upper=3.14 effort=0.1 velocity=100.0, mimic joint=arm_A_dhag95_gripper_finger1_joint multiplier=1.49462955 offset=0
- added joint arm_A_dhag95_gripper_finger2_inner_knuckle_joint: type continuous, parent arm_A_dhag95_gripper_base_link, child arm_A_dhag95_gripper_finger2_inner_knuckle_link, origin xyz=0.016 0 0.10586 rpy=0 0 0, axis 0 -1 0, limit lower=-3.14 upper=3.14 effort=0.1 velocity=100.0, mimic joint=arm_A_dhag95_gripper_finger1_joint multiplier=1.49462955 offset=0
- added joint arm_A_dhag95_gripper_finger2_joint: type revolute, parent arm_A_dhag95_gripper_base_link, child arm_A_dhag95_gripper_finger2_knuckle_link, origin xyz=0.016 0 0.10586 rpy=0 0 0, axis 0 -1 0, limit lower=-3.14 upper=3.14 effort=1000 velocity=100.0, mimic joint=arm_A_dhag95_gripper_finger1_joint multiplier=1.0 offset=0.0
- added joint arm_B_dhag95_gripper_base_joint: type fixed, parent arm_B_realsense_shelf_child_side, child arm_B_dhag95_gripper_base_link, origin xyz=0 0 -0.0035 rpy=0 0 0
- added joint arm_B_dhag95_gripper_finger1_finger_joint: type continuous, parent arm_B_dhag95_gripper_finger1_knuckle_link, child arm_B_dhag95_gripper_finger1_finger_link, origin xyz=0.0292080077784 0 -0.0227132622407 rpy=0 0 0, axis 0 -1 0, limit lower=-3.14 upper=3.14 effort=0.1 velocity=100.0, mimic joint=arm_B_dhag95_gripper_finger1_joint multiplier=0.4563942 offset=0
- added joint arm_B_dhag95_gripper_finger1_finger_tip_joint: type continuous, parent arm_B_dhag95_gripper_finger1_inner_knuckle_link, child arm_B_dhag95_gripper_finger1_finger_tip_link, origin xyz=0.0394969463769 0 0.0382752038125 rpy=0 0 0, axis 0 1 0, limit lower=-3.14 upper=3.14 effort=0.1 velocity=100.0, mimic joint=arm_B_dhag95_gripper_finger1_joint multiplier=1.49462955 offset=0
- added joint arm_B_dhag95_gripper_finger1_inner_knuckle_joint: type continuous, parent arm_B_dhag95_gripper_base_link, child arm_B_dhag95_gripper_finger1_inner_knuckle_link, origin xyz=-0.016 0 0.10586 rpy=0 0 3.141592653589793, axis 0 -1 0, limit lower=-3.14 upper=3.14 effort=0.1 velocity=100.0, mimic joint=arm_B_dhag95_gripper_finger1_joint multiplier=1.49462955 offset=0
- added joint arm_B_dhag95_gripper_finger1_joint: type revolute, parent arm_B_dhag95_gripper_base_link, child arm_B_dhag95_gripper_finger1_knuckle_link, origin xyz=-0.016 0 0.10586 rpy=0 0 3.141592653589793, axis 0 -1 0, limit lower=0.0 upper=0.65 effort=1000 velocity=2.0
- added joint arm_B_dhag95_gripper_finger2_finger_joint: type continuous, parent arm_B_dhag95_gripper_finger2_knuckle_link, child arm_B_dhag95_gripper_finger2_finger_link, origin xyz=0.0292080077784 0 -0.0227132622407 rpy=0 0 0, axis 0 -1 0, limit lower=-3.14 upper=3.14 effort=0.1 velocity=100.0, mimic joint=arm_B_dhag95_gripper_finger1_joint multiplier=0.4563942 offset=0
- added joint arm_B_dhag95_gripper_finger2_finger_tip_joint: type continuous, parent arm_B_dhag95_gripper_finger2_inner_knuckle_link, child arm_B_dhag95_gripper_finger2_finger_tip_link, origin xyz=0.0394969463769 0 0.0382752038125 rpy=0 0 0, axis 0 1 0, limit lower=-3.14 upper=3.14 effort=0.1 velocity=100.0, mimic joint=arm_B_dhag95_gripper_finger1_joint multiplier=1.49462955 offset=0
- added joint arm_B_dhag95_gripper_finger2_inner_knuckle_joint: type continuous, parent arm_B_dhag95_gripper_base_link, child arm_B_dhag95_gripper_finger2_inner_knuckle_link, origin xyz=0.016 0 0.10586 rpy=0 0 0, axis 0 -1 0, limit lower=-3.14 upper=3.14 effort=0.1 velocity=100.0, mimic joint=arm_B_dhag95_gripper_finger1_joint multiplier=1.49462955 offset=0
- added joint arm_B_dhag95_gripper_finger2_joint: type revolute, parent arm_B_dhag95_gripper_base_link, child arm_B_dhag95_gripper_finger2_knuckle_link, origin xyz=0.016 0 0.10586 rpy=0 0 0, axis 0 -1 0, limit lower=-3.14 upper=3.14 effort=1000 velocity=100.0, mimic joint=arm_B_dhag95_gripper_finger1_joint multiplier=1.0 offset=0.0
- joint arm_A__tcp_joint: parent arm_A_gripper_base_link -> arm_A_dhag95_gripper_base_link
- joint arm_B__tcp_joint: parent arm_B_gripper_base_link -> arm_B_dhag95_gripper_base_link

File: src/my_env/my_env_mujoco/urdf/my_env_mujoco.urdf.xacro (robot description, xacro)
@@ -5,22 +5,11 @@
   <!-- Jazzy: mujoco ros2_control 宏（已移至 my_env_mujoco 包） -->
   <xacro:include filename="$(find my_env_mujoco)/urdf/my_arm_mujoco_control.urdf.xacro"/>
-  <!-- 我们需要指定用于参数化描述的参数 -->
-  <!-- 为所需的ur_type创建一个文件夹，并从ur_description包中复制文件到那里 -->
-  <!-- UR_A 机器人参数 (固定为 property) -->
-  <xacro:property name="arm_A_tf_prefix" value="arm_A_"/>
-  <xacro:property name="ur_A_ur_type" value="ur5"/>
-  <!-- UR_B 机器人参数 (固定为 property) -->
-  <xacro:property name="arm_B_tf_prefix" value="arm_B_"/>
-  <xacro:property name="ur_B_ur_type" value="ur5e"/>
   <!-- 控制参数 -->
-  <xacro:arg name="use_fake_hardware" default="true" />
-  <xacro:arg name="fake_sensor_commands" default="true" />
-  <xacro:arg name="use_sim_mujoco" default="true" />
   <xacro:arg name="mjcf_file_path" default="$(find my_env_mujoco)/mjcf/my_env_mujoco.xml"/>
-  <xacro:arg name="generate_ros2_control" default="false" />
-  <!-- <xacro:arg name="ur_A_initial_positions" default="{shoulder_pan_joint=0.0,shoulder_lift_joint=-1.57,elbow_joint=0.0,wrist_1_joint=-1.57,wrist_2_joint=0.0,wrist_3_joint=0.0}"/> -->
-  <!-- <xacro:arg name="ur_B_initial_positions" default="{shoulder_pan_joint=0.0,shoulder_lift_joint=-1.57,elbow_joint=0.0,wrist_1_joint=-1.57,wrist_2_joint=0.0,wrist_3_joint=0.0}"/> -->
+  <xacro:arg name="pids_config_file_path" default="$(find my_env_control)/config/mujoco_pids_config.yaml"/>
+  <xacro:arg name="ur_A_initial_positions_file" default="$(find my_env_control)/config/ur_A_initial_positions.yaml"/>
+  <xacro:arg name="ur_B_initial_positions_file" default="$(find my_env_control)/config/ur_B_initial_positions.yaml"/>
   <!-- 夹爪和相机参数 -->
-  <xacro:arg name="camera_use_nominal_extrinsics" default="true"/>
+  <xacro:arg name="camera_use_nominal_extrinsics" default="false"/>
   <!-- UR 安全限位和路径参数（几何用） -->
   <xacro:arg name="safety_limits" default="false"/>
@@ -33,7 +22,6 @@
   <xacro:arg name="mujoco_sim_speed_factor" default="1.0"/>
   <xacro:arg name="mujoco_headless" default="false"/>
-  <!-- 两臂初始关节角（property 形式，可在 launch 文件中通过 xacro 参数覆盖） -->
-  <xacro:property name="ur_A_initial_positions" value="${dict(shoulder_pan_joint=-1.57,shoulder_lift_joint=-1.27,elbow_joint=1.0,wrist_1_joint=-1.3,wrist_2_joint=-1.57,wrist_3_joint=-1.57)}"/>
-  <xacro:property name="ur_B_initial_positions" value="${dict(shoulder_pan_joint=-1.57,shoulder_lift_joint=-2.27,elbow_joint=-0.2,wrist_1_joint=-2.24,wrist_2_joint=1.57,wrist_3_joint=1.57)}"/>
+  <xacro:property name="ur_A_initial_positions_file" value="$(arg ur_A_initial_positions_file)"/>
+  <xacro:property name="ur_B_initial_positions_file" value="$(arg ur_B_initial_positions_file)"/>
   <!-- Jazzy: 纯几何描述（仅传几何参数给 my_env） -->
   <xacro:my_env
@@ -48,32 +36,33 @@
   <!-- 只保留一个 ros2_control system：只启动一次 MujocoSystemInterface -->
   <!-- ============================================ -->
-  <xacro:if value="$(arg use_sim_mujoco)">
-    <xacro:property name="arm_A_ur_prefix" value="${arm_A_tf_prefix}ur_"/> <!-- ! Match the prefix in my_arm_macro.urdf.xacro -->
-    <xacro:property name="arm_B_ur_prefix" value="${arm_B_tf_prefix}ur_"/> <!-- ! Match the prefix in my_arm_macro.urdf.xacro -->
-    <xacro:property name="arm_A_realsense_prefix" value="${arm_A_tf_prefix}realsense_"/> <!-- ! append the '_' in the prefix -->
-    <xacro:property name="arm_B_realsense_prefix" value="${arm_B_tf_prefix}realsense_"/> <!-- ! append the '_' in the prefix -->
-    <xacro:property name="arm_A_gripper_prefix" value="${arm_A_tf_prefix}"/> <!-- ! Match the prefix in my_arm_macro.urdf.xacro -->
-    <xacro:property name="arm_B_gripper_prefix" value="${arm_B_tf_prefix}"/> <!-- ! Match the prefix in my_arm_macro.urdf.xacro -->
-    <ros2_control name="my_env_ros2_mujoco" type="system">
-      <hardware>
-        <plugin>mujoco_ros2_control/MujocoSystemInterface</plugin>
-        <param name="mujoco_model">$(arg mjcf_file_path)</param>
-        <!-- Override the slowdown settings in the Simulate App -->
-        <param name="sim_speed_factor">$(arg mujoco_sim_speed_factor)</param>
-        <!-- If set to true, will not launch the Simulate App window -->
-        <param name="headless">$(arg mujoco_headless)</param>
-      </hardware>
-      <!-- 把两套机械臂的 joint/sensor 接口“塞进同一个 system”里 -->
-      <xacro:my_arm_mujoco_control
-          ur_tf_prefix="${arm_A_ur_prefix}"
-          realsense_tf_prefix="${arm_A_realsense_prefix}"
-          gripper_tf_prefix="${arm_A_gripper_prefix}"
-          ur_initial_positions="${ur_A_initial_positions}"/>
-      <xacro:my_arm_mujoco_control
-          ur_tf_prefix="${arm_B_ur_prefix}"
-          realsense_tf_prefix="${arm_B_realsense_prefix}"
-          gripper_tf_prefix="${arm_B_gripper_prefix}"
-          ur_initial_positions="${ur_B_initial_positions}"/>
-    </ros2_control>
-  </xacro:if>
+  <xacro:property name="arm_A_ur_prefix" value="${arm_A_tf_prefix}ur_"/> <!-- ! Match the prefix in my_arm_macro.urdf.xacro -->
+  <xacro:property name="arm_B_ur_prefix" value="${arm_B_tf_prefix}ur_"/> <!-- ! Match the prefix in my_arm_macro.urdf.xacro -->
+  <xacro:property name="arm_A_realsense_prefix" value="${arm_A_tf_prefix}realsense_"/> <!-- ! append the '_' in the prefix -->
+  <xacro:property name="arm_B_realsense_prefix" value="${arm_B_tf_prefix}realsense_"/> <!-- ! append the '_' in the prefix -->
+  <xacro:property name="arm_A_gripper_prefix" value="${arm_A_tf_prefix}dhag95_"/> <!-- ! Match the prefix in my_arm_macro.urdf.xacro -->
+  <xacro:property name="arm_B_gripper_prefix" value="${arm_B_tf_prefix}dhag95_"/> <!-- ! Match the prefix in my_arm_macro.urdf.xacro -->
+  <ros2_control name="my_env_ros2_mujoco" type="system">
+    <hardware>
+      <plugin>mujoco_ros2_control/MujocoSystemInterface</plugin>
+      <param name="mujoco_model">$(arg mjcf_file_path)</param>
+      <!-- Optional: load PID gains from a ROS parameters YAML file.
+        Enables position/velocity PID control for velocity, motor, and custom actuators. -->
+      <param name="pids_config_file">$(arg pids_config_file_path)</param>
+      <!-- Override the slowdown settings in the Simulate App -->
+      <param name="sim_speed_factor">$(arg mujoco_sim_speed_factor)</param>
+      <!-- If set to true, will not launch the Simulate App window -->
+      <param name="headless">$(arg mujoco_headless)</param>
+    </hardware>
+    <!-- 把两套机械臂的 joint/sensor 接口“塞进同一个 system”里 -->
+    <xacro:my_arm_mujoco_control
+        ur_tf_prefix="${arm_A_ur_prefix}"
+        realsense_tf_prefix="${arm_A_realsense_prefix}"
+        gripper_tf_prefix="${arm_A_gripper_prefix}"
+        ur_initial_positions="${xacro.load_yaml(ur_A_initial_positions_file)}"/>
+    <xacro:my_arm_mujoco_control
+        ur_tf_prefix="${arm_B_ur_prefix}"
+        realsense_tf_prefix="${arm_B_realsense_prefix}"
+        gripper_tf_prefix="${arm_B_gripper_prefix}"
+        ur_initial_positions="${xacro.load_yaml(ur_B_initial_positions_file)}"/>
+  </ros2_control>
 </robot>
