Commit message: 修复了dhag95夹爪的命名，跑通了 mujoco control 的 forward_position_controller ， joint_trajectory_controller 暂时不可用

File: src/my_env/my_env_mujoco/urdf/my_env_mujoco_fixed.urdf (robot description, URDF)
Before this commit: robot my_env, 73 links, 72 joints
Links:
- removed link arm_A_gripper_base_link
- removed link arm_A_gripper_finger1_finger_link
- removed link arm_A_gripper_finger1_finger_tip_link
- removed link arm_A_gripper_finger1_inner_knuckle_link
- removed link arm_A_gripper_finger1_knuckle_link
- removed link arm_A_gripper_finger2_finger_link
- removed link arm_A_gripper_finger2_finger_tip_link
- removed link arm_A_gripper_finger2_inner_knuckle_link
- removed link arm_A_gripper_finger2_knuckle_link
- removed link arm_A_realsense_color_frame
- removed link arm_A_realsense_color_optical_frame
- removed link arm_A_realsense_depth_frame
- removed link arm_A_realsense_depth_optical_frame
- removed link arm_A_realsense_infra1_frame
- removed link arm_A_realsense_infra1_optical_frame
- removed link arm_A_realsense_infra2_frame
- removed link arm_A_realsense_infra2_optical_frame
- removed link arm_B_gripper_base_link
- removed link arm_B_gripper_finger1_finger_link
- removed link arm_B_gripper_finger1_finger_tip_link
- removed link arm_B_gripper_finger1_inner_knuckle_link
- removed link arm_B_gripper_finger1_knuckle_link
- removed link arm_B_gripper_finger2_finger_link
- removed link arm_B_gripper_finger2_finger_tip_link
- removed link arm_B_gripper_finger2_inner_knuckle_link
- removed link arm_B_gripper_finger2_knuckle_link
- removed link arm_B_realsense_color_frame
- removed link arm_B_realsense_color_optical_frame
- removed link arm_B_realsense_depth_frame
- removed link arm_B_realsense_depth_optical_frame
- removed link arm_B_realsense_infra1_frame
- removed link arm_B_realsense_infra1_optical_frame
- removed link arm_B_realsense_infra2_frame
- removed link arm_B_realsense_infra2_optical_frame
- added link arm_A_dhag95_gripper_base_link, mass 0.83416; collision mesh filename=../meshes/base_link_36df6ff8.STL; visual mesh filename=../meshes/base_link_36df6ff8.STL
- added link arm_A_dhag95_gripper_finger1_finger_link, mass 0.0222871; collision mesh filename=../meshes/rod_Link_4ed0e7b8.STL; visual mesh filename=../meshes/rod_Link_4ed0e7b8.STL
- added link arm_A_dhag95_gripper_finger1_finger_tip_link, mass 0.0124305; collision mesh filename=../meshes/distal_phalanx_Link_710b7cbe.STL; visual mesh filename=../meshes/distal_phalanx_Link_710b7cbe.STL
- added link arm_A_dhag95_gripper_finger1_inner_knuckle_link, mass 0.0318004; collision mesh filename=../meshes/proximal_phalanx_Link_d2c93b56.STL; visual mesh filename=../meshes/proximal_phalanx_Link_d2c93b56.STL
- added link arm_A_dhag95_gripper_finger1_knuckle_link, mass 0.011111; collision mesh filename=../meshes/crank_Link_27946ce5.STL; visual mesh filename=../meshes/crank_Link_27946ce5.STL
- added link arm_A_dhag95_gripper_finger2_finger_link, mass 0.0222871; collision mesh filename=../meshes/rod_Link_4ed0e7b8.STL; visual mesh filename=../meshes/rod_Link_4ed0e7b8.STL
- added link arm_A_dhag95_gripper_finger2_finger_tip_link, mass 0.0124305; collision mesh filename=../meshes/distal_phalanx_Link_710b7cbe.STL; visual mesh filename=../meshes/distal_phalanx_Link_710b7cbe.STL
- added link arm_A_dhag95_gripper_finger2_inner_knuckle_link, mass 0.0318004; collision mesh filename=../meshes/proximal_phalanx_Link_d2c93b56.STL; visual mesh filename=../meshes/proximal_phalanx_Link_d2c93b56.STL
- added link arm_A_dhag95_gripper_finger2_knuckle_link, mass 0.011111; collision mesh filename=../meshes/crank_Link_27946ce5.STL; visual mesh filename=../meshes/crank_Link_27946ce5.STL
- added link arm_B_dhag95_gripper_base_link, mass 0.83416; collision mesh filename=../meshes/base_link_36df6ff8.STL; visual mesh filename=../meshes/base_link_36df6ff8.STL
- added link arm_B_dhag95_gripper_finger1_finger_link, mass 0.0222871; collision mesh filename=../meshes/rod_Link_4ed0e7b8.STL; visual mesh filename=../meshes/rod_Link_4ed0e7b8.STL
- added link arm_B_dhag95_gripper_finger1_finger_tip_link, mass 0.0124305; collision mesh filename=../meshes/distal_phalanx_Link_710b7cbe.STL; visual mesh filename=../meshes/distal_phalanx_Link_710b7cbe.STL
- added link arm_B_dhag95_gripper_finger1_inner_knuckle_link, mass 0.0318004; collision mesh filename=../meshes/proximal_phalanx_Link_d2c93b56.STL; visual mesh filename=../meshes/proximal_phalanx_Link_d2c93b56.STL
- added link arm_B_dhag95_gripper_finger1_knuckle_link, mass 0.011111; collision mesh filename=../meshes/crank_Link_27946ce5.STL; visual mesh filename=../meshes/crank_Link_27946ce5.STL
- added link arm_B_dhag95_gripper_finger2_finger_link, mass 0.0222871; collision mesh filename=../meshes/rod_Link_4ed0e7b8.STL; visual mesh filename=../meshes/rod_Link_4ed0e7b8.STL
- added link arm_B_dhag95_gripper_finger2_finger_tip_link, mass 0.0124305; collision mesh filename=../meshes/distal_phalanx_Link_710b7cbe.STL; visual mesh filename=../meshes/distal_phalanx_Link_710b7cbe.STL
- added link arm_B_dhag95_gripper_finger2_inner_knuckle_link, mass 0.0318004; collision mesh filename=../meshes/proximal_phalanx_Link_d2c93b56.STL; visual mesh filename=../meshes/proximal_phalanx_Link_d2c93b56.STL
- added link arm_B_dhag95_gripper_finger2_knuckle_link, mass 0.011111; collision mesh filename=../meshes/crank_Link_27946ce5.STL; visual mesh filename=../meshes/crank_Link_27946ce5.STL
Joints:
- removed joint arm_A_gripper_base_joint
- removed joint arm_A_gripper_finger1_finger_joint
- removed joint arm_A_gripper_finger1_finger_tip_joint
- removed joint arm_A_gripper_finger1_inner_knuckle_joint
- removed joint arm_A_gripper_finger1_joint
- removed joint arm_A_gripper_finger2_finger_joint
- removed joint arm_A_gripper_finger2_finger_tip_joint
- removed joint arm_A_gripper_finger2_inner_knuckle_joint
- removed joint arm_A_gripper_finger2_joint
- removed joint arm_A_realsense_color_joint
- removed joint arm_A_realsense_color_optical_joint
- removed joint arm_A_realsense_depth_joint
- removed joint arm_A_realsense_depth_optical_joint
- removed joint arm_A_realsense_infra1_joint
- removed joint arm_A_realsense_infra1_optical_joint
- removed joint arm_A_realsense_infra2_joint
- removed joint arm_A_realsense_infra2_optical_joint
- removed joint arm_B_gripper_base_joint
- removed joint arm_B_gripper_finger1_finger_joint
- removed joint arm_B_gripper_finger1_finger_tip_joint
- removed joint arm_B_gripper_finger1_inner_knuckle_joint
- removed joint arm_B_gripper_finger1_joint
- removed joint arm_B_gripper_finger2_finger_joint
- removed joint arm_B_gripper_finger2_finger_tip_joint
- removed joint arm_B_gripper_finger2_inner_knuckle_joint
- removed joint arm_B_gripper_finger2_joint
- removed joint arm_B_realsense_color_joint
- removed joint arm_B_realsense_color_optical_joint
- removed joint arm_B_realsense_depth_joint
- removed joint arm_B_realsense_depth_optical_joint
- removed joint arm_B_realsense_infra1_joint
- removed joint arm_B_realsense_infra1_optical_joint
- removed joint arm_B_realsense_infra2_joint
- removed joint arm_B_realsense_infra2_optical_joint
- added joint arm_A_dhag95_gripper_base_joint: type fixed, parent arm_A_realsense_shelf_child_side, child arm_A_dhag95_gripper_base_link, origin xyz=0 0 -0.0035 rpy=0 0 0
- added joint arm_A_dhag95_gripper_finger1_finger_joint: type continuous, parent arm_A_dhag95_gripper_finger1_knuckle_link, child arm_A_dhag95_gripper_finger1_finger_link, origin xyz=0.0292080077784 0 -0.0227132622407 rpy=0 0 0, axis 0 -1 0, limit lower=-3.14 upper=3.14 effort=0.1 velocity=100.0, mimic joint=arm_A_dhag95_gripper_finger1_joint multiplier=0.4563942 offset=0
- added joint arm_A_dhag95_gripper_finger1_finger_tip_joint: type continuous, parent arm_A_dhag95_gripper_finger1_inner_knuckle_link, child arm_A_dhag95_gripper_finger1_finger_tip_link, origin xyz=0.0394969463769 0 0.0382752038125 rpy=0 0 0, axis 0 1 0, limit lower=-3.14 upper=3.14 effort=0.1 velocity=100.0, mimic joint=arm_A_dhag95_gripper_finger1_joint multiplier=1.49462955 offset=0
- added joint arm_A_dhag95_gripper_finger1_inner_knuckle_joint: type continuous, parent arm_A_dhag95_gripper_base_link, child arm_A_dhag95_gripper_finger1_inner_knuckle_link, origin xyz=-0.016 0 0.10586 rpy=0 0 3.141592653589793, axis 0 -1 0, limit lower=-3.14 upper=3.14 effort=0.1 velocity=100.0, mimic joint=arm_A_dhag95_gripper_finger1_joint multiplier=1.49462955 offset=0
- added joint arm_A_dhag95_gripper_finger1_joint: type revolute, parent arm_A_dhag95_gripper_base_link, child arm_A_dhag95_gripper_finger1_knuckle_link, origin xyz=-0.016 0 0.10586 rpy=0 0 3.141592653589793, axis 0 -1 0, limit lower=0.0 upper=0.65 effort=1000 velocity=2.0
- added joint arm_A_dhag95_gripper_finger2_finger_joint: type continuous, parent arm_A_dhag95_gripper_finger2_knuckle_link, child arm_A_dhag95_gripper_finger2_finger_link, origin xyz=0.0292080077784 0 -0.0227132622407 rpy=0 0 0, axis 0 -1 0, limit lower=-3.14 upper=3.14 effort=0.1 velocity=100.0, mimic joint=arm_A_dhag95_gripper_finger1_joint multiplier=0.4563942 offset=0
- added joint arm_A_dhag95_gripper_finger2_finger_tip_joint: type continuous, parent arm_A_dhag95_gripper_finger2_inner_knuckle_link, child arm_A_dhag95_gripper_finger2_finger_tip_link, origin xyz=0.0394969463769 0 0.0382752038125 rpy=0 0 0, axis 0 1 0, limit lower=-3.14 upper=3.14 effort=0.1 velocity=100.0, mimic joint=arm_A_dhag95_gripper_finger1_joint multiplier=1.49462955 offset=0
- added joint arm_A_dhag95_gripper_finger2_inner_knuckle_joint: type continuous, parent arm_A_dhag95_gripper_base_link, child arm_A_dhag95_gripper_finger2_inner_knuckle_link, origin xyz=0.016 0 0.10586 rpy=0 0 0, axis 0 -1 0, limit lower=-3.14 upper=3.14 effort=0.1 velocity=100.0, mimic joint=arm_A_dhag95_gripper_finger1_joint multiplier=1.49462955 offset=0
- added joint arm_A_dhag95_gripper_finger2_joint: type revolute, parent arm_A_dhag95_gripper_base_link, child arm_A_dhag95_gripper_finger2_knuckle_link, origin xyz=0.016 0 0.10586 rpy=0 0 0, axis 0 -1 0, limit lower=-3.14 upper=3.14 effort=1000 velocity=100.0, mimic joint=arm_A_dhag95_gripper_finger1_joint multiplier=1.0 offset=0.0
- added joint arm_B_dhag95_gripper_base_joint: type fixed, parent arm_B_realsense_shelf_child_side, child arm_B_dhag95_gripper_base_link, origin xyz=0 0 -0.0035 rpy=0 0 0
- added joint arm_B_dhag95_gripper_finger1_finger_joint: type continuous, parent arm_B_dhag95_gripper_finger1_knuckle_link, child arm_B_dhag95_gripper_finger1_finger_link, origin xyz=0.0292080077784 0 -0.0227132622407 rpy=0 0 0, axis 0 -1 0, limit lower=-3.14 upper=3.14 effort=0.1 velocity=100.0, mimic joint=arm_B_dhag95_gripper_finger1_joint multiplier=0.4563942 offset=0
- added joint arm_B_dhag95_gripper_finger1_finger_tip_joint: type continuous, parent arm_B_dhag95_gripper_finger1_inner_knuckle_link, child arm_B_dhag95_gripper_finger1_finger_tip_link, origin xyz=0.0394969463769 0 0.0382752038125 rpy=0 0 0, axis 0 1 0, limit lower=-3.14 upper=3.14 effort=0.1 velocity=100.0, mimic joint=arm_B_dhag95_gripper_finger1_joint multiplier=1.49462955 offset=0
- added joint arm_B_dhag95_gripper_finger1_inner_knuckle_joint: type continuous, parent arm_B_dhag95_gripper_base_link, child arm_B_dhag95_gripper_finger1_inner_knuckle_link, origin xyz=-0.016 0 0.10586 rpy=0 0 3.141592653589793, axis 0 -1 0, limit lower=-3.14 upper=3.14 effort=0.1 velocity=100.0, mimic joint=arm_B_dhag95_gripper_finger1_joint multiplier=1.49462955 offset=0
- added joint arm_B_dhag95_gripper_finger1_joint: type revolute, parent arm_B_dhag95_gripper_base_link, child arm_B_dhag95_gripper_finger1_knuckle_link, origin xyz=-0.016 0 0.10586 rpy=0 0 3.141592653589793, axis 0 -1 0, limit lower=0.0 upper=0.65 effort=1000 velocity=2.0
- added joint arm_B_dhag95_gripper_finger2_finger_joint: type continuous, parent arm_B_dhag95_gripper_finger2_knuckle_link, child arm_B_dhag95_gripper_finger2_finger_link, origin xyz=0.0292080077784 0 -0.0227132622407 rpy=0 0 0, axis 0 -1 0, limit lower=-3.14 upper=3.14 effort=0.1 velocity=100.0, mimic joint=arm_B_dhag95_gripper_finger1_joint multiplier=0.4563942 offset=0
- added joint arm_B_dhag95_gripper_finger2_finger_tip_joint: type continuous, parent arm_B_dhag95_gripper_finger2_inner_knuckle_link, child arm_B_dhag95_gripper_finger2_finger_tip_link, origin xyz=0.0394969463769 0 0.0382752038125 rpy=0 0 0, axis 0 1 0, limit lower=-3.14 upper=3.14 effort=0.1 velocity=100.0, mimic joint=arm_B_dhag95_gripper_finger1_joint multiplier=1.49462955 offset=0
- added joint arm_B_dhag95_gripper_finger2_inner_knuckle_joint: type continuous, parent arm_B_dhag95_gripper_base_link, child arm_B_dhag95_gripper_finger2_inner_knuckle_link, origin xyz=0.016 0 0.10586 rpy=0 0 0, axis 0 -1 0, limit lower=-3.14 upper=3.14 effort=0.1 velocity=100.0, mimic joint=arm_B_dhag95_gripper_finger1_joint multiplier=1.49462955 offset=0
- added joint arm_B_dhag95_gripper_finger2_joint: type revolute, parent arm_B_dhag95_gripper_base_link, child arm_B_dhag95_gripper_finger2_knuckle_link, origin xyz=0.016 0 0.10586 rpy=0 0 0, axis 0 -1 0, limit lower=-3.14 upper=3.14 effort=1000 velocity=100.0, mimic joint=arm_B_dhag95_gripper_finger1_joint multiplier=1.0 offset=0.0
- joint arm_A__tcp_joint: parent arm_A_gripper_base_link -> arm_A_dhag95_gripper_base_link
- joint arm_B__tcp_joint: parent arm_B_gripper_base_link -> arm_B_dhag95_gripper_base_link
