Commit message: 修复了 my_env mujoco ros2 control 的配置

File: src/my_env/my_env_mujoco/urdf/my_arm_mujoco_control.urdf.xacro (robot description, xacro)
@@ -4,12 +4,10 @@
     ur_tf_prefix
     realsense_tf_prefix
-    g2f85_tf_prefix
+    gripper_tf_prefix
     ur_initial_positions:=${dict(shoulder_pan_joint=0.0,shoulder_lift_joint=-1.57,elbow_joint=0.0,wrist_1_joint=-1.57,wrist_2_joint=0.0,wrist_3_joint=0.0)}
   ">
     <xacro:property name="_ur_tf_prefix" value="${ur_tf_prefix}"/>
     <xacro:property name="_ur_initial_positions" value="${ur_initial_positions}"/>
-    <xacro:property name="_realsense_tf_prefix" value="${realsense_tf_prefix}"/>
-    <xacro:property name="_g2f85_tf_prefix" value="${g2f85_tf_prefix}"/>
-    <xacro:property name="_g2f85_closed_position" value="0.7929"/>
+    <xacro:property name="_gripper_tf_prefix" value="${gripper_tf_prefix}"/>
     <!-- UR 机械臂相关 -->
     <joint name="${_ur_tf_prefix}shoulder_pan_joint">
@@ -95,20 +93,28 @@
       <state_interface name="torque.z"/>
     </sensor>
-      <!-- ! For cameras, the sensor name _must_ match the camera name in the MJCF -->
-    <sensor name="${_realsense_tf_prefix}camera">
-      <!-- Parameters will be used as is -->
-      <param name="frame_name">${_realsense_tf_prefix}link</param>
-      <param name="info_topic">/${_realsense_tf_prefix}camera/camera_info</param>
-      <param name="image_topic">/${_realsense_tf_prefix}camera/color</param>
-      <param name="depth_topic">/${_realsense_tf_prefix}camera/depth</param>
-    </sensor>
-    <!-- Robotiq 2f85 Gripper 相关 -->
-    <joint name="${_g2f85_tf_prefix}robotiq_85_left_knuckle_joint">
+    <!-- ============================================ -->
+    <!-- 夹爪（根据 gripper_type 条件选择）            -->
+    <!-- gripper_type 由 dual_arm_config.xacro 定义   -->
+    <!-- ============================================ -->
+    <!-- Robotiq 2F-85 夹爪 -->
+    <xacro:if value="${gripper_type == 'robotiq_2f85'}">
+    <joint name="${_gripper_tf_prefix}robotiq_85_left_knuckle_joint">
         <command_interface name="position" />
         <state_interface name="position">
-            <param name="initial_value">${_g2f85_closed_position}</param>
+            <param name="initial_value">0.7929</param>
         </state_interface>
         <state_interface name="velocity"/>
     </joint>
+    </xacro:if>
+    <!-- DH-Robotics AG-95 夹爪 -->
+    <xacro:if value="${gripper_type == 'dh_ag95'}">
+    <joint name="${_gripper_tf_prefix}gripper_finger1_joint">
+        <command_interface name="position" />
+        <state_interface name="position">
+            <param name="initial_value">0.0</param>
+        </state_interface>
+        <state_interface name="velocity"/>
+    </joint>
+    </xacro:if>
   </xacro:macro>
 </robot>

File: src/my_env/my_env_mujoco/urdf/my_env_mujoco.urdf.xacro (robot description, xacro)
@@ -33,6 +33,4 @@
   <xacro:arg name="mujoco_sim_speed_factor" default="1.0"/>
   <xacro:arg name="mujoco_headless" default="false"/>
-  <xacro:arg name="mujoco_camera_publish_rate" default="30.0"/>
-  <xacro:arg name="mujoco_lidar_publish_rate" default="10.0"/>
   <!-- 两臂初始关节角（property 形式，可在 launch 文件中通过 xacro 参数覆盖） -->
   <xacro:property name="ur_A_initial_positions" value="${dict(shoulder_pan_joint=-1.57,shoulder_lift_joint=-1.27,elbow_joint=1.0,wrist_1_joint=-1.3,wrist_2_joint=-1.57,wrist_3_joint=-1.57)}"/>
@@ -40,8 +38,4 @@
   <!-- Jazzy: 纯几何描述（仅传几何参数给 my_env） -->
   <xacro:my_env
-    arm_A_tf_prefix="${arm_A_tf_prefix}"
-    arm_B_tf_prefix="${arm_B_tf_prefix}"
-    ur_A_ur_type="${ur_A_ur_type}"
-    ur_B_ur_type="${ur_B_ur_type}"
     camera_use_nominal_extrinsics="$(arg camera_use_nominal_extrinsics)"
     safety_limits="$(arg safety_limits)"
@@ -59,9 +53,9 @@
     <xacro:property name="arm_A_realsense_prefix" value="${arm_A_tf_prefix}realsense_"/> <!-- ! append the '_' in the prefix -->
     <xacro:property name="arm_B_realsense_prefix" value="${arm_B_tf_prefix}realsense_"/> <!-- ! append the '_' in the prefix -->
-    <xacro:property name="arm_A_g2f85_prefix" value="${arm_A_tf_prefix}"/> <!-- ! Match the prefix in my_arm_macro.urdf.xacro -->
-    <xacro:property name="arm_B_g2f85_prefix" value="${arm_B_tf_prefix}"/> <!-- ! Match the prefix in my_arm_macro.urdf.xacro -->
+    <xacro:property name="arm_A_gripper_prefix" value="${arm_A_tf_prefix}"/> <!-- ! Match the prefix in my_arm_macro.urdf.xacro -->
+    <xacro:property name="arm_B_gripper_prefix" value="${arm_B_tf_prefix}"/> <!-- ! Match the prefix in my_arm_macro.urdf.xacro -->
     <ros2_control name="my_env_ros2_mujoco" type="system">
       <hardware>
-        <plugin>mujoco_ros2_simulation/MujocoSystemInterface</plugin>
+        <plugin>mujoco_ros2_control/MujocoSystemInterface</plugin>
         <param name="mujoco_model">$(arg mjcf_file_path)</param>
         <!-- Override the slowdown settings in the Simulate App -->
@@ -69,8 +63,4 @@
         <!-- If set to true, will not launch the Simulate App window -->
         <param name="headless">$(arg mujoco_headless)</param>
-        <!-- Publish camera images -->
-        <param name="camera_publish_rate">$(arg mujoco_camera_publish_rate)</param>
-        <!-- Publish lidar scans at 10 hz -->
-        <param name="lidar_publish_rate">$(arg mujoco_lidar_publish_rate)</param>
       </hardware>
       <!-- 把两套机械臂的 joint/sensor 接口“塞进同一个 system”里 -->
@@ -78,10 +68,10 @@
           ur_tf_prefix="${arm_A_ur_prefix}"
           realsense_tf_prefix="${arm_A_realsense_prefix}"
-          g2f85_tf_prefix="${arm_A_g2f85_prefix}"
+          gripper_tf_prefix="${arm_A_gripper_prefix}"
           ur_initial_positions="${ur_A_initial_positions}"/>
       <xacro:my_arm_mujoco_control
           ur_tf_prefix="${arm_B_ur_prefix}"
           realsense_tf_prefix="${arm_B_realsense_prefix}"
-          g2f85_tf_prefix="${arm_B_g2f85_prefix}"
+          gripper_tf_prefix="${arm_B_gripper_prefix}"
           ur_initial_positions="${ur_B_initial_positions}"/>
     </ros2_control>
