Commit message: 新增：部分完善了 space_sim 环境

File: src/envs/space_sim/space_sim_description/xacro/space_sim.xacro (robot description, xacro)
@@ -7,4 +7,5 @@
   <!-- 夹爪类型统一由 dual_arm_config.xacro 配置 -->
   <!-- UR 安全限位和路径参数 -->
+  <xacro:arg name="camera_use_nominal_extrinsics" default="false"/>
   <xacro:arg name="safety_limits" default="false"/>
   <xacro:arg name="safety_pos_margin" default="0.15"/>
@@ -13,4 +14,5 @@
   <!-- Jazzy: 纯描述入口，用于 RViz/MoveIt，不包含 ros2_control -->
   <xacro:space_sim
+    camera_use_nominal_extrinsics="$(arg camera_use_nominal_extrinsics)"
     safety_limits="$(arg safety_limits)"
     safety_pos_margin="$(arg safety_pos_margin)"

File: src/envs/space_sim/space_sim_description/xacro/space_sim_arm_macro.xacro (robot description, xacro)
@@ -2,7 +2,8 @@
 <robot xmlns:xacro="http://ros.org/wiki/xacro">
   <!-- ============================================ -->
-  <!-- 通用依赖（UR 机械臂本体）                    -->
+  <!-- 通用依赖（UR 机械臂本体 + RealSense 相机）   -->
   <!-- ============================================ -->
   <xacro:include filename="$(find ur_description)/urdf/ur_macro.xacro"/>
+  <xacro:include filename="$(find realsense2_description)/urdf/_d435.urdf.xacro" />
   <!-- ============================================ -->
   <!-- 夹爪类型条件依赖（预留，后续添加时启用）     -->
@@ -17,5 +18,5 @@
   </xacro:if>
   -->
-  <!-- 宏定义自己的机械臂结构 UR（无夹爪、无相机） -->
+  <!-- 宏定义自己的机械臂结构 UR + RealSense（无夹爪） -->
   <!-- Jazzy: 仅纯几何描述，不包含任何 ros2_control -->
   <xacro:macro name="space_sim_arm" params="
@@ -26,4 +27,5 @@
     kinematics_parameters_file:=''
     gripper_type:=none
+    realsense_use_nominal_extrinsics:=false
     safety_limits:=false
     safety_pos_margin:=0.15
@@ -45,4 +47,10 @@
     <xacro:property name="_ur_physical_parameters_file" value="$(find ur_description)/config/${ur_type}/physical_parameters.yaml"/>
     <xacro:property name="_ur_visual_parameters_file" value="$(find ur_description)/config/${ur_type}/visual_parameters.yaml"/>
+    <!-- RealSense parameters -->
+    <xacro:property name="_realsense_name" value="${tf_prefix}realsense" />
+    <xacro:property name="_realsense_prefix" value="${tf_prefix}realsense" />
+    <xacro:property name="_realsense_use_nominal_extrinsics" value="${realsense_use_nominal_extrinsics}" />
+    <xacro:property name="_realsense_add_plug" value="false" />
+    <xacro:property name="_realsense_use_mesh" value="true" />
     <!-- 创建 UR 机器人 使用宏定义 (Jazzy: 纯描述，无 ros2_control 参数) -->
     <xacro:ur_robot
@@ -62,16 +70,60 @@
     </xacro:ur_robot>
     <!-- ============================================ -->
+    <!-- RealSense 相机支架                           -->
+    <!-- 该支架的相机螺纹孔距离机械臂末端圆心100mm，  -->
+    <!-- 支架厚度3mm（与 lab_bench 使用同一支架）     -->
+    <!-- ============================================ -->
+    <link name="${_realsense_prefix}_shelf">
+      <inertial>
+        <origin xyz="0.0 0.044 0.0015" rpy="0.0 0.0 0.0"/>
+        <mass value="0.038"/>
+        <inertia ixx="0.00006673" ixy="0.0" ixz="0.0" iyy="0.00000850" iyz="0.0" izz="0.00007517"/>
+      </inertial>
+      <visual>
+        <geometry>
+          <mesh filename="package://space_sim_description/meshes/RealSense_D435_Shelf.STL"/>
+        </geometry>
+        <material name="anodized_aluminum">
+          <color rgba="0.7 0.7 0.7 1.0"/>
+        </material>
+      </visual>
+      <collision>
+        <geometry>
+          <mesh filename="package://space_sim_description/meshes/RealSense_D435_Shelf.STL"/>
+        </geometry>
+      </collision>
+    </link>
+    <joint name="${_realsense_prefix}_tool0_to_realsense_shelf" type="fixed">
+      <parent link="${_ur_tf_prefix}tool0"/>
+      <child link="${_realsense_prefix}_shelf"/>
+      <origin xyz="0.0 0.0 0.0" rpy="0 0 ${pi}" />
+    </joint>
+    <!-- ============================================ -->
+    <!-- RealSense D435 相机（无夹爪，直接挂在支架上） -->
+    <!-- ============================================ -->
+    <!-- params 'name' is actually tf_prefix with '_' -->
+    <xacro:sensor_d435
+      parent="${_realsense_prefix}_shelf"
+      name="${_realsense_prefix}"
+      use_nominal_extrinsics="${_realsense_use_nominal_extrinsics}"
+      add_plug="${_realsense_add_plug}"
+      use_mesh="${_realsense_use_mesh}"
+    >
+      <!-- RealSense 的基座位于相机底部的1/4螺纹孔，距离后背面10mm，底部平面距离后背2个螺纹孔所在直线12.5mm -->
+      <origin xyz="0 0.0875 0.013" rpy="0 ${-pi/2} ${-pi/2}"/>
+    </xacro:sensor_d435>
+    <!-- ============================================ -->
     <!-- 夹爪挂载点（预留）                            -->
     <!-- ============================================ -->
     <!--
       后续添加夹爪时，在此处根据 gripper_type 条件实例化夹爪宏，
-      父 link 为 ${_ur_tf_prefix}tool0。
+      父 link 为 ${_realsense_prefix}_shelf（相机支架末端）。
       示例（dh_ag95）：
       <xacro:if value="${gripper_type == 'dh_ag95'}">
         <xacro:dh_ag95_gripper
           prefix="${tf_prefix}dhag95_"
-          parent="${_ur_tf_prefix}tool0"
+          parent="${_realsense_prefix}_shelf"
         >
-          <origin xyz="0 0 0" rpy="0 0 0" />
+          <origin xyz="0 0 -0.0035" rpy="0 0 0" />
         </xacro:dh_ag95_gripper>
       </xacro:if>

File: src/envs/space_sim/space_sim_description/xacro/space_sim_macro.xacro (robot description, xacro)
@@ -5,4 +5,5 @@
   <!-- Jazzy: 纯几何描述，不包含 ros2_control -->
   <xacro:macro name="space_sim" params="
+  camera_use_nominal_extrinsics:=false
   safety_limits:=false
   safety_pos_margin:=0.15
@@ -11,24 +12,29 @@
   ">
   <!-- 定义材料 -->
-  <material name="cube_material">
-    <color rgba="0.55 0.55 0.60 1"/>
+  <material name="satellite_material">
+    <color rgba="0.70 0.60 0.20 1"/>
   </material>
-  <material name="hex_prism_material">
+  <material name="len_material">
     <color rgba="0.75 0.60 0.20 1"/>
   </material>
   <link name="world"/>
-  <!-- world 到 base_cube 的固定连接 -->
-  <joint name="world_to_base_cube" type="fixed">
+  <link name="base_link"/>
+  <joint name="world_to_base_link" type="fixed">
     <parent link="world" />
-    <child link="base_cube" />
+    <child link="base_link" />
+  </joint>
+  <!-- base_link 到 satellite 的固定连接 -->
+  <joint name="base_link_to_satellite" type="fixed">
+    <parent link="base_link" />
+    <child link="satellite" />
     <origin xyz="0 0 0" rpy="0 0 0" />
   </joint>
   <!-- ============================================ -->
-  <!-- 固定方块 base_cube (0.6*0.6*0.6 m, 300 kg)   -->
+  <!-- 固定方块 satellite (0.6*0.6*0.6 m, 300 kg)   -->
   <!-- 固定在 world 原点，中心在 (0,0,0)            -->
   <!-- 惯量: 均匀立方体 I = m/12*(a²+b²)           -->
   <!--       = 300/12*(0.6²+0.6²) = 18 kg·m²       -->
   <!-- ============================================ -->
-  <link name="base_cube">
+  <link name="satellite">
     <inertial>
       <mass value="300.0"/>
@@ -42,5 +48,5 @@
       </geometry>
       <origin rpy="0 0 0" xyz="0 0 0" />
-      <material name="cube_material"/>
+      <material name="satellite_material"/>
     </visual>
     <collision>
@@ -56,5 +62,5 @@
   <!-- 方块顶面 z = 0.3，棱柱中心 z = 0.3+0.025      -->
   <!-- ============================================ -->
-  <link name="hex_prism">
+  <link name="len_shelf">
     <inertial>
       <mass value="5.0"/>
@@ -68,20 +74,49 @@
     <visual>
       <geometry>
-        <mesh filename="package://space_sim_description/meshes/len.stl"/>
+        <cylinder radius="0.03" length="1.5"/>
       </geometry>
-      <origin rpy="0 0 0" xyz="0 0 0" />
-      <material name="hex_prism_material"/>
+      <origin rpy="0 0 0" xyz="0 0 0.75" />
+      <material name="len_material"/>
     </visual>
     <collision>
       <geometry>
-        <mesh filename="package://space_sim_description/meshes/len.stl"/>
+        <cylinder radius="0.03" length="1.5"/>
+      </geometry>
+      <origin rpy="0 0 0" xyz="0 0 0.75" />
+    </collision>
+  </link>
+  <joint name="satellite_to_len_shelf" type="fixed">
+    <parent link="satellite" />
+    <child link="len_shelf" />
+    <origin xyz="0 0 0.30" rpy="0 0 0" />
+  </joint>
+  <link name="len_center">
+    <inertial>
+      <mass value="5.0"/>
+      <!-- 正六边形棱柱: R=0.3/√3≈0.173205, h=0.05   -->
+      <!-- Izz = m*(5R²/12) = 0.0625                  -->
+      <!-- Ixx = Iyy = m*(5R²/24 + h²/12) ≈ 0.032292  -->
+      <inertia ixx="0.032292" ixy="0.0" ixz="0.0"
+               iyy="0.032292" iyz="0.0"
+               izz="0.0625"/>
+    </inertial>
+    <visual>
+      <geometry>
+        <mesh filename="package://space_sim_description/meshes/len_center.stl"/>
+      </geometry>
+      <origin rpy="0 0 0" xyz="0 0 0" />
+      <material name="len_material"/>
+    </visual>
+    <collision>
+      <geometry>
+        <mesh filename="package://space_sim_description/meshes/len_center.stl"/>
       </geometry>
       <origin rpy="0 0 0" xyz="0 0 0" />
     </collision>
   </link>
-  <joint name="base_cube_to_hex_prism" type="fixed">
-    <parent link="base_cube" />
-    <child link="hex_prism" />
-    <origin xyz="0 0 0.325" rpy="0 0 0" />
+  <joint name="len_shelf_to_center" type="fixed">
+    <parent link="len_shelf" />
+    <child link="len_center" />
+    <origin xyz="0 0 0.1" rpy="3.1416 0 0" />
   </joint>
   <!-- ============================================ -->
@@ -91,12 +126,12 @@
   <!-- ============================================ -->
   <link name="ur_mount_A"/>
-  <joint name="base_cube_to_ur_mount_A" type="fixed">
-    <parent link="base_cube"/>
+  <joint name="satellite_to_ur_mount_A" type="fixed">
+    <parent link="satellite"/>
     <child link="ur_mount_A"/>
     <origin xyz="0.3 0 0" rpy="0 ${pi/2} 0" />
   </joint>
   <link name="ur_mount_B"/>
-  <joint name="base_cube_to_ur_mount_B" type="fixed">
-    <parent link="base_cube"/>
+  <joint name="satellite_to_ur_mount_B" type="fixed">
+    <parent link="satellite"/>
     <child link="ur_mount_B"/>
     <origin xyz="-0.3 0 0" rpy="0 ${-pi/2} 0" />
@@ -110,4 +145,5 @@
     kinematics_parameters_file = "${ur_A_kinematics_parameters_file}"
     gripper_type = "${gripper_type}"
+    realsense_use_nominal_extrinsics = "${camera_use_nominal_extrinsics}"
     safety_limits = "${safety_limits}"
     safety_pos_margin = "${safety_pos_margin}"
@@ -124,4 +160,5 @@
     kinematics_parameters_file = "${ur_B_kinematics_parameters_file}"
     gripper_type = "${gripper_type}"
+    realsense_use_nominal_extrinsics = "${camera_use_nominal_extrinsics}"
     safety_limits = "${safety_limits}"
     safety_pos_margin = "${safety_pos_margin}"

File: src/envs/space_sim/space_sim_mujoco_description/xacro/ros2_control/space_sim_mujoco.xacro (robot description, xacro)
@@ -15,4 +15,9 @@
   <xacro:arg name="safety_k_position" default="20"/>
   <xacro:arg name="force_abs_paths" default="false"/>
+  <!-- 相机参数：
+       space_sim 双臂末端已挂载 RealSense D435 相机（几何描述），
+       launch_controller 的 mujoco 分支会统一传入
+       camera_use_nominal_extrinsics:=false，因此必须声明该 arg 并透传。 -->
+  <xacro:arg name="camera_use_nominal_extrinsics" default="false"/>
   <!-- ============================================ -->
   <!-- Mujoco ros2_control 可选参数                  -->
@@ -24,4 +29,5 @@
   <!-- Jazzy: 纯几何描述（仅传几何参数给 space_sim） -->
   <xacro:space_sim
+    camera_use_nominal_extrinsics="$(arg camera_use_nominal_extrinsics)"
     safety_limits="$(arg safety_limits)"
     safety_pos_margin="$(arg safety_pos_margin)"
