Commit message: 新增：完善了 space_sim 环境

File: src/envs/space_sim/space_sim_description/xacro/space_sim_arm_macro.xacro (robot description, xacro)
@@ -34,8 +34,10 @@
     *origin
     ">
+    <!-- 机械臂基座 parameters -->
+    <xacro:property name="_arm_base_name" value="${tf_prefix}base"/>
     <!-- UR parameters (Jazzy: 仅 yaml 配置文件路径) -->
     <xacro:property name="_ur_name" value="${name}_ur"/>
     <xacro:property name="_ur_tf_prefix" value="${tf_prefix}ur_"/>
-    <xacro:property name="_ur_parent" value="${parent}"/>
+    <xacro:property name="_ur_parent" value="${_arm_base_name}_main"/>
     <xacro:property name="_ur_joint_limits_parameters_file" value="$(find ur_description)/config/${ur_type}/joint_limits.yaml"/>
     <xacro:if value="${kinematics_parameters_file == ''}">
@@ -53,4 +55,61 @@
     <xacro:property name="_realsense_add_plug" value="false" />
     <xacro:property name="_realsense_use_mesh" value="true" />
+    <!-- gripper parameters -->
+    <xacro:property name="_gripper_name" value="${tf_prefix}gripper" />
+    <!-- 机械臂基座-->
+    <link name="${_arm_base_name}_dock">
+      <inertial>
+        <origin xyz="0.0 0.0 0.0" rpy="0.0 0.0 0.0"/>
+        <mass value="0.6"/>
+        <inertia ixx="0.0" ixy="0.0" ixz="0.0" iyy="0.0" iyz="0.0" izz="0.0"/>
+      </inertial>
+      <visual>
+        <geometry>
+          <cylinder radius="0.07" length="0.025"/>
+        </geometry>
+        <material name="arm_base_dock_material">
+          <color rgba="0.2 0.2 0.2 1"/>
+        </material>
+        <origin xyz="0 0 0" rpy="0 0 0"/>
+      </visual>
+      <collision>
+        <geometry>
+          <cylinder radius="0.07" length="0.025"/>
+        </geometry>
+        <origin xyz="0 0 0" rpy="0 0 0"/>
+      </collision>
+    </link>
+    <joint name="${_arm_base_name}_dock_joint" type="fixed">
+      <parent link="${parent}"/>
+      <child link="${_arm_base_name}_dock"/>
+      <origin xyz="0 0 0.0125" rpy="0 0 0"/>
+    </joint>
+    <link name="${_arm_base_name}_main">
+      <inertial>
+        <origin xyz="0.0 0.0 0.0" rpy="0.0 0.0 0.0"/>
+        <mass value="35.0"/>
+        <inertia ixx="0.182" ixy="0.0" ixz="0.0" iyy="0.182" iyz="0.0" izz="0.233"/>
+      </inertial>
+      <visual>
+        <geometry>
+          <box size="0.3 0.3 0.2"/>
+        </geometry>
+        <material name="arm_base_main_material">
+          <texture filename="package://space_sim_description/meshes/gold_leaf.png"/>
+        </material>
+        <origin xyz="0 0 0" rpy="0 0 0"/>
+      </visual>
+      <collision>
+        <geometry>
+          <box size="0.3 0.3 0.2"/>
+        </geometry>
+        <origin xyz="0 0 0" rpy="0 0 0"/>
+      </collision>
+    </link>
+    <joint name="${_arm_base_name}_dock_to_main_joint" type="fixed">
+      <parent link="${_arm_base_name}_dock"/>
+      <child link="${_arm_base_name}_main"/>
+      <origin xyz="0 0 0.1125" rpy="0 0 0"/>
+    </joint>
     <!-- 创建 UR 机器人 使用宏定义 (Jazzy: 纯描述，无 ros2_control 参数) -->
     <xacro:ur_robot
@@ -67,5 +126,6 @@
       force_abs_paths="${force_abs_paths}"
     >
-      <xacro:insert_block name="origin" />
+      <!-- <xacro:insert_block name="origin" /> -->
+      <origin xyz="0 0 0.1" rpy="0 0 0" />
     </xacro:ur_robot>
     <!-- ============================================ -->
@@ -98,4 +158,12 @@
       <child link="${_realsense_prefix}_shelf"/>
       <origin xyz="0.0 0.0 0.0" rpy="0 0 ${pi}" />
+    </joint>
+    <!-- 创建 RealSense 相机支架 child 端的 link 和 joint -->
+    <link name="${_realsense_prefix}_shelf_child_side"/>
+    <joint name="${_realsense_prefix}_shelf_to_child_side" type="fixed">
+      <parent link="${_realsense_prefix}_shelf"/>
+      <child link="${_realsense_prefix}_shelf_child_side"/>
+      <!-- 相机支架厚度 3mm + 夹爪底座坐标z轴偏移3mm -->
+      <origin xyz="0.0 0.0 0.006" rpy="0 0 0" />
     </joint>
     <!-- ============================================ -->
@@ -114,19 +182,64 @@
     </xacro:sensor_d435>
     <!-- ============================================ -->
-    <!-- 夹爪挂载点（预留）                            -->
-    <!-- ============================================ -->
-    <!--
-      后续添加夹爪时，在此处根据 gripper_type 条件实例化夹爪宏，
-      父 link 为 ${_realsense_prefix}_shelf（相机支架末端）。
-      示例（dh_ag95）：
-      <xacro:if value="${gripper_type == 'dh_ag95'}">
-        <xacro:dh_ag95_gripper
-          prefix="${tf_prefix}dhag95_"
-          parent="${_realsense_prefix}_shelf"
-        >
-          <origin xyz="0 0 -0.0035" rpy="0 0 0" />
-        </xacro:dh_ag95_gripper>
-      </xacro:if>
-    -->
+    <!-- 夹爪                                         -->
+    <!-- ============================================ -->
+    <link name="${_gripper_name}_base">
+      <inertial>
+        <origin xyz="0.0 0.0 0.055348" rpy="0.0 0.0 0.0"/>
+        <mass value="1.203"/>
+        <inertia ixx=" 0.001246" ixy="0.0" ixz="0.0" iyy="0.001777" iyz="0.0" izz="0.001085"/>
+      </inertial>
+      <visual>
+        <geometry>
+          <mesh filename="package://space_sim_description/meshes/magnetic_gripper.STL"/>
+        </geometry>
+        <material name="gripper_base_material">
+          <color rgba="0.6 0.6 0.6 1"/>
+        </material>
+      </visual>
+      <collision>
+        <geometry>
+          <mesh filename="package://space_sim_description/meshes/magnetic_gripper.STL"/>
+        </geometry>
+      </collision>
+    </link>
+    <joint name="${_realsense_prefix}_shelf_to_${_gripper_name}_base" type="fixed">
+      <parent link="${_realsense_prefix}_shelf_child_side"/>
+      <child link="${_gripper_name}_base"/>
+      <origin xyz="0 0 0" rpy="0 0 0"/>
+    </joint>
+    <link name="${_gripper_name}_dock">
+      <inertial>
+        <origin xyz="0.0 0.0 0.0" rpy="0.0 0.0 0.0"/>
+        <mass value="0.3"/>
+        <inertia ixx="0.0001" ixy="0.0" ixz="0.0" iyy="0.0001" iyz="0.0" izz="0.0001"/>
+      </inertial>
+      <visual>
+        <geometry>
+          <box size="0.1 0.04 0.02"/>
+        </geometry>
+        <material name="gripper_dock_material">
+          <color rgba="0.2 0.2 0.2 1"/>
+        </material>
+        <origin xyz="0 0 0.01" rpy="0 0 0"/>
+      </visual>
+      <collision>
+        <geometry>
+          <box size="0.1 0.04 0.02"/>
+        </geometry>
+        <origin xyz="0 0 0.01" rpy="0 0 0"/>
+      </collision>
+    </link>
+    <joint name="${_gripper_name}_base_to_${_gripper_name}_dock" type="fixed">
+      <parent link="${_gripper_name}_base"/>
+      <child link="${_gripper_name}_dock"/>
+      <origin xyz="0 0 0.1" rpy="0 0 0"/>
+    </joint>
+    <link name="${tf_prefix}_tcp"/>
+      <joint name="${tf_prefix}_tcp_joint" type="fixed">
+          <origin xyz="0 0 0.12" rpy="0 0 0"/>
+          <parent link="${_gripper_name}_base"/>
+          <child link="${tf_prefix}_tcp"/>
+      </joint>
   </xacro:macro>
 </robot>

File: src/envs/space_sim/space_sim_description/xacro/space_sim_macro.xacro (robot description, xacro)
@@ -13,8 +13,8 @@
   <!-- 定义材料 -->
   <material name="satellite_material">
-    <color rgba="0.70 0.60 0.20 1"/>
+    <texture filename="package://space_sim_description/meshes/gold_leaf.png" />
   </material>
-  <material name="len_material">
-    <color rgba="0.75 0.60 0.20 1"/>
+  <material name="len_shelf_material">
+    <color rgba="0.60 0.60 0.60 1"/>
   </material>
   <link name="world"/>
@@ -39,7 +39,5 @@
     <inertial>
       <mass value="300.0"/>
-      <inertia ixx="18.0" ixy="0.0" ixz="0.0"
-               iyy="18.0" iyz="0.0"
-               izz="18.0"/>
+      <inertia ixx="18.0" ixy="0.0" ixz="0.0" iyy="18.0" iyz="0.0" izz="18.0"/>
     </inertial>
     <visual>
@@ -58,28 +56,29 @@
   </link>
   <!-- ============================================ -->
-  <!-- 正六边棱柱 hex_prism                          -->
-  <!-- 对向边距 0.3m，高 0.05m，固定在方块顶面中心   -->
-  <!-- 方块顶面 z = 0.3，棱柱中心 z = 0.3+0.025      -->
-  <!-- ============================================ -->
+  <!-- 镜片部分                                      -->
+  <!-- ============================================ -->
+  <!-- 镜片支架 -->
   <link name="len_shelf">
     <inertial>
       <mass value="5.0"/>
-      <!-- 正六边形棱柱: R=0.3/√3≈0.173205, h=0.05   -->
-      <!-- Izz = m*(5R²/12) = 0.0625                  -->
-      <!-- Ixx = Iyy = m*(5R²/24 + h²/12) ≈ 0.032292  -->
-      <inertia ixx="0.032292" ixy="0.0" ixz="0.0"
-               iyy="0.032292" iyz="0.0"
-               izz="0.0625"/>
-    </inertial>
-    <visual>
-      <geometry>
-        <cylinder radius="0.03" length="1.5"/>
+      <inertia ixx="0.032292" ixy="0.0" ixz="0.0" iyy="0.032292" iyz="0.0" izz="0.0625"/>
+    </inertial>
+    <visual>
+      <geometry>
+        <cylinder radius="0.02" length="1.5"/>
       </geometry>
       <origin rpy="0 0 0" xyz="0 0 0.75" />
-      <material name="len_material"/>
-    </visual>
-    <collision>
-      <geometry>
-        <cylinder radius="0.03" length="1.5"/>
+      <material name="len_shelf_material"/>
+    </visual>
+    <visual>
+      <geometry>
+        <cylinder radius="0.05" length="0.08"/>
+      </geometry>
+      <origin rpy="0 0 0" xyz="0 0 1.5" />
+      <material name="len_shelf_material"/>
+    </visual>
+    <collision>
+      <geometry>
+        <cylinder radius="0.02" length="1.5"/>
       </geometry>
       <origin rpy="0 0 0" xyz="0 0 0.75" />
@@ -91,26 +90,19 @@
     <origin xyz="0 0 0.30" rpy="0 0 0" />
   </joint>
+  <!-- 中心镜片 -->
   <link name="len_center">
     <inertial>
       <mass value="5.0"/>
-      <!-- 正六边形棱柱: R=0.3/√3≈0.173205, h=0.05   -->
-      <!-- Izz = m*(5R²/12) = 0.0625                  -->
-      <!-- Ixx = Iyy = m*(5R²/24 + h²/12) ≈ 0.032292  -->
-      <inertia ixx="0.032292" ixy="0.0" ixz="0.0"
-               iyy="0.032292" iyz="0.0"
-               izz="0.0625"/>
-    </inertial>
-    <visual>
+      <inertia ixx="0.032292" ixy="0.0" ixz="0.0" iyy="0.032292" iyz="0.0" izz="0.0625"/>
+    </inertial>
+    <visual>
+      <geometry>
+        <mesh filename="package://space_sim_description/meshes/len_center.obj"/>
+      </geometry>
+    </visual>
+    <collision>
       <geometry>
         <mesh filename="package://space_sim_description/meshes/len_center.stl"/>
       </geometry>
-      <origin rpy="0 0 0" xyz="0 0 0" />
-      <material name="len_material"/>
-    </visual>
-    <collision>
-      <geometry>
-        <mesh filename="package://space_sim_description/meshes/len_center.stl"/>
-      </geometry>
-      <origin rpy="0 0 0" xyz="0 0 0" />
     </collision>
   </link>
@@ -118,5 +110,75 @@
     <parent link="len_shelf" />
     <child link="len_center" />
-    <origin xyz="0 0 0.1" rpy="3.1416 0 0" />
+    <origin xyz="0 0 0.1" rpy="0 0 0" />
+  </joint>
+  <!-- <link name="len_ring1_1">
+    <inertial>
+      <mass value="5.0"/>
+      <inertia ixx="0.032292" ixy="0.0" ixz="0.0" iyy="0.032292" iyz="0.0" izz="0.0625"/>
+    </inertial>
+    <visual>
+      <geometry>
+        <mesh filename="package://space_sim_description/meshes/len_ring1.obj"/>
+      </geometry>
+    </visual>
+    <collision>
+      <geometry>
+        <mesh filename="package://space_sim_description/meshes/len_ring1.stl"/>
+      </geometry>
+    </collision>
+  </link>
+  <joint name="len_center_to_ring1_1" type="fixed">
+    <parent link="len_center" />
+    <child link="len_ring1_1" />
+    <origin xyz="-0.5130 -0.0000 0.0905" rpy="-0.349066 -0.000000 -1.570796"/>
+  </joint> -->
+  <!-- ============================================ -->
+  <!-- 卫星附件 太阳能板                            -->
+  <!-- 对侧安装: 在 +/-Y 侧面                       -->
+  <!-- 方块半宽 0.3，安装面在 y=±0.3                -->
+  <!-- ============================================ -->
+  <link name="solar_panel_A">
+    <inertial>
+      <mass value="6.580"/>
+      <origin xyz="-1.309 0.003 0.000" rpy="0 0 0" />
+      <inertia ixx="0.1246" ixy="0.0" ixz="0.0" iyy="2.090" iyz="0.0" izz="1.965"/>
+    </inertial>
+    <visual>
+      <geometry>
+        <mesh filename="package://space_sim_description/meshes/solar_panel.obj"/>
+      </geometry>
+    </visual>
+    <collision>
+      <geometry>
+        <mesh filename="package://space_sim_description/meshes/solar_panel.obj"/>
+      </geometry>
+    </collision>
+  </link>
+  <joint name="satellite_to_solar_panel_A" type="fixed">
+    <parent link="satellite" />
+    <child link="solar_panel_A" />
+    <origin xyz="0 0.3 0" rpy="0 0 ${-pi/2}" />
+  </joint>
+  <link name="solar_panel_B">
+    <inertial>
+      <mass value="6.580"/>
+      <origin xyz="-1.309 0.003 0.000" rpy="0 0 0" />
+      <inertia ixx="0.1246" ixy="0.0" ixz="0.0" iyy="2.090" iyz="0.0" izz="1.965"/>
+    </inertial>
+    <visual>
+      <geometry>
+        <mesh filename="package://space_sim_description/meshes/solar_panel.obj"/>
+      </geometry>
+    </visual>
+    <collision>
+      <geometry>
+        <mesh filename="package://space_sim_description/meshes/solar_panel.obj"/>
+      </geometry>
+    </collision>
+  </link>
+  <joint name="satellite_to_solar_panel_B" type="fixed">
+    <parent link="satellite" />
+    <child link="solar_panel_B" />
+    <origin xyz="0 -0.3 0" rpy="0 0 ${pi/2}" />
   </joint>
   <!-- ============================================ -->

Commit message: 新增：添加了 space_sim 环境的六个镜片；添加了对接口模拟插件

File: src/envs/space_sim/space_sim_description/xacro/space_sim_arm_macro.xacro (robot description, xacro)
@@ -165,5 +165,5 @@
       <child link="${_realsense_prefix}_shelf_child_side"/>
       <!-- 相机支架厚度 3mm + 夹爪底座坐标z轴偏移3mm -->
-      <origin xyz="0.0 0.0 0.006" rpy="0 0 0" />
+      <origin xyz="0.0 0.0 0.003" rpy="0 0 0" />
     </joint>
     <!-- ============================================ -->

File: src/envs/space_sim/space_sim_description/xacro/space_sim_macro.xacro (robot description, xacro)
@@ -3,4 +3,5 @@
   <xacro:include filename="$(find space_sim_description)/xacro/dual_arm_config.xacro"/>
   <xacro:include filename="$(find space_sim_description)/xacro/space_sim_arm_macro.xacro"/>
+  <xacro:include filename="$(find space_sim_description)/xacro/len_macro.xacro"/>
   <!-- Jazzy: 纯几何描述，不包含 ros2_control -->
   <xacro:macro name="space_sim" params="
@@ -112,25 +113,4 @@
     <origin xyz="0 0 0.1" rpy="0 0 0" />
   </joint>
-  <!-- <link name="len_ring1_1">
-    <inertial>
-      <mass value="5.0"/>
-      <inertia ixx="0.032292" ixy="0.0" ixz="0.0" iyy="0.032292" iyz="0.0" izz="0.0625"/>
-    </inertial>
-    <visual>
-      <geometry>
-        <mesh filename="package://space_sim_description/meshes/len_ring1.obj"/>
-      </geometry>
-    </visual>
-    <collision>
-      <geometry>
-        <mesh filename="package://space_sim_description/meshes/len_ring1.stl"/>
-      </geometry>
-    </collision>
-  </link>
-  <joint name="len_center_to_ring1_1" type="fixed">
-    <parent link="len_center" />
-    <child link="len_ring1_1" />
-    <origin xyz="-0.5130 -0.0000 0.0905" rpy="-0.349066 -0.000000 -1.570796"/>
-  </joint> -->
   <!-- ============================================ -->
   <!-- 卫星附件 太阳能板                            -->
@@ -182,4 +162,9 @@
     <origin xyz="0 -0.3 0" rpy="0 0 ${pi/2}" />
   </joint>
+  <!-- ============================================ -->
+  <!-- 卫星底部镜片接口盘 + 6 个镜片接口 + 6 片待装配镜片 -->
+  <!-- 详见 len_macro.xacro 中的几何说明            -->
+  <!-- ============================================ -->
+  <xacro:len_dock_assembly_macro parent="satellite"/>
   <!-- ============================================ -->
   <!-- UR 安装座 link & joint                        -->
